File: eagle/ProjectX/Amplifier.brd (EAGLE design)
At the start: 100 x 80 mm, 5 parts, among them U1 TC4427COA

Commit message: Board update
Parts:
- added C3: 4.7uF, rcl:C0805
- added C4: 100nF, rcl:C0805
- added U2: TC4427COA, Microchip_By_element14_Batch_1:SOIC127P600X175-8N
- moved SV1 17.5 mm to (53.3, 24.1)
- moved C1 12.1 mm to (80.0, 43.4), flipped to the top, turned to 180 degrees
- moved C2 8.89 mm to (80.0, 45.7), flipped to the top, turned to 180 degrees
- moved U1 3.30 mm to (79.8, 50.0), flipped to the top, turned to 0 degrees
Connections:
- new net N$1: SV2.34, U2.4
- new net N$6: SV2.36, U2.2
- new net N$7: SV1.35, U2.7
- new net N$8: SV1.33, U2.5
- net GND: now also C3.2, C4.2, U2.3
- net N$2: now also U1.7; no longer U1.5
- net N$3: now also U1.5; no longer U1.7
- net N$4: now also SV2.38; no longer SV2.40
- net N$5: now also SV2.40; no longer SV2.38
- net VCC: now also C3.1, C4.1, U2.6
Routing:
- net VCC: track 8.01 -> 0.00 mm
- net GND: track 2.29 -> 0.00 mm
