File: eagle/ProjectX/BigDaddy.brd (EAGLE design)
At the start: 100 x 100 mm, 180 parts, among them U10 TC4427AEOA, U11 TC4427AEOA, U12 TC4427AEOA, U13 TC4427AEOA, U19 TC4427AEOA, U20 TC4427AEOA, U21 TC4427AEOA, U22 TC4427AEOA, U23 TC4427AEOA, U24 TC4427AEOA, U25 TC4427AEOA, U26 TC4427AEOA, U27 TC4427AEOA, U28 TC4427AEOA, U29 TC4427AEOA, U3 TC4427AEOA, U30 TC4427AEOA, U31 TC4427AEOA, U32 TC4427AEOA, U34 TC4427AEOA, U35 TC4427AEOA, U36 TC4427AEOA, U37 TC4427AEOA, U38 TC4427AEOA, U39 TC4427AEOA, U4 TC4427AEOA, U40 TC4427AEOA, U41 TC4427AEOA, U42 TC4427AEOA, U43 TC4427AEOA, U44 TC4427AEOA, U45 TC4427AEOA, U5 TC4427AEOA, U55 TC4427AEOA, U56 TC4427AEOA, U57 TC4427AEOA, U58 TC4427AEOA, U59 TC4427AEOA, U60 TC4427AEOA, U61 TC4427AEOA, U62 TC4427AEOA, U63 TC4427AEOA, U7 TC4427AEOA, U9 TC4427AEOA

Commit message: Netted up all the remaining amplifiers, need to route and net the FPGA pins to the amplifiers
Connections:
- new net 17: U12.4
- new net 18: U12.2
- new net 19: U4.4
- new net 20: U4.2
- new net 21: U10.4
- new net 22: U10.2
- new net 23: U7.4
- new net 24: U7.2
- new net 25: U11.2
- new net 26: U3.4
- new net 27: U3.2
- new net 28: U5.4
- new net 29: U5.2
- new net 30: U13.4
- new net 31: U13.2
- new net 32: U9.4
- new net 33: U9.2
- new net 34: U11.4
- new net 35: U19.4
- new net 36: U19.2
- new net 37: U24.4
- new net 38: U24.2
- new net 39: U26.4
- new net 40: U26.2
- new net 41: U21.4
- new net 42: U21.2
- new net 43: U23.2
- new net 44: U20.4
- new net 45: U20.2
- new net 46: U25.4
- new net 47: U25.2
- new net 48: U27.4
- new net 49: U27.2
- new net 50: U22.4
- new net 51: U22.2
- new net 52: U23.4
- new net 53: U37.4
- new net 54: U37.2
- new net 55: U42.4
- new net 56: U42.2
- new net 57: U44.4
- new net 58: U44.2
- new net 59: U39.4
- new net 60: U39.2
- new net 61: U41.2
- new net 62: U38.4
- new net 63: U38.2
- new net 64: U43.4
- new net 65: U43.2
- new net 66: U45.4
- new net 67: U45.2
- new net 68: U40.4
- new net 69: U40.2
- new net 70: U41.4
- new net 71: U55.4
- new net 72: U55.2
- new net 73: U60.4
- new net 74: U60.2
- new net 75: U62.4
- new net 76: U62.2
- new net 77: U57.4
- new net 78: U57.2
- new net 79: U59.2
- new net 80: U56.4
- new net 81: U56.2
- new net 82: U61.4
- new net 83: U61.2
- new net 84: U63.4
- new net 85: U63.2
- new net 86: U58.4
- new net 87: U58.2
- new net 88: U59.4
Changed lines of the file:
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@@
 <grid distance="9.84251969" unitdist="mil" unit="mil" style="lines" multiple="1" display="yes" altdistance="787.401575" altunitdist="mil" altunit="mil"/>
 <layers>
-<layer number="1" name="Top" color="4" fill="1" visible="no" active="yes"/>
+<layer number="1" name="Top" color="4" fill="1" visible="yes" active="yes"/>
 <layer number="2" name="Route2" color="1" fill="3" visible="no" active="no"/>
 <layer number="3" name="Route3" color="4" fill="3" visible="no" active="no"/>
@@
 <layer number="19" name="Unrouted" color="6" fill="1" visible="yes" active="yes"/>
 <layer number="20" name="Dimension" color="24" fill="1" visible="yes" active="yes"/>
-<layer number="21" name="tPlace" color="7" fill="1" visible="no" active="yes"/>
+<layer number="21" name="tPlace" color="7" fill="1" visible="yes" active="yes"/>
 <layer number="22" name="bPlace" color="7" fill="1" visible="yes" active="yes"/>
-<layer number="23" name="tOrigins" color="15" fill="1" visible="no" active="yes"/>
+<layer number="23" name="tOrigins" color="15" fill="1" visible="yes" active="yes"/>
 <layer number="24" name="bOrigins" color="15" fill="1" visible="yes" active="yes"/>
-<layer number="25" name="tNames" color="7" fill="1" visible="no" active="yes"/>
+<layer number="25" name="tNames" color="7" fill="1" visible="yes" active="yes"/>
 <layer number="26" name="bNames" color="7" fill="1" visible="yes" active="yes"/>
-<layer number="27" name="tValues" color="7" fill="1" visible="no" active="yes"/>
-<layer number="28" name="bValues" color="7" fill="1" visible="no" active="yes"/>
+<layer number="27" name="tValues" color="7" fill="1" visible="yes" active="yes"/>
+<layer number="28" name="bValues" color="7" fill="1" visible="yes" active="yes"/>
 <layer number="29" name="tStop" color="7" fill="3" visible="no" active="yes"/>
 <layer number="30" name="bStop" color="7" fill="6" visible="no" active="yes"/>
@@
 <layer number="37" name="tTest" color="7" fill="1" visible="no" active="yes"/>
 <layer number="38" name="bTest" color="7" fill="1" visible="no" active="yes"/>
-<layer number="39" name="tKeepout" color="4" fill="11" visible="no" active="yes"/>
+<layer number="39" name="tKeepout" color="4" fill="11" visible="yes" active="yes"/>
 <layer number="40" name="bKeepout" color="1" fill="11" visible="yes" active="yes"/>
-<layer number="41" name="tRestrict" color="4" fill="10" visible="no" active="yes"/>
+<layer number="41" name="tRestrict" color="4" fill="10" visible="yes" active="yes"/>
 <layer number="42" name="bRestrict" color="1" fill="10" visible="yes" active="yes"/>
 <layer number="43" name="vRestrict" color="2" fill="10" visible="no" active="yes"/>
-<layer number="44" name="Drills" color="7" fill="1" visible="no" active="yes"/>
+<layer number="44" name="Drills" color="7" fill="1" visible="yes" active="yes"/>
 <layer number="45" name="Holes" color="7" fill="1" visible="yes" active="yes"/>
 <layer number="46" name="Milling" color="3" fill="1" visible="no" active="yes"/>
@@
 <layer number="49" name="Reference" color="7" fill="1" visible="no" active="yes"/>
 <layer number="50" name="dxf" color="7" fill="1" visible="no" active="no"/>
-<layer number="51" name="tDocu" color="7" fill="1" visible="no" active="yes"/>
+<layer number="51" name="tDocu" color="7" fill="1" visible="yes" active="yes"/>
 <layer number="52" name="bDocu" color="7" fill="1" visible="yes" active="yes"/>
 <layer number="53" name="tGND_GNDA" color="7" fill="9" visible="no" active="no"/>
@@
 <wire x1="51.814475" y1="89.9908" x2="48.2408" y2="89.9908" width="0.254" layer="16"/>
 </signal>
+<signal name="17">
+<contactref element="U12" pad="4"/>
+</signal>
+<signal name="18">
+<contactref element="U12" pad="2"/>
+</signal>
+<signal name="19">
+<contactref element="U4" pad="4"/>
+</signal>
+<signal name="20">
+<contactref element="U4" pad="2"/>
+</signal>
+<signal name="21">
+<contactref element="U10" pad="4"/>
+</signal>
+<signal name="22">
+<contactref element="U10" pad="2"/>
+</signal>
+<signal name="23">
+<contactref element="U7" pad="4"/>
+</signal>
+<signal name="24">
+<contactref element="U7" pad="2"/>
+</signal>
+<signal name="25">
+<contactref element="U11" pad="2"/>
+</signal>
+<signal name="27">
+<contactref element="U3" pad="2"/>
+</signal>
+<signal name="26">
+<contactref element="U3" pad="4"/>
+</signal>
+<signal name="28">
+<contactref element="U5" pad="4"/>
+</signal>
+<signal name="29">
+<contactref element="U5" pad="2"/>
+</signal>
+<signal name="30">
+<contactref element="U13" pad="4"/>
+</signal>
+<signal name="31">
+<contactref element="U13" pad="2"/>
+</signal>
+<signal name="32">
+<contactref element="U9" pad="4"/>
+</signal>
+<signal name="33">
+<contactref element="U9" pad="2"/>
+</signal>
+<signal name="34">
+<contactref element="U11" pad="4"/>
+</signal>
+<signal name="35">
+<contactref element="U19" pad="4"/>
+</signal>
+<signal name="36">
+<contactref element="U19" pad="2"/>
+</signal>
+<signal name="37">
+<contactref element="U24" pad="4"/>
+</signal>
+<signal name="38">
+<contactref element="U24" pad="2"/>
+</signal>
+<signal name="39">
+<contactref element="U26" pad="4"/>
+</signal>
+<signal name="40">
+<contactref element="U26" pad="2"/>
+</signal>
+<signal name="41">
+<contactref element="U21" pad="4"/>
+</signal>
+<signal name="42">
+<contactref element="U21" pad="2"/>
+</signal>
+<signal name="43">
+<contactref element="U23" pad="2"/>
+</signal>
+<signal name="52">
+<contactref element="U23" pad="4"/>
+</signal>
+<signal name="44">
+<contactref element="U20" pad="4"/>
+</signal>
+<signal name="45">
+<contactref element="U20" pad="2"/>
+</signal>
+<signal name="46">
+<contactref element="U25" pad="4"/>
+</signal>
+<signal name="47">
+<contactref element="U25" pad="2"/>
+</signal>
+<signal name="48">
+<contactref element="U27" pad="4"/>
+</signal>
+<signal name="49">
+<contactref element="U27" pad="2"/>
+</signal>
+<signal name="50">
+<contactref element="U22" pad="4"/>
+</signal>
+<signal name="51">
+<contactref element="U22" pad="2"/>
+</signal>
+<signal name="53">
+<contactref element="U37" pad="4"/>
+</signal>
+<signal name="54">
+<contactref element="U37" pad="2"/>
+</signal>
+<signal name="55">
+<contactref element="U42" pad="4"/>
+</signal>
+<signal name="56">
+<contactref element="U42" pad="2"/>
+</signal>
+<signal name="57">
+<contactref element="U44" pad="4"/>
+</signal>
+<signal name="58">
+<contactref element="U44" pad="2"/>
+</signal>
+<signal name="59">
+<contactref element="U39" pad="4"/>
+</signal>
+<signal name="60">
+<contactref element="U39" pad="2"/>
+</signal>
+<signal name="61">
+<contactref element="U41" pad="2"/>
+</signal>
+<signal name="70">
+<contactref element="U41" pad="4"/>
+</signal>
+<signal name="62">
+<contactref element="U38" pad="4"/>
+</signal>
+<signal name="63">
+<contactref element="U38" pad="2"/>
+</signal>
+<signal name="64">
+<contactref element="U43" pad="4"/>
+</signal>
+<signal name="65">
+<contactref element="U43" pad="2"/>
+</signal>
+<signal name="66">
+<contactref element="U45" pad="4"/>
+</signal>
+<signal name="67">
+<contactref element="U45" pad="2"/>
+</signal>
+<signal name="68">
+<contactref element="U40" pad="4"/>
+</signal>
+<signal name="69">
+<contactref element="U40" pad="2"/>
+</signal>
+<signal name="71">
+<contactref element="U55" pad="4"/>
+</signal>
+<signal name="72">
+<contactref element="U55" pad="2"/>
+</signal>
+<signal name="73">
+<contactref element="U60" pad="4"/>
+</signal>
+<signal name="74">
+<contactref element="U60" pad="2"/>
+</signal>
+<signal name="75">
+<contactref element="U62" pad="4"/>
+</signal>
+<signal name="76">
+<contactref element="U62" pad="2"/>
+</signal>
+<signal name="77">
+<contactref element="U57" pad="4"/>
+</signal>
+<signal name="78">
+<contactref element="U57" pad="2"/>
+</signal>
+<signal name="79">
+<contactref element="U59" pad="2"/>
+</signal>
+<signal name="88">
+<contactref element="U59" pad="4"/>
+</signal>
+<signal name="80">
+<contactref element="U56" pad="4"/>
+</signal>
+<signal name="81">
+<contactref element="U56" pad="2"/>
+</signal>
+<signal name="82">
+<contactref element="U61" pad="4"/>
+</signal>
+<signal name="83">
+<contactref element="U61" pad="2"/>
+</signal>
+<signal name="84">
+<contactref element="U63" pad="4"/>
+</signal>
+<signal name="85">
+<contactref element="U63" pad="2"/>
+</signal>
+<signal name="86">
+<contactref element="U58" pad="4"/>
+</signal>
+<signal name="87">
+<contactref element="U58" pad="2"/>
+</signal>
 </signals>

Commit message: About 40% complete wiring of signals
Connections:
- net 10: now also DIP1.192; no longer DIP1.189
- net 11: now also DIP1.189; no longer DIP1.186
- net 17: now also DIP1.11
- net 18: now also DIP1.15
- net 19: now also DIP1.19
- net 20: now also DIP1.16
- net 21: now also DIP1.186
- net 22: now also DIP1.181
- net 26: now also DIP1.30
- net 27: now also DIP1.33
- net 28: now also DIP1.31
- net 29: now also DIP1.29
- net 35: now also DIP1.35
- net 36: now also DIP1.39
- net 37: now also DIP1.40
- net 38: now also DIP1.36
- net 44: now also DIP1.41
- net 45: now also DIP1.45
- net 46: now also DIP1.47
- net 47: now also DIP1.42
- net 53: now also DIP1.48
- net 54: now also DIP1.50
- net 55: now also DIP1.55
- net 56: now also DIP1.49
- net 62: now also DIP1.77
- net 63: now also DIP1.75
- net 64: now also DIP1.63
- net 65: now also DIP1.61
- net 71: now also DIP1.69
- net 72: now also DIP1.64
- net 73: now also DIP1.74
- net 74: now also DIP1.65
- net 80: now also DIP1.62
- net 81: now also DIP1.60
- net 82: now also DIP1.82
- net 83: now also DIP1.76
Routing:
- net 81: track 0.00 -> 51.8 mm
- net 80: track 0.00 -> 51.6 mm
- net 72: track 0.00 -> 37.1 mm
- net 71: track 0.00 -> 36.8 mm
- net 22: track 0.00 -> 27.7 mm, vias 0 -> 2
- net 53: track 0.00 -> 25.4 mm
- net 21: track 0.00 -> 25.2 mm, vias 0 -> 2
- net 63: track 0.00 -> 22.3 mm
- net 62: track 0.00 -> 21.3 mm
- net 54: track 0.00 -> 20.7 mm
- net 44: track 0.00 -> 18.3 mm, vias 0 -> 2
- net 20: track 0.00 -> 15.1 mm
- net 35: track 0.00 -> 14.7 mm
- net 45: track 0.00 -> 14.6 mm, vias 0 -> 2
- net 17: track 0.00 -> 12.6 mm
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