File: eagle/ProjectX/BigDaddy.brd (EAGLE design)
At the start: 100 x 100 mm, 180 parts, among them T1 MA40S4S, T10 MA40S4S, T11 MA40S4S, T12 MA40S4S, T13 MA40S4S, T14 MA40S4S, T15 MA40S4S, T16 MA40S4S, T17 MA40S4S, T18 MA40S4S, T19 MA40S4S, T2 MA40S4S, T20 MA40S4S, T21 MA40S4S, T22 MA40S4S, T23 MA40S4S, T24 MA40S4S, T25 MA40S4S, T26 MA40S4S, T27 MA40S4S, T28 MA40S4S, T3 MA40S4S, T30 MA40S4S, T31 MA40S4S, T32 MA40S4S, T33 MA40S4S, T34 MA40S4S, T35 MA40S4S, T36 MA40S4S, T37 MA40S4S, T38 MA40S4S, T39 MA40S4S, T4 MA40S4S, T40 MA40S4S, T41 MA40S4S, T42 MA40S4S, T43 MA40S4S, T44 MA40S4S, T45 MA40S4S, T46 MA40S4S, T47 MA40S4S, T48 MA40S4S, T49 MA40S4S, T5 MA40S4S, T50 MA40S4S, T51 MA40S4S, T52 MA40S4S, T53 MA40S4S, T54 MA40S4S, T55 MA40S4S, T56 MA40S4S, T57 MA40S4S, T58 MA40S4S, T59 MA40S4S, T6 MA40S4S, T60 MA40S4S, T61 MA40S4S, T62 MA40S4S, T63 MA40S4S, T64 MA40S4S, T65 MA40S4S, T66 MA40S4S, T67 MA40S4S, T68 MA40S4S, T69 MA40S4S, T7 MA40S4S, T70 MA40S4S, T71 MA40S4S, T72 MA40S4S, T73 MA40S4S, T74 MA40S4S, T75 MA40S4S, T76 MA40S4S, T77 MA40S4S, T78 MA40S4S, T79 MA40S4S, T8 MA40S4S, T80 MA40S4S, T81 MA40S4S, T82 MA40S4S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

Commit message: Numbering T29
Parts:
- renumbered 29 to T29
Changed lines of the file:
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@@
 <attribute name="VALUE" x="29.96" y="76.27" size="1.27" layer="27" rot="R270"/>
 </element>
-<element name="29" library="Parts" package="MA40" value="MA40S4S" x="40" y="65" rot="MR270"/>
+<element name="T29" library="Parts" package="MA40" value="MA40S4S" x="40" y="65" rot="MR270"/>
 <element name="T28" library="Parts" package="MA40" value="MA40S4S" x="30" y="65" rot="MR270"/>
 <element name="U5" library="Parts" package="SOIC127P600X175-8N" value="TC4427AEOA" x="36" y="65" rot="R270">
@@
 <contactref element="U4" pad="3"/>
 <contactref element="C4" pad="1"/>
-<contactref element="29" pad="-"/>
+<contactref element="T29" pad="-"/>
 <contactref element="T28" pad="-"/>
 <contactref element="U5" pad="3"/>
@@
 <signal name="N$9">
 <contactref element="U5" pad="7"/>
-<contactref element="29" pad="+"/>
+<contactref element="T29" pad="+"/>
 <wire x1="38.4144" y1="64.0856" x2="40" y2="62.5" width="0.508" layer="1"/>
 <wire x1="36.635" y1="62.6378" x2="36.635" y2="64.0856" width="0.508" layer="1"/>
