File: eagle/ProjectX/BigDaddy.sch (EAGLE design)
At the start: 180 parts, among them U10 TC4427AEOA, U11 TC4427AEOA, U12 TC4427AEOA, U13 TC4427AEOA, U19 TC4427AEOA, U20 TC4427AEOA, U21 TC4427AEOA, U22 TC4427AEOA, U23 TC4427AEOA, U24 TC4427AEOA, U25 TC4427AEOA, U26 TC4427AEOA, U27 TC4427AEOA, U28 TC4427AEOA, U29 TC4427AEOA, U3 TC4427AEOA, U30 TC4427AEOA, U31 TC4427AEOA, U32 TC4427AEOA, U34 TC4427AEOA, U35 TC4427AEOA, U36 TC4427AEOA, U37 TC4427AEOA, U38 TC4427AEOA, U39 TC4427AEOA, U4 TC4427AEOA, U40 TC4427AEOA, U41 TC4427AEOA, U42 TC4427AEOA, U43 TC4427AEOA, U44 TC4427AEOA, U45 TC4427AEOA, U5 TC4427AEOA, U55 TC4427AEOA, U56 TC4427AEOA, U57 TC4427AEOA, U58 TC4427AEOA, U59 TC4427AEOA, U60 TC4427AEOA, U61 TC4427AEOA, U62 TC4427AEOA, U63 TC4427AEOA, U7 TC4427AEOA, U9 TC4427AEOA

Commit message: Still routing traces
Parts:
- J1: value (none) -> +20V
- J2: value (none) -> Data
Connections:
- net 23: now also DIP1.152
- net 24: now also DIP1.160
- net 25: now also DIP1.150
- net 30: now also DIP1.153
- net 31: now also DIP1.151
- net 34: now also DIP1.146
- net 39: now also DIP1.145
- net 40: now also DIP1.147
Changed lines of the file:
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@@
 <part name="SUPPLY38" library="SparkFun-PowerSymbols" library_urn="urn:adsk.eagle:library:530" deviceset="VDD" device=""/>
 <part name="C36" library="resistor" library_urn="urn:adsk.eagle:library:348" deviceset="C-EU" device="C0805" package3d_urn="urn:adsk.eagle:package:26137/1"/>
-<part name="J1" library="SparkFun-Connectors" library_urn="urn:adsk.eagle:library:513" deviceset="CONN_02" device="LOCK_LONGPADS" package3d_urn="urn:adsk.eagle:package:38047/1"/>
+<part name="J1" library="SparkFun-Connectors" library_urn="urn:adsk.eagle:library:513" deviceset="CONN_02" device="LOCK_LONGPADS" package3d_urn="urn:adsk.eagle:package:38047/1" value="+20V"/>
 <part name="SUPPLY1" library="SparkFun-PowerSymbols" library_urn="urn:adsk.eagle:library:530" deviceset="VDD" device=""/>
 <part name="GND1" library="supply1" library_urn="urn:adsk.eagle:library:371" deviceset="GND" device=""/>
@@
 <part name="SUPPLY4" library="SparkFun-PowerSymbols" library_urn="urn:adsk.eagle:library:530" deviceset="VDD" device=""/>
 <part name="SUPPLY8" library="supply2" library_urn="urn:adsk.eagle:library:372" deviceset="+5V" device=""/>
-<part name="J2" library="SparkFun-Connectors" library_urn="urn:adsk.eagle:library:513" deviceset="CONN_10" device="&quot;" package3d_urn="urn:adsk.eagle:package:38157/1"/>
+<part name="J2" library="SparkFun-Connectors" library_urn="urn:adsk.eagle:library:513" deviceset="CONN_10" device="&quot;" package3d_urn="urn:adsk.eagle:package:38157/1" value="Data"/>
 </parts>
 <sheets>
@@
 <wire x1="83.82" y1="-12.7" x2="83.82" y2="7.62" width="0.1524" layer="91"/>
 </segment>
+<segment>
+<pinref part="DIP1" gate="G$1" pin="152"/>
+<wire x1="264.16" y1="-40.64" x2="279.4" y2="-40.64" width="0.1524" layer="91"/>
+</segment>
 </net>
 <net name="24" class="0">
@@
 <wire x1="86.36" y1="-15.24" x2="86.36" y2="7.62" width="0.1524" layer="91"/>
 </segment>
+<segment>
+<pinref part="DIP1" gate="G$1" pin="160"/>
+<wire x1="264.16" y1="-38.1" x2="279.4" y2="-38.1" width="0.1524" layer="91"/>
+</segment>
 </net>
 <net name="25" class="0">
@@
 <pinref part="U11" gate="A" pin="IN_A"/>
 <wire x1="109.22" y1="-2.54" x2="109.22" y2="7.62" width="0.1524" layer="91"/>
+</segment>
+<segment>
+<pinref part="DIP1" gate="G$1" pin="150"/>
+<wire x1="264.16" y1="-43.18" x2="279.4" y2="-43.18" width="0.1524" layer="91"/>
 </segment>
 </net>
@@
 <wire x1="20.32" y1="-35.56" x2="20.32" y2="-50.8" width="0.1524" layer="91"/>
 </segment>
+<segment>
+<pinref part="DIP1" gate="G$1" pin="153"/>
+<wire x1="241.3" y1="-38.1" x2="226.06" y2="-38.1" width="0.1524" layer="91"/>
+</segment>
 </net>
 <net name="31" class="0">
@@
 <wire x1="17.78" y1="-38.1" x2="17.78" y2="-50.8" width="0.1524" layer="91"/>
 </segment>
+<segment>
+<pinref part="DIP1" gate="G$1" pin="151"/>
+<wire x1="241.3" y1="-40.64" x2="226.06" y2="-40.64" width="0.1524" layer="91"/>
+</segment>
 </net>
 <net name="32" class="0">
@@
 <wire x1="106.68" y1="-2.54" x2="106.68" y2="7.62" width="0.1524" layer="91"/>
 </segment>
+<segment>
+<pinref part="DIP1" gate="G$1" pin="146"/>
+<wire x1="264.16" y1="-45.72" x2="279.4" y2="-45.72" width="0.1524" layer="91"/>
+</segment>
 </net>
 <net name="35" class="0">
@@
 <wire x1="22.86" y1="-68.58" x2="22.86" y2="-50.8" width="0.1524" layer="91"/>
 </segment>
+<segment>
+<pinref part="DIP1" gate="G$1" pin="145"/>
+<wire x1="241.3" y1="-45.72" x2="226.06" y2="-45.72" width="0.1524" layer="91"/>
+</segment>
 </net>
 <net name="40" class="0">
@@
 <wire x1="25.4" y1="-71.12" x2="25.4" y2="-50.8" width="0.1524" layer="91"/>
 </segment>
-</net>
+<segment>
+<pinref part="DIP1" gate="G$1" pin="147"/>
+<wire x1="241.3" y1="-43.18" x2="226.06" y2="-43.18" width="0.1524" layer="91"/>
+</segment>
+</net>

Commit message: About 80% complete routing
Connections:
- net 32: now also DIP1.139
- net 33: now also DIP1.144
- net 39: now also DIP1.147; no longer DIP1.145
- net 40: now also DIP1.145; no longer DIP1.147
- net 48: now also DIP1.140
- net 49: now also DIP1.138
- net 57: now also DIP1.135
- net 58: now also DIP1.133
- net 66: now also DIP1.129
- net 67: now also DIP1.127
- net 75: now also DIP1.123
- net 76: now also DIP1.120
- net 84: now also DIP1.116
- net 85: now also DIP1.113
Changed lines of the file:
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@@
 <wire x1="81.28" y1="-35.56" x2="81.28" y2="-50.8" width="0.1524" layer="91"/>
+</segment>
+<segment>
+<pinref part="DIP1" gate="G$1" pin="139"/>
+<wire x1="279.4" y1="-50.8" x2="264.16" y2="-50.8" width="0.1524" layer="91"/>
 </segment>
 </net>
@@
 <wire x1="78.74" y1="-38.1" x2="78.74" y2="-50.8" width="0.1524" layer="91"/>
 </segment>
+<segment>
+<pinref part="DIP1" gate="G$1" pin="144"/>
+<wire x1="264.16" y1="-48.26" x2="279.4" y2="-48.26" width="0.1524" layer="91"/>
+</segment>
 </net>
 <net name="34" class="0">
@@
 </segment>
 <segment>
-<pinref part="DIP1" gate="G$1" pin="145"/>
-<wire x1="241.3" y1="-45.72" x2="226.06" y2="-45.72" width="0.1524" layer="91"/>
+<pinref part="DIP1" gate="G$1" pin="147"/>
+<wire x1="241.3" y1="-43.18" x2="226.06" y2="-43.18" width="0.1524" layer="91"/>
 </segment>
 </net>
@@
 </segment>
 <segment>
-<pinref part="DIP1" gate="G$1" pin="147"/>
-<wire x1="241.3" y1="-43.18" x2="226.06" y2="-43.18" width="0.1524" layer="91"/>
+<pinref part="DIP1" gate="G$1" pin="145"/>
+<wire x1="241.3" y1="-45.72" x2="226.06" y2="-45.72" width="0.1524" layer="91"/>
 </segment>
 </net>
@@
 <wire x1="22.86" y1="-91.44" x2="22.86" y2="-106.68" width="0.1524" layer="91"/>
 </segment>
+<segment>
+<pinref part="DIP1" gate="G$1" pin="140"/>
+<wire x1="241.3" y1="-48.26" x2="226.06" y2="-48.26" width="0.1524" layer="91"/>
+</segment>
 </net>
 <net name="49" class="0">
@@
 <wire x1="20.32" y1="-93.98" x2="20.32" y2="-106.68" width="0.1524" layer="91"/>
 </segment>
+<segment>
+<pinref part="DIP1" gate="G$1" pin="138"/>
+<wire x1="241.3" y1="-50.8" x2="226.06" y2="-50.8" width="0.1524" layer="91"/>
+</segment>
 </net>
 <net name="50" class="0">
@@
 <wire x1="22.86" y1="-127" x2="22.86" y2="-106.68" width="0.1524" layer="91"/>
 </segment>
+<segment>
+<pinref part="DIP1" gate="G$1" pin="135"/>
+<wire x1="241.3" y1="-53.34" x2="226.06" y2="-53.34" width="0.1524" layer="91"/>
+</segment>
 </net>
 <net name="58" class="0">
@@
 <wire x1="25.4" y1="-129.54" x2="25.4" y2="-106.68" width="0.1524" layer="91"/>
 </segment>
+<segment>
+<pinref part="DIP1" gate="G$1" pin="133"/>
+<wire x1="241.3" y1="-55.88" x2="226.06" y2="-55.88" width="0.1524" layer="91"/>
+</segment>
 </net>
 <net name="59" class="0">
@@
 <wire x1="20.32" y1="-149.86" x2="20.32" y2="-170.18" width="0.1524" layer="91"/>
 </segment>
+<segment>
+<pinref part="DIP1" gate="G$1" pin="129"/>
+<wire x1="241.3" y1="-58.42" x2="226.06" y2="-58.42" width="0.1524" layer="91"/>
+</segment>
 </net>
 <net name="67" class="0">
@@
 <wire x1="17.78" y1="-152.4" x2="17.78" y2="-170.18" width="0.1524" layer="91"/>
 </segment>
+<segment>
+<pinref part="DIP1" gate="G$1" pin="127"/>
+<wire x1="241.3" y1="-60.96" x2="226.06" y2="-60.96" width="0.1524" layer="91"/>
+</segment>
 </net>
 <net name="68" class="0">
@@
 <wire x1="22.86" y1="-187.96" x2="22.86" y2="-170.18" width="0.1524" layer="91"/>
 </segment>
+<segment>
+<pinref part="DIP1" gate="G$1" pin="123"/>
+<wire x1="241.3" y1="-66.04" x2="226.06" y2="-66.04" width="0.1524" layer="91"/>
+</segment>
 </net>
 <net name="76" class="0">
@@
 <wire x1="25.4" y1="-190.5" x2="25.4" y2="-170.18" width="0.1524" layer="91"/>
 </segment>
+<segment>
+<pinref part="DIP1" gate="G$1" pin="120"/>
+<wire x1="241.3" y1="-68.58" x2="226.06" y2="-68.58" width="0.1524" layer="91"/>
+</segment>
 </net>
 <net name="77" class="0">
@@
 <wire x1="22.86" y1="-210.82" x2="22.86" y2="-233.68" width="0.1524" layer="91"/>
 </segment>
+<segment>
+<pinref part="DIP1" gate="G$1" pin="116"/>
+<wire x1="241.3" y1="-71.12" x2="226.06" y2="-71.12" width="0.1524" layer="91"/>
+</segment>
 </net>
 <net name="85" class="0">
@@
 <wire x1="20.32" y1="-213.36" x2="20.32" y2="-233.68" width="0.1524" layer="91"/>
 </segment>
-</net>
+<segment>
+<pinref part="DIP1" gate="G$1" pin="113"/>
+<wire x1="241.3" y1="-73.66" x2="226.06" y2="-73.66" width="0.1524" layer="91"/>
+</segment>
+</net>

Commit message: Nearly done!
Connections:
- net 41: now also DIP1.122
- net 42: now also DIP1.126
- net 43: now also DIP1.119
- net 50: now also DIP1.108
- net 51: now also DIP1.112
- net 52: now also DIP1.115
- net 59: now also DIP1.100
- net 60: now also DIP1.106
- net 61: now also DIP1.98
- net 68: now also DIP1.90
- net 69: now also DIP1.93
- net 70: now also DIP1.96
- net 77: now also DIP1.97
- net 78: now also DIP1.94
- net 79: now also DIP1.99
- net 86: now also DIP1.109
- net 87: now also DIP1.107
- net 88: now also DIP1.102
Changed lines of the file:
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@@
 <wire x1="86.36" y1="-68.58" x2="86.36" y2="-50.8" width="0.1524" layer="91"/>
+</segment>
+<segment>
+<pinref part="DIP1" gate="G$1" pin="122"/>
+<wire x1="264.16" y1="-68.58" x2="279.4" y2="-68.58" width="0.1524" layer="91"/>
 </segment>
 </net>
@@
 <wire x1="88.9" y1="-71.12" x2="88.9" y2="-50.8" width="0.1524" layer="91"/>
 </segment>
+<segment>
+<pinref part="DIP1" gate="G$1" pin="126"/>
+<wire x1="264.16" y1="-66.04" x2="279.4" y2="-66.04" width="0.1524" layer="91"/>
+</segment>
 </net>
 <net name="43" class="0">
@@
 <wire x1="109.22" y1="-58.42" x2="109.22" y2="-50.8" width="0.1524" layer="91"/>
 </segment>
+<segment>
+<pinref part="DIP1" gate="G$1" pin="119"/>
+<wire x1="264.16" y1="-71.12" x2="279.4" y2="-71.12" width="0.1524" layer="91"/>
+</segment>
 </net>
 <net name="52" class="0">
@@
 <pinref part="U23" gate="A" pin="IN_B"/>
 <wire x1="106.68" y1="-50.8" x2="106.68" y2="-58.42" width="0.1524" layer="91"/>
+</segment>
+<segment>
+<pinref part="DIP1" gate="G$1" pin="115"/>
+<wire x1="264.16" y1="-73.66" x2="279.4" y2="-73.66" width="0.1524" layer="91"/>
 </segment>
 </net>
@@
 <wire x1="81.28" y1="-91.44" x2="81.28" y2="-106.68" width="0.1524" layer="91"/>
 </segment>
+<segment>
+<pinref part="DIP1" gate="G$1" pin="108"/>
+<wire x1="264.16" y1="-78.74" x2="279.4" y2="-78.74" width="0.1524" layer="91"/>
+</segment>
 </net>
 <net name="51" class="0">
@@
 <wire x1="78.74" y1="-93.98" x2="78.74" y2="-106.68" width="0.1524" layer="91"/>
 </segment>
+<segment>
+<pinref part="DIP1" gate="G$1" pin="112"/>
+<wire x1="264.16" y1="-76.2" x2="279.4" y2="-76.2" width="0.1524" layer="91"/>
+</segment>
 </net>
 <net name="53" class="0">
@@
 <wire x1="83.82" y1="-127" x2="83.82" y2="-106.68" width="0.1524" layer="91"/>
 </segment>
+<segment>
+<pinref part="DIP1" gate="G$1" pin="100"/>
+<wire x1="264.16" y1="-83.82" x2="279.4" y2="-83.82" width="0.1524" layer="91"/>
+</segment>
 </net>
 <net name="60" class="0">
@@
 <wire x1="86.36" y1="-129.54" x2="86.36" y2="-106.68" width="0.1524" layer="91"/>
 </segment>
+<segment>
+<pinref part="DIP1" gate="G$1" pin="106"/>
+<wire x1="264.16" y1="-81.28" x2="279.4" y2="-81.28" width="0.1524" layer="91"/>
+</segment>
 </net>
 <net name="61" class="0">
@@
 <wire x1="111.76" y1="-106.68" x2="111.76" y2="-116.84" width="0.1524" layer="91"/>
 </segment>
+<segment>
+<pinref part="DIP1" gate="G$1" pin="98"/>
+<wire x1="264.16" y1="-86.36" x2="279.4" y2="-86.36" width="0.1524" layer="91"/>
+</segment>
 </net>
 <net name="70" class="0">
@@
 <pinref part="U41" gate="A" pin="IN_B"/>
 <wire x1="109.22" y1="-106.68" x2="109.22" y2="-116.84" width="0.1524" layer="91"/>
+</segment>
+<segment>
+<pinref part="DIP1" gate="G$1" pin="96"/>
+<wire x1="264.16" y1="-88.9" x2="279.4" y2="-88.9" width="0.1524" layer="91"/>
 </segment>
 </net>
@@
 <wire x1="81.28" y1="-149.86" x2="81.28" y2="-170.18" width="0.1524" layer="91"/>
 </segment>
+<segment>
+<pinref part="DIP1" gate="G$1" pin="90"/>
+<wire x1="241.3" y1="-91.44" x2="226.06" y2="-91.44" width="0.1524" layer="91"/>
+</segment>
 </net>
 <net name="69" class="0">
@@
 <wire x1="78.74" y1="-152.4" x2="78.74" y2="-170.18" width="0.1524" layer="91"/>
 </segment>
+<segment>
+<pinref part="DIP1" gate="G$1" pin="93"/>
+<wire x1="264.16" y1="-91.44" x2="279.4" y2="-91.44" width="0.1524" layer="91"/>
+</segment>
 </net>
 <net name="71" class="0">
@@
 <wire x1="83.82" y1="-187.96" x2="83.82" y2="-170.18" width="0.1524" layer="91"/>
 </segment>
+<segment>
+<pinref part="DIP1" gate="G$1" pin="97"/>
+<wire x1="241.3" y1="-86.36" x2="226.06" y2="-86.36" width="0.1524" layer="91"/>
+</segment>
 </net>
 <net name="78" class="0">
@@
 <wire x1="86.36" y1="-190.5" x2="86.36" y2="-170.18" width="0.1524" layer="91"/>
 </segment>
+<segment>
+<pinref part="DIP1" gate="G$1" pin="94"/>
+<wire x1="241.3" y1="-88.9" x2="226.06" y2="-88.9" width="0.1524" layer="91"/>
+</segment>
 </net>
 <net name="79" class="0">
@@
 <wire x1="111.76" y1="-180.34" x2="111.76" y2="-170.18" width="0.1524" layer="91"/>
 </segment>
+<segment>
+<pinref part="DIP1" gate="G$1" pin="99"/>
+<wire x1="241.3" y1="-83.82" x2="226.06" y2="-83.82" width="0.1524" layer="91"/>
+</segment>
 </net>
 <net name="88" class="0">
@@
 <pinref part="U59" gate="A" pin="IN_B"/>
 <wire x1="109.22" y1="-180.34" x2="109.22" y2="-170.18" width="0.1524" layer="91"/>
+</segment>
+<segment>
+<pinref part="DIP1" gate="G$1" pin="102"/>
+<wire x1="241.3" y1="-81.28" x2="226.06" y2="-81.28" width="0.1524" layer="91"/>
 </segment>
 </net>
@@
 <wire x1="81.28" y1="-210.82" x2="81.28" y2="-233.68" width="0.1524" layer="91"/>
 </segment>
+<segment>
+<pinref part="DIP1" gate="G$1" pin="109"/>
+<wire x1="241.3" y1="-76.2" x2="226.06" y2="-76.2" width="0.1524" layer="91"/>
+</segment>
 </net>
 <net name="87" class="0">
@@
 <wire x1="78.74" y1="-213.36" x2="78.74" y2="-233.68" width="0.1524" layer="91"/>
 </segment>
-</net>
+<segment>
+<pinref part="DIP1" gate="G$1" pin="107"/>
+<wire x1="241.3" y1="-78.74" x2="226.06" y2="-78.74" width="0.1524" layer="91"/>
+</segment>
+</net>

Commit message: Minor revision to add ground to the data port
Parts:
- removed J2: Data, SparkFun-Connectors:CONN_10"
- added DATA: Data, SparkFun-Connectors:CONN_11
- C10, C11, C12, C13, C19, C20, C21, C22, C23, C24, C25, C26, C27, C28, C29, C3, C30, C31, C32, C34, C35, C36, C37, C38, C39, C4, C40, C41, C42, C43, C44, C45, C5, C55, C56, C57, C58, C59, C60, C61, C62, C63, C7, C9: value (none) -> 100nF
- renumbered J1 to 20V-PWR, U$1 to 5V-REG
Connections:
- net 68: now also DIP1.109; no longer DIP1.90
- net 77: now also DIP1.102; no longer DIP1.97
- net 78: now also DIP1.107; no longer DIP1.94
- net 86: now also DIP1.94; no longer DIP1.109
- net 87: now also DIP1.90; no longer DIP1.107
- net 88: now also DIP1.97; no longer DIP1.102
- net GND: now also DATA.11
- net N$1: now also DATA.1; no longer J2.1
- net N$13: now also DATA.5; no longer J2.5
- net N$14: now also DATA.6; no longer J2.6
- net N$17: now also DATA.7; no longer J2.7
- net N$18: now also DATA.8; no longer J2.8
- net N$2: now also DATA.2; no longer J2.2
- net N$29: now also DATA.9; no longer J2.9
- net N$3: now also DATA.3; no longer J2.3
- net N$30: now also DATA.10; no longer J2.10
- net N$4: now also DATA.4; no longer J2.4
