File: eagle/ProjectX/Driver_Board_Niall.brd (EAGLE design)
At the start: 160 x 100 mm, 13 parts, among them IC1 LM317MBSTT3

Commit message: Work in progress driver board
Parts:
- added R6: 100K, resistor:M0805
- added U1, U2: ADA4091-2ARZ-RL, SnapEDA-Library:ADA4091-2ARZ-RL_SOIC127P600X175-8N
- added VAR-RESISTOR: MCP4011T-503E/SN, SnapEDA-Library:SOIC127P600X175-8N
Connections:
- removed net VO: C2.+, D1.A, D2.C, IC1.4, R1.2, R3.2
- new net 12VOLT: C2.+, D1.A, D2.C, IC1.4, R1.2, R3.2, U1.8
- new net N$4: U1.1, U1.2
- new net V+: U2.8
- new net V-: U2.4
- new net VDD: VAR-RESISTOR.1
- net GND: now also U1.4, VAR-RESISTOR.3
- net N$2: now also U1.3, VAR-RESISTOR.4
Changed lines of the file:
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@@
 </autorouter>
 <elements>
-<element name="C1" library="rcl" library_urn="urn:adsk.eagle:library:334" package="C075-052X106" package3d_urn="urn:adsk.eagle:package:23650/1" value="0.1uF" x="-19.05" y="31.75"/>
-<element name="C2" library="resistor" library_urn="urn:adsk.eagle:library:348" package="085CS_1AR" package3d_urn="urn:adsk.eagle:package:25875/1" value="1uF" x="-19.05" y="24.13"/>
-<element name="C3" library="resistor" library_urn="urn:adsk.eagle:library:348" package="085CS_1AR" package3d_urn="urn:adsk.eagle:package:25875/1" value="10uF" x="-30.48" y="24.13"/>
+<element name="C1" library="rcl" library_urn="urn:adsk.eagle:library:334" package="C075-052X106" package3d_urn="urn:adsk.eagle:package:23650/1" value="0.1uF" x="-19.05" y="31.75">
+<attribute name="SPICEPREFIX" value="C" x="-19.05" y="31.75" size="1.778" layer="27" display="off"/>
+</element>
+<element name="C2" library="resistor" library_urn="urn:adsk.eagle:library:348" package="085CS_1AR" package3d_urn="urn:adsk.eagle:package:23396/1" value="1uF" x="-19.05" y="24.13"/>
+<element name="C3" library="resistor" library_urn="urn:adsk.eagle:library:348" package="085CS_1AR" package3d_urn="urn:adsk.eagle:package:23396/1" value="10uF" x="-30.48" y="24.13"/>
 <element name="D1" library="diode" package="DO41-10" package3d_urn="urn:adsk.eagle:package:43336/1" value="1N4002" x="-30.48" y="33.02"/>
 <element name="D2" library="diode" package="DO41-10" package3d_urn="urn:adsk.eagle:package:43336/1" value="1N4002" x="-43.18" y="33.02"/>
@@
 <attribute name="PARTNUMBER" value="LM317M" x="-46.99" y="24.13" size="1.778" layer="27" display="off"/>
 </element>
-<element name="R1" library="resistor" library_urn="urn:adsk.eagle:library:348" package="M0805" package3d_urn="urn:adsk.eagle:package:26079/1" value="240Ω" x="-53.34" y="31.75"/>
-<element name="R2" library="resistor" library_urn="urn:adsk.eagle:library:348" package="M0805" package3d_urn="urn:adsk.eagle:package:26079/1" value="2.1K" x="-16.51" y="40.64"/>
-<element name="R3" library="resistor" library_urn="urn:adsk.eagle:library:348" package="M0805" package3d_urn="urn:adsk.eagle:package:26079/1" value="10K" x="-21.59" y="40.64"/>
-<element name="R4" library="resistor" library_urn="urn:adsk.eagle:library:348" package="M0805" package3d_urn="urn:adsk.eagle:package:26079/1" value="9K" x="-26.67" y="40.64"/>
-<element name="R5" library="resistor" library_urn="urn:adsk.eagle:library:348" package="M0805" package3d_urn="urn:adsk.eagle:package:26079/1" value="1K" x="-31.75" y="40.64"/>
+<element name="R1" library="resistor" library_urn="urn:adsk.eagle:library:348" package="M0805" package3d_urn="urn:adsk.eagle:package:23556/1" value="240Ω" x="-53.34" y="31.75"/>
+<element name="R2" library="resistor" library_urn="urn:adsk.eagle:library:348" package="M0805" package3d_urn="urn:adsk.eagle:package:23556/1" value="2.1K" x="-16.51" y="40.64"/>
+<element name="R3" library="resistor" library_urn="urn:adsk.eagle:library:348" package="M0805" package3d_urn="urn:adsk.eagle:package:23556/1" value="10K" x="-21.59" y="40.64"/>
+<element name="R4" library="resistor" library_urn="urn:adsk.eagle:library:348" package="M0805" package3d_urn="urn:adsk.eagle:package:23556/1" value="9K" x="-26.67" y="40.64"/>
+<element name="R5" library="resistor" library_urn="urn:adsk.eagle:library:348" package="M0805" package3d_urn="urn:adsk.eagle:package:23556/1" value="1K" x="-31.75" y="40.64"/>
 <element name="U$2" library="Teensy356" package="TEENSY_3.5/3.6" value="TEENSY_3.5/3.6" x="-45.72" y="10.16"/>
 <element name="ZENER1" library="diode" library_urn="urn:adsk.eagle:library:210" package="C1702-15" package3d_urn="urn:adsk.eagle:package:43351/1" value="3.3V" x="-44.45" y="39.37"/>
+<element name="U1" library="SnapEDA-Library" package="ADA4091-2ARZ-RL_SOIC127P600X175-8N" value="ADA4091-2ARZ-RL" x="-85.09" y="7.62">
+<attribute name="MPN" value="ADA4091-2ARZ-RL" x="-85.09" y="7.62" size="1.778" layer="27" display="off"/>
+<attribute name="OC_FARNELL" value="1702289" x="-85.09" y="7.62" size="1.778" layer="27" display="off"/>
+<attribute name="OC_NEWARK" value="34P2964" x="-85.09" y="7.62" size="1.778" layer="27" display="off"/>
+<attribute name="PACKAGE" value="SOIC-8" x="-85.09" y="7.62" size="1.778" layer="27" display="off"/>
+<attribute name="SUPPLIER" value="Analog Devices" x="-85.09" y="7.62" size="1.778" layer="27" display="off"/>
+</element>
+<element name="U2" library="SnapEDA-Library" package="ADA4091-2ARZ-RL_SOIC127P600X175-8N" value="ADA4091-2ARZ-RL" x="-99.06" y="7.62">
+<attribute name="MPN" value="ADA4091-2ARZ-RL" x="-99.06" y="7.62" size="1.778" layer="27" display="off"/>
+<attribute name="OC_FARNELL" value="1702289" x="-99.06" y="7.62" size="1.778" layer="27" display="off"/>
+<attribute name="OC_NEWARK" value="34P2964" x="-99.06" y="7.62" size="1.778" layer="27" display="off"/>
+<attribute name="PACKAGE" value="SOIC-8" x="-99.06" y="7.62" size="1.778" layer="27" display="off"/>
+<attribute name="SUPPLIER" value="Analog Devices" x="-99.06" y="7.62" size="1.778" layer="27" display="off"/>
+</element>
+<element name="R6" library="resistor" library_urn="urn:adsk.eagle:library:348" package="M0805" package3d_urn="urn:adsk.eagle:package:23556/1" value="100K" x="-100.33" y="-3.81"/>
+<element name="VAR-RESISTOR" library="SnapEDA-Library" package="SOIC127P600X175-8N" value="MCP4011T-503E/SN" x="-96.52" y="-13.97">
+<attribute name="MPN" value="MCP4011T-503E/SN" x="-96.52" y="-13.97" size="1.778" layer="27" display="off"/>
+<attribute name="OC_FARNELL" value="1332103" x="-96.52" y="-13.97" size="1.778" layer="27" display="off"/>
+<attribute name="OC_NEWARK" value="34M7452" x="-96.52" y="-13.97" size="1.778" layer="27" display="off"/>
+<attribute name="PACKAGE" value="SOIC-8" x="-96.52" y="-13.97" size="1.778" layer="27" display="off"/>
+<attribute name="SUPPLIER" value="MICROCHIP" x="-96.52" y="-13.97" size="1.778" layer="27" display="off"/>
+</element>
 </elements>
 <signals>
@@
 <contactref element="ZENER1" pad="A"/>
 <contactref element="R5" pad="1"/>
-<wire x1="-15.24" y1="31.75" x2="-17.46" y2="40.64" width="0" layer="19" extent="1-1"/>
-<wire x1="-22.3" y1="24.13" x2="-15.24" y2="31.75" width="0" layer="19" extent="1-1"/>
-<wire x1="-33.73" y1="24.13" x2="-22.3" y2="24.13" width="0" layer="19" extent="1-1"/>
+<contactref element="U1" pad="4"/>
+<contactref element="VAR-RESISTOR" pad="3"/>
+<wire x1="-87.5538" y1="5.715" x2="-98.8822" y2="-14.605" width="0" layer="19" extent="1-1"/>
+<wire x1="-33.73" y1="24.13" x2="-87.5538" y2="5.715" width="0" layer="19" extent="1-1"/>
+<wire x1="-22.3" y1="24.13" x2="-33.73" y2="24.13" width="0" layer="19" extent="1-1"/>
+<wire x1="-15.24" y1="31.75" x2="-22.3" y2="24.13" width="0" layer="19" extent="1-1"/>
+<wire x1="-17.46" y1="40.64" x2="-15.24" y2="31.75" width="0" layer="19" extent="1-1"/>
 <wire x1="-32.7" y1="40.64" x2="-17.46" y2="40.64" width="0" layer="19" extent="1-1"/>
 <wire x1="-36.83" y1="39.37" x2="-32.7" y2="40.64" width="0" layer="19" extent="1-1"/>
@@
 <wire x1="-15.56" y1="40.64" x2="-27.23" y2="24.13" width="0" layer="19" extent="1-1"/>
 </signal>
-<signal name="VO">
+<signal name="12VOLT">
 <contactref element="D2" pad="C"/>
 <contactref element="IC1" pad="4"/>
@@
 <contactref element="C2" pad="+"/>
 <contactref element="R3" pad="2"/>
-<wire x1="-48.26" y1="33.02" x2="-46.99" y2="27.28" width="0" layer="19" extent="1-1"/>
-<wire x1="-52.39" y1="31.75" x2="-48.26" y2="33.02" width="0" layer="19" extent="1-1"/>
+<contactref element="U1" pad="8"/>
+<wire x1="-52.39" y1="31.75" x2="-82.6262" y2="9.525" width="0" layer="19" extent="1-1"/>
+<wire x1="-48.26" y1="33.02" x2="-52.39" y2="31.75" width="0" layer="19" extent="1-1"/>
+<wire x1="-46.99" y1="27.28" x2="-48.26" y2="33.02" width="0" layer="19" extent="1-1"/>
 <wire x1="-25.4" y1="33.02" x2="-46.99" y2="27.28" width="0" layer="19" extent="1-1"/>
 <wire x1="-20.64" y1="40.64" x2="-25.4" y2="33.02" width="0" layer="19" extent="1-1"/>
@@
 <contactref element="R4" pad="1"/>
 <contactref element="R5" pad="2"/>
-<wire x1="-30.8" y1="40.64" x2="-27.62" y2="40.64" width="0" layer="19" extent="1-1"/>
+<contactref element="U1" pad="3"/>
+<contactref element="VAR-RESISTOR" pad="4"/>
+<wire x1="-87.5538" y1="6.985" x2="-98.8822" y2="-15.875" width="0" layer="19" extent="1-1"/>
+<wire x1="-30.8" y1="40.64" x2="-87.5538" y2="6.985" width="0" layer="19" extent="1-1"/>
+<wire x1="-27.62" y1="40.64" x2="-30.8" y2="40.64" width="0" layer="19" extent="1-1"/>
+</signal>
+<signal name="N$4">
+<contactref element="U1" pad="1"/>
+<contactref element="U1" pad="2"/>
+<wire x1="-87.5538" y1="8.255" x2="-87.5538" y2="9.525" width="0" layer="19" extent="1-1"/>
+</signal>
+<signal name="V+">
+<contactref element="U2" pad="8"/>
+</signal>
+<signal name="V-">
+<contactref element="U2" pad="4"/>
+</signal>
+<signal name="VDD">
+<contactref element="VAR-RESISTOR" pad="1"/>
 </signal>
 </signals>

Commit message: Eagle work- niall
Parts:
- removed VAR-RESISTOR: MCP4011T-503E/SN, SnapEDA-Library:SOIC127P600X175-8N
- added C35: 100nF, resistor:C0805
- added Q1: 2N7000G, SnapEDA-Library:TO92-INLINE
- added R10: 1.2k, resistor:M0805
- added R11: 330, resistor:M0805
- added R12: 1M, resistor:M0805
- added R13: 100, resistor:M0805
- added R14: 10k, resistor:M0805
- added R7: 100K, resistor:M0805
- added R8: 33K, resistor:M0805
- added R9: 1K, resistor:M0805
- added T3: MA40S4S, Parts:MA40
- added U35: TC4427AEOA, Parts:SOIC127P600X175-8N
- R4: value 9K -> 10K
Connections:
- removed net 12VOLT: C2.+, D1.A, D2.C, IC1.4, R1.2, R3.2, U1.8
- removed net V+: U2.8
- removed net V-: U2.4
- new net N$10: R12.2, R13.2, U$2.35/A16
- new net N$11: Q1.2, R13.1
- new net N$12: R14.2, T3.-
- new net N$13: U$2.36/A17, U35.4
- new net N$5: R6.1, R7.2, U2.3
- new net N$6: Q1.3, R6.2
- new net N$7: R10.2, R8.1, U2.1
- new net N$72: R14.1, T3.+, U35.5
- new net N$8: R8.2, R9.1, U2.2
- new net N$9: R10.1, R11.2, U$2.23/A9
- net GND: now also C35.1, Q1.1, R11.1, R12.1, R9.2, U2.4, U35.3; no longer VAR-RESISTOR.3
- net N$2: no longer VAR-RESISTOR.4
- net N$4: now also R7.1
- net VDD: now also C2.+, D1.A, D2.C, IC1.4, R1.2, R3.2, U1.8, U2.8; no longer VAR-RESISTOR.1
- net VIN: now also C35.2, U35.6

Commit message: Niall bord edits
Parts:
- added C4, C5: 100nF, resistor:C0805
- added R15, R16: (no value), pot:CA6V
- moved R14 160.0 mm to (10.0, 12.9), turned to 270 degrees
- moved U2 154.7 mm to (55.6, 11.2)
- moved R8 153.9 mm to (47.3, 14.3)
- moved R7 152.2 mm to (21.3, 68.7)
- moved R6 149.8 mm to (32.3, 65.7)
- moved C35 148.9 mm to (-0.94, 14.4)
- moved U35 141.0 mm to (6.49, 17.5)
- moved U1 136.4 mm to (34.6, 73.2)
- moved T3 132.9 mm to (6.40, 6.30), turned to 180 degrees
- moved IC1 131.7 mm to (77.7, 66.7)
- moved C1 130.4 mm to (101.6, 81.3)
- moved D2 130.4 mm to (77.5, 82.5)
- moved R1 130.4 mm to (67.3, 81.3)
- moved R2 130.4 mm to (104.1, 90.2)
- moved R3 130.4 mm to (99.1, 90.2)
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Connections:
- removed net N$8: R8.2, R9.1, U2.2
- new net N$14: R16.A, R8.2, R9.1, U2.2
- net GND: now also C4.2, C5.2
- net N$2: now also R15.S
- net N$3: now also R15.A
- net N$7: now also R16.S
- net VDD: now also C4.1, C5.1
Other:
- board size 160 x 100 mm -> 100 x 100 mm

Commit message: Niall Board layout first attempt
Parts:
- removed ZENER1: 3.3V, diode:C1702-15
- added J1: 694102303002, SnapEDA-Library:69410X303002
- added ZENER: 3.3V, diode:DO34Z7
- moved R13 106.7 mm to (56.0, 95.0)
- moved C5 105.2 mm to (51.0, 88.0)
- moved C4 104.9 mm to (62.0, 88.0)
- moved R12 99.6 mm to (51.0, 95.0), turned to 0 degrees
- moved Q1 97.4 mm to (57.0, 91.0), turned to 180 degrees
- moved C1 93.7 mm to (9.28, 65.4), turned to 270 degrees
- moved R16 90.0 mm to (49.5, 73.2)
- moved T3 88.1 mm to (5.70, 94.4), turned to 270 degrees
- moved R11 83.7 mm to (43.0, 85.0), turned to 270 degrees
- moved R14 81.2 mm to (13.0, 94.1), turned to 90 degrees
- moved R9 81.0 mm to (47.0, 84.0), turned to 90 degrees
- moved C2 80.3 mm to (16.3, 65.6), turned to 90 degrees
- moved D1 80.3 mm to (9.17, 73.5)
- moved R2 79.1 mm to (26.0, 78.0), turned to 90 degrees
- moved R10 78.2 mm to (43.0, 80.0), turned to 270 degrees
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Connections:
- net VDD renamed $VDD
- removed net GND: C1.2, C2.-, C3.-, C35.1, C4.2, C5.2, Q1.1, R11.1, R12.1, R2.1, R5.1, R9.2, U1.4, U2.4, U35.3, ZENER1.A
- removed net N$6: Q1.3, R6.2
- removed net VIN: C1.1, C35.2, D1.C, IC1.3, U35.6
- new net $GND: C1.2, C2.-, C3.-, C35.1, C4.2, C5.2, J1.2, Q1.1, R11.1, R12.1, R2.1, R5.1, R9.2, U$2.GND, U1.4, U2.4, U35.3, ZENER.A
- new net $VIN: C1.1, C35.2, D1.C, IC1.3, J1.1, U35.6
- net N$12: now also Q1.3, R6.2
- net N$3: now also ZENER.C; no longer ZENER1.C
Routing:
- net N$13: track 0.00 -> 61.8 mm, vias 0 -> 1
- net N$12: track 0.00 -> 58.9 mm
- net N$9: track 0.00 -> 51.7 mm
- net N$10: track 0.00 -> 49.5 mm, vias 0 -> 1
- net $VDD: track 0.00 -> 45.7 mm, vias 0 -> 4
- net $VIN: track 0.00 -> 37.8 mm
- net N$7: track 0.00 -> 35.6 mm
- net $GND: track 0.00 -> 32.4 mm, vias 0 -> 15
- net N$1: track 0.00 -> 29.1 mm
- net N$2: track 0.00 -> 21.9 mm
- net N$3: track 0.00 -> 20.9 mm
- net N$14: track 0.00 -> 13.7 mm
- net N$5: track 0.00 -> 12.0 mm
- net N$72: track 0.00 -> 10.3 mm
- net N$4: track 0.00 -> 7.05 mm
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- added copper zone on layer 2, net $GND
- added copper zone on layer 3, net $VDD

Commit message: Niall Board layout first attempt
Parts:
- moved C3 10.3 mm to (25.0, 83.0), turned to 0 degrees
- moved C4 6.00 mm to (56.0, 88.0)
- moved C5 6.00 mm to (45.0, 88.0)
- moved Q1 6.00 mm to (51.0, 91.0)
- moved R10 6.00 mm to (37.0, 80.0)
- moved R11 6.00 mm to (37.0, 85.0)
- moved R12 6.00 mm to (45.0, 95.0)
- moved R13 6.00 mm to (50.0, 95.0)
- moved R15 6.00 mm to (55.0, 73.0)
- moved R16 6.00 mm to (43.5, 73.2)
- moved R3 6.00 mm to (61.0, 80.0)
- moved R4 6.00 mm to (61.0, 73.0)
- moved R5 6.00 mm to (57.0, 67.0)
- moved R6 6.00 mm to (50.0, 83.0)
- moved R7 6.00 mm to (51.0, 79.0)
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Routing:
- net N$1: track 29.1 -> 43.4 mm
- net N$7: track 35.6 -> 23.8 mm
- net N$12: track 58.9 -> 52.9 mm
- net N$9: track 51.7 -> 46.3 mm
- net $VDD: track 45.7 -> 43.0 mm
- net N$10: track 49.5 -> 52.0 mm
- net N$4: track 7.05 -> 5.35 mm

Commit message: Niall Board layout first attempt
Routing:
- net $VIN: track 37.8 -> 51.2 mm
- net N$72: track 10.3 -> 13.9 mm
- net $VDD: track 43.0 -> 45.7 mm
- net N$4: track 5.35 -> 7.00 mm
- net N$14: track 13.7 -> 14.2 mm
Changed lines of the file:
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@@
 <via x="41" y="87" extent="1-16" drill="0.35"/>
 <wire x1="45.95" y1="88" x2="48" y2="88" width="1.016" layer="1"/>
-<wire x1="56.95" y1="88" x2="59" y2="88" width="1.016" layer="1"/>
-<via x="59" y="88" extent="1-16" drill="0.35"/>
 <wire x1="64" y1="70.19" x2="64" y2="68" width="1.016" layer="1"/>
 <via x="64" y="68" extent="1-16" drill="0.35"/>
@@
 <via x="47" y="79" extent="1-16" drill="0.35"/>
 <via x="48" y="88" extent="1-16" drill="0.35"/>
+<wire x1="56.95" y1="88" x2="59" y2="88" width="1.016" layer="1"/>
+<via x="59" y="88" extent="1-16" drill="0.35"/>
 </signal>
 <signal name="N$1">
@@
 <contactref element="D1" pad="C"/>
 <wire x1="9" y1="73.55" x2="4.09" y2="73.55" width="1.016" layer="1"/>
-<wire x1="12" y1="80" x2="12" y2="73.55" width="1.016" layer="1"/>
-<wire x1="11.9" y1="80" x2="15" y2="80" width="1.016" layer="1"/>
+<wire x1="12" y1="80" x2="12" y2="76" width="1.016" layer="1"/>
+<wire x1="12" y1="76" x2="12" y2="73.55" width="1.016" layer="1"/>
 <wire x1="11.9" y1="80" x2="11.9" y2="82.9" width="1.016" layer="1"/>
 <wire x1="11.9" y1="82.9" x2="16" y2="87" width="1.016" layer="1"/>
@@
 <wire x1="16.365" y1="91.6378" x2="16.365" y2="87.365" width="1.016" layer="1"/>
 <wire x1="16.365" y1="87.365" x2="16" y2="87" width="1.016" layer="1"/>
-<wire x1="15" y1="80" x2="15.04" y2="80.49" width="0" layer="19" extent="1-1"/>
+<wire x1="15.04" y1="80.49" x2="15.04" y2="79.04" width="1.016" layer="1"/>
+<wire x1="15.04" y1="79.04" x2="15" y2="79" width="1.016" layer="1"/>
+<wire x1="15.04" y1="80.49" x2="15.04" y2="86.04" width="1.016" layer="1"/>
+<wire x1="15.04" y1="86.04" x2="16.365" y2="87.365" width="1.016" layer="1"/>
+<wire x1="15" y1="79" x2="12" y2="76" width="1.016" layer="1"/>
+<wire x1="15.04" y1="80.49" x2="12.39" y2="80.49" width="1.016" layer="1"/>
+<wire x1="12.39" y1="80.49" x2="11.9" y2="80" width="1.016" layer="1"/>
 </signal>
 <signal name="N$2">
@@
 <contactref element="R7" pad="1"/>
 <wire x1="54" y1="79" x2="51.95" y2="79" width="1.016" layer="1"/>
-<wire x1="60.095" y1="80.5362" x2="61.365" y2="80.5362" width="1.016" layer="1"/>
-<wire x1="60.095" y1="80.5362" x2="60" y2="80.5362" width="1.016" layer="1"/>
-<wire x1="61.365" y1="80.5362" x2="60" y2="79.1712" width="1.016" layer="1" curve="90"/>
+<wire x1="54.095" y1="80.5362" x2="54" y2="80.4412" width="1.016" layer="1"/>
+<wire x1="54" y1="80.4412" x2="54" y2="79" width="1.016" layer="1"/>
+<wire x1="55.365" y1="80.5362" x2="54.095" y2="80.5362" width="1.016" layer="1"/>
+<wire x1="55.365" y1="80.5362" x2="54" y2="79.1712" width="1.016" layer="1"/>
+<wire x1="54" y1="79.1712" x2="54" y2="79" width="1.016" layer="1"/>
 </signal>
 <signal name="N$5">
@@
 <contactref element="U35" pad="5"/>
 <contactref element="R14" pad="1"/>
-<wire x1="12.97" y1="93.11" x2="14.08" y2="92" width="1.016" layer="1"/>
-<wire x1="14.08" y1="92" x2="15" y2="92" width="1.016" layer="1"/>
 <wire x1="5.7" y1="91.9" x2="11.76" y2="91.9" width="1.016" layer="1"/>
-<wire x1="11.76" y1="91.9" x2="12.97" y2="93.11" width="1.016" layer="1"/>
-<wire x1="15" y1="92" x2="15.095" y2="91.6378" width="0" layer="19" extent="1-1"/>
+<wire x1="11.76" y1="91.9" x2="11.93" y2="92.07" width="1.016" layer="1"/>
+<wire x1="11.93" y1="92.07" x2="12.97" y2="93.11" width="1.016" layer="1"/>
+<wire x1="15.095" y1="91.6378" x2="14.6628" y2="92.07" width="1.016" layer="1"/>
+<wire x1="14.6628" y1="92.07" x2="11.93" y2="92.07" width="1.016" layer="1"/>
+<wire x1="15.095" y1="91.6378" x2="13.6228" y2="93.11" width="1.016" layer="1"/>
+<wire x1="13.6228" y1="93.11" x2="12.97" y2="93.11" width="1.016" layer="1"/>
 </signal>
 <signal name="N$12">
@@
 <wire x1="44.365" y1="80.5362" x2="44.365" y2="77.325" width="1.016" layer="1"/>
 <wire x1="44.365" y1="77.325" x2="45.99" y2="75.7" width="1.016" layer="1" curve="90"/>
-<wire x1="41" y1="83.05" x2="41.8512" y2="83.05" width="1.016" layer="1"/>
-<wire x1="41.8512" y1="83.05" x2="44.365" y2="80.5362" width="1.016" layer="1" curve="-90"/>
+<wire x1="41" y1="83.05" x2="42.8512" y2="83.05" width="1.016" layer="1"/>
+<wire x1="42.8512" y1="83.05" x2="44.365" y2="81.5362" width="1.016" layer="1" curve="-90"/>
+<wire x1="44.365" y1="81.5362" x2="44.365" y2="80.5362" width="1.016" layer="1"/>
 </signal>
 <signal name="$VDD">
@@
 <wire x1="23" y1="76.16" x2="20.39" y2="73.55" width="1.016" layer="1"/>
 <via x="17" y="72" extent="1-16" drill="0.35"/>
-<wire x1="54.095" y1="85.4638" x2="54.095" y2="87.045" width="1.016" layer="1"/>
-<wire x1="61.05" y1="88" x2="59" y2="88" width="1.016" layer="1"/>
-<wire x1="59" y1="88" x2="59.14" y2="88" width="1.016" layer="1"/>
+<wire x1="54.095" y1="87.045" x2="54.095" y2="85.4638" width="1.016" layer="1"/>
 <via x="53" y="88" extent="1-16" drill="0.35"/>
 <wire x1="61" y1="80.95" x2="61" y2="83" width="1.016" layer="1"/>
@@
 <wire x1="19" y1="73" x2="18" y2="72" width="1.016" layer="1" curve="-90"/>
 <wire x1="18" y1="72" x2="16.05" y2="72.9" width="1.016" layer="1" curve="-49.550281"/>
+<wire x1="55.05" y1="88" x2="54.095" y2="87.045" width="1.016" layer="1"/>
+<wire x1="53" y1="88" x2="53.955" y2="87.045" width="1.016" layer="1"/>
+<wire x1="53.955" y1="87.045" x2="54.095" y2="87.045" width="1.016" layer="1"/>
+<wire x1="53" y1="88" x2="55.05" y2="88" width="1.016" layer="1"/>
 </signal>
 <signal name="N$3">

Commit message: Niall Board layout first attempt
Parts:
- moved C3 4.00 mm to (25.0, 79.0)
- moved D1 4.00 mm to (9.17, 69.5)
- moved D2 4.00 mm to (25.5, 69.5)
- moved IC1 4.00 mm to (17.3, 73.3)
- moved J1 4.00 mm to (1.00, 76.0)
- moved R1 4.00 mm to (23.0, 74.0)
- moved R2 4.00 mm to (26.0, 74.0)
- moved C1 3.94 mm to (5.40, 64.7), turned to 180 degrees
- moved C4 2.83 mm to (54.0, 86.0)
- moved C5 2.83 mm to (43.0, 86.0)
- moved Q1 2.83 mm to (49.0, 89.0)
- moved R10 2.83 mm to (35.0, 78.0)
- moved R11 2.83 mm to (35.0, 83.0)
- moved R12 2.83 mm to (43.0, 93.0)
- moved R13 2.83 mm to (48.0, 93.0)
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Routing:
- net $VDD: track 45.7 -> 70.3 mm
- net $VIN: track 51.2 -> 59.6 mm
- net N$13: track 61.9 -> 65.6 mm
- net N$4: track 7.00 -> 9.78 mm
- net N$12: track 52.9 -> 51.7 mm
- net N$10: track 52.0 -> 50.8 mm
- net $GND: track 32.0 -> 31.5 mm
