File: eagle/ProjectX/Driver_Board_Niall.brd (EAGLE design)
At the start: 100 x 100 mm, 33 parts, among them IC1 LM317MBSTT3, J1 694102303002, Q1 2N7000G, T3 MA40S4S, U1 ADA4091-2ARZ-RL, U2 ADA4091-2ARZ-RL, U35 TC4427AEOA

Commit message: niall's crap board
Parts:
- moved Q1 37.7 mm to (12.0, 96.0), turned to 270 degrees
- moved R14 4.12 mm to (8.97, 93.1)
- moved U35 1.00 mm to (18.0, 94.0)
- moved T3 0.60 mm to (6.30, 94.4), flipped to the bottom
Routing:
- net N$12: track 51.7 -> 14.5 mm
- net $GND: track 31.5 -> 36.8 mm
- net N$72: track 13.9 -> 10.3 mm
- net N$11: track 4.00 -> 1.76 mm
Changed lines of the file:
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@@
 <setting verticaltext="up"/>
 </settings>
-<grid distance="1" unitdist="mm" unit="mm" style="lines" multiple="1" display="no" altdistance="5" altunitdist="mil" altunit="mil"/>
+<grid distance="0.5" unitdist="mm" unit="mm" style="lines" multiple="1" display="yes" altdistance="5" altunitdist="mil" altunit="mil"/>
 <layers>
 <layer number="1" name="Top" color="4" fill="1" visible="yes" active="yes"/>
@@
 <element name="R10" library="resistor" library_urn="urn:adsk.eagle:library:348" package="M0805" package3d_urn="urn:adsk.eagle:package:23556/1" value="1.2k" x="35" y="78" rot="R270"/>
 <element name="R11" library="resistor" library_urn="urn:adsk.eagle:library:348" package="M0805" package3d_urn="urn:adsk.eagle:package:23556/1" value="330" x="35" y="83" rot="R270"/>
-<element name="Q1" library="SnapEDA-Library" package="TO92-INLINE" value="2N7000G" x="49" y="89" rot="R180"/>
+<element name="Q1" library="SnapEDA-Library" package="TO92-INLINE" value="2N7000G" x="12" y="96" rot="R270"/>
 <element name="R12" library="resistor" library_urn="urn:adsk.eagle:library:348" package="M0805" package3d_urn="urn:adsk.eagle:package:23556/1" value="1M" x="43" y="93"/>
 <element name="R13" library="resistor" library_urn="urn:adsk.eagle:library:348" package="M0805" package3d_urn="urn:adsk.eagle:package:23556/1" value="100" x="48" y="93" rot="R180"/>
-<element name="T3" library="Parts" package="MA40" value="MA40S4S" x="5.7" y="94.4" rot="R270"/>
-<element name="U35" library="Parts" package="SOIC127P600X175-8N" value="TC4427AEOA" x="17" y="94" rot="R270">
-<attribute name="MPN" value="TC4427AEOA" x="14.46" y="113.05" size="1.778" layer="27" rot="R270" display="off"/>
-<attribute name="OC_FARNELL" value="1292285" x="14.46" y="113.05" size="1.778" layer="27" rot="R270" display="off"/>
-<attribute name="OC_NEWARK" value="96K4020" x="14.46" y="113.05" size="1.778" layer="27" rot="R270" display="off"/>
-<attribute name="PACKAGE" value="SOIC-8" x="14.46" y="113.05" size="1.778" layer="27" rot="R270" display="off"/>
-<attribute name="SUPPLIER" value="Microchip" x="14.46" y="113.05" size="1.778" layer="27" rot="R270" display="off"/>
+<element name="T3" library="Parts" package="MA40" value="MA40S4S" x="6.3" y="94.4" rot="MR270"/>
+<element name="U35" library="Parts" package="SOIC127P600X175-8N" value="TC4427AEOA" x="18" y="94" rot="R270">
+<attribute name="MPN" value="TC4427AEOA" x="15.46" y="113.05" size="1.778" layer="27" rot="R270" display="off"/>
+<attribute name="OC_FARNELL" value="1292285" x="15.46" y="113.05" size="1.778" layer="27" rot="R270" display="off"/>
+<attribute name="OC_NEWARK" value="96K4020" x="15.46" y="113.05" size="1.778" layer="27" rot="R270" display="off"/>
+<attribute name="PACKAGE" value="SOIC-8" x="15.46" y="113.05" size="1.778" layer="27" rot="R270" display="off"/>
+<attribute name="SUPPLIER" value="Microchip" x="15.46" y="113.05" size="1.778" layer="27" rot="R270" display="off"/>
 </element>
 <element name="C35" library="resistor" library_urn="urn:adsk.eagle:library:348" package="C0805" package3d_urn="urn:adsk.eagle:package:23617/2" value="100nF" x="15" y="89"/>
-<element name="R14" library="resistor" library_urn="urn:adsk.eagle:library:348" package="M0805" package3d_urn="urn:adsk.eagle:package:23556/1" value="10k" x="12.97" y="94.06" rot="R90"/>
+<element name="R14" library="resistor" library_urn="urn:adsk.eagle:library:348" package="M0805" package3d_urn="urn:adsk.eagle:package:23556/1" value="10k" x="8.97" y="93.06" rot="R90"/>
 <element name="R15" library="pot" library_urn="urn:adsk.eagle:library:331" package="CA6V" package3d_urn="urn:adsk.eagle:package:22691/1" value="" x="53" y="71" rot="R180"/>
 <element name="R16" library="pot" library_urn="urn:adsk.eagle:library:331" package="CA6V" package3d_urn="urn:adsk.eagle:package:22691/1" value="" x="41.45" y="71.16" rot="R180"/>
@@
 <contactref element="J1" pad="2"/>
 <contactref element="U$2" pad="GND"/>
-<via x="16" y="98" extent="1-16" drill="0.35"/>
-<wire x1="16.365" y1="96.3622" x2="16.365" y2="98" width="0.2032" layer="1"/>
-<wire x1="16.365" y1="98" x2="16" y2="98" width="0.2032" layer="1"/>
+<via x="17.5" y="98" extent="1-16" drill="0.5"/>
 <via x="12" y="89" extent="1-16" drill="0.35"/>
 <wire x1="14" y1="89" x2="14.05" y2="89" width="0.2032" layer="1"/>
@@
 <wire x1="42.05" y1="93" x2="40" y2="93" width="1.016" layer="1"/>
 <via x="40" y="93" extent="1-16" drill="0.35"/>
-<wire x1="51.54" y1="89" x2="53" y2="89" width="1.016" layer="1"/>
 <via x="53" y="89" extent="1-16" drill="0.35"/>
 <wire x1="13.35" y1="64.66" x2="13.6052375" y2="64.151053125" width="1.016" layer="1" curve="90"/>
@@
 <wire x1="54.95" y1="86" x2="57" y2="86" width="1.016" layer="1"/>
 <via x="57" y="86" extent="1-16" drill="0.35"/>
+<wire x1="48" y1="94" x2="53" y2="89" width="1.016" layer="1"/>
+<wire x1="17.365" y1="96.3622" x2="17.365" y2="97.865" width="0.4064" layer="1"/>
+<wire x1="17.365" y1="97.865" x2="17.5" y2="98" width="0.4064" layer="1"/>
 </signal>
 <signal name="N$1">
@@
 <wire x1="16" y1="83" x2="16" y2="88.95" width="1.016" layer="1"/>
 <wire x1="16" y1="88.95" x2="15.95" y2="89" width="1.016" layer="1"/>
-<wire x1="16.365" y1="91.6378" x2="16.365" y2="83.365" width="1.016" layer="1"/>
-<wire x1="16.365" y1="83.365" x2="16" y2="83" width="1.016" layer="1"/>
+<wire x1="17.365" y1="91.6378" x2="17.365" y2="84.365" width="1.016" layer="1"/>
+<wire x1="17.365" y1="84.365" x2="16.365" y2="83.365" width="1.016" layer="1"/>
 <wire x1="15.04" y1="76.49" x2="15.04" y2="75.04" width="1.016" layer="1"/>
 <wire x1="15.04" y1="75.04" x2="15" y2="75" width="1.016" layer="1"/>
@@
 <wire x1="15.04" y1="76.49" x2="12.39" y2="76.49" width="1.016" layer="1"/>
 <wire x1="12.39" y1="76.49" x2="11.9" y2="76" width="1.016" layer="1"/>
+<wire x1="16.365" y1="83.365" x2="16" y2="83" width="1.016" layer="1"/>
 </signal>
 <signal name="N$2">
@@
 <contactref element="R13" pad="1"/>
 <contactref element="Q1" pad="2"/>
-<wire x1="48.95" y1="93" x2="49" y2="89" width="1.016" layer="1"/>
+<wire x1="47.703703125" y1="94.246296875" x2="48.95" y2="93" width="1.016" layer="1"/>
+<wire x1="12" y1="96" x2="47.703703125" y2="94.246296875" width="0" layer="19" extent="1-1"/>
 </signal>
 <signal name="N$72">
@@
 <contactref element="U35" pad="5"/>
 <contactref element="R14" pad="1"/>
-<wire x1="5.7" y1="91.9" x2="11.76" y2="91.9" width="1.016" layer="1"/>
-<wire x1="11.76" y1="91.9" x2="11.93" y2="92.07" width="1.016" layer="1"/>
-<wire x1="11.93" y1="92.07" x2="12.97" y2="93.11" width="1.016" layer="1"/>
-<wire x1="15.095" y1="91.6378" x2="14.6628" y2="92.07" width="1.016" layer="1"/>
-<wire x1="14.6628" y1="92.07" x2="11.93" y2="92.07" width="1.016" layer="1"/>
-<wire x1="15.095" y1="91.6378" x2="13.6228" y2="93.11" width="1.016" layer="1"/>
-<wire x1="13.6228" y1="93.11" x2="12.97" y2="93.11" width="1.016" layer="1"/>
+<wire x1="8.76" y1="91.9" x2="8.93" y2="92.07" width="0.508" layer="1"/>
+<wire x1="9.4422" y1="91.6378" x2="16.095" y2="91.6378" width="0.508" layer="1"/>
+<wire x1="9.4422" y1="91.6378" x2="8.97" y2="92.11" width="0.508" layer="1"/>
+<wire x1="6.3" y1="91.9" x2="6.47" y2="92.07" width="1.016" layer="1"/>
+<wire x1="6.47" y1="92.07" x2="8.93" y2="92.07" width="1.016" layer="1"/>
+<wire x1="8.93" y1="92.07" x2="8.97" y2="92.11" width="1.016" layer="1"/>
 </signal>
 <signal name="N$12">
@@
 <contactref element="R6" pad="2"/>
 <contactref element="Q1" pad="3"/>
-<wire x1="12.97" y1="95.01" x2="13.5088" y2="94.4712" width="1.016" layer="1"/>
-<wire x1="13.5088" y1="94.4712" x2="14.0645875" y2="94.4712" width="1.016" layer="1"/>
-<wire x1="14.0645875" y1="94.4712" x2="14.5357875" y2="94" width="1.016" layer="1"/>
-<wire x1="35" y1="94" x2="40" y2="89" width="1.016" layer="1"/>
-<wire x1="40" y1="89" x2="46.46" y2="89" width="1.016" layer="1"/>
-<wire x1="14.5357875" y1="94" x2="35" y2="94" width="1.016" layer="1"/>
-<wire x1="5.7" y1="96.9" x2="11.08" y2="96.9" width="1.016" layer="1"/>
-<wire x1="11.08" y1="96.9" x2="12.97" y2="95.01" width="1.016" layer="1"/>
-<wire x1="48" y1="81.95" x2="48" y2="87.46" width="1.016" layer="1"/>
-<wire x1="48" y1="87.46" x2="46.46" y2="89" width="1.016" layer="1" curve="90"/>
+<wire x1="8.97" y1="94.01" x2="6.3" y2="96.68" width="1.016" layer="1"/>
+<wire x1="48" y1="81.95" x2="37.51" y2="81.95" width="1.016" layer="1"/>
+<wire x1="6.3" y1="96.68" x2="6.3" y2="96.9" width="1.016" layer="1"/>
+<wire x1="8.97" y1="94.01" x2="12" y2="93.46" width="0" layer="19" extent="1-1"/>
+<wire x1="37.51" y1="81.95" x2="12" y2="93.46" width="0" layer="19" extent="1-1"/>
 </signal>
 <signal name="N$13">
 <contactref element="U35" pad="4"/>
 <contactref element="U$2" pad="36/A17"/>
-<wire x1="15.095" y1="96.905" x2="15.095" y2="96.3622" width="1.016" layer="1"/>
-<wire x1="15.095" y1="96.905" x2="14" y2="98" width="1.016" layer="1" curve="90"/>
-<via x="14" y="98" extent="1-16" drill="0.35"/>
+<via x="16" y="98" extent="1-16" drill="0.5"/>
 <wire x1="23" y1="84.1" x2="52.79" y2="54.31" width="1.016" layer="16"/>
-<wire x1="23" y1="94" x2="23" y2="84.1" width="1.016" layer="16"/>
-<wire x1="18" y1="99" x2="23" y2="94" width="1.016" layer="16"/>
-<wire x1="15" y1="99" x2="18" y2="99" width="1.016" layer="16"/>
-<wire x1="14" y1="98" x2="15" y2="99" width="1.016" layer="16"/>
+<wire x1="23" y1="97" x2="23" y2="84.1" width="1.016" layer="16"/>
+<wire x1="16.095" y1="96.3622" x2="16.095" y2="97.905" width="0.508" layer="1"/>
+<wire x1="16.095" y1="97.905" x2="16" y2="98" width="0.508" layer="1"/>
+<wire x1="20.6604" y1="99.3396" x2="23" y2="97" width="0.8128" layer="16"/>
+<wire x1="16" y1="98" x2="17.3396" y2="99.3396" width="0.8128" layer="16"/>
+<wire x1="17.3396" y1="99.3396" x2="20.6604" y2="99.3396" width="0.8128" layer="16"/>
 </signal>
 <signal name="N$14">
