File: eagle/ProjectX/Driver_Board_Niall.sch (EAGLE design)
At the start: 13 parts, among them IC1 LM317MBSTT3

Commit message: Work in progress driver board
Parts:
- added R6: 100K, resistor:R-US_M0805
- added U1, U2: ADA4091-2ARZ-RL, SnapEDA-Library:ADA4091-2ARZ-RL
- added VAR-RESISTOR: MCP4011T-503E/SN, SnapEDA-Library:MCP4011T-503E/SN
Connections:
- removed net VO: C2.+, D1.A, D2.C, IC1.OUT, R1.2, R3.2
- new net 12VOLT: C2.+, D1.A, D2.C, IC1.OUT, R1.2, R3.2, U1.V+
- new net N$4: U1.INA-, U1.OUTA
- net GND: now also U1.V-, VAR-RESISTOR.A
- net N$2: now also U1.INA+, VAR-RESISTOR.W
Other:
- moved on the sheet: R4, R5
Changed lines of the file:
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@@
 <attribute name="PARTNUMBER" value="LM317M"/>
 </part>
-<part name="R1" library="resistor" library_urn="urn:adsk.eagle:library:348" deviceset="R-US_" device="M0805" package3d_urn="urn:adsk.eagle:package:26079/1" value="240Ω"/>
+<part name="R1" library="resistor" library_urn="urn:adsk.eagle:library:348" deviceset="R-US_" device="M0805" package3d_urn="urn:adsk.eagle:package:23556/1" value="240Ω"/>
 <part name="C1" library="rcl" library_urn="urn:adsk.eagle:library:334" deviceset="C-EU" device="075-052X106" package3d_urn="urn:adsk.eagle:package:23650/1" value="0.1uF"/>
-<part name="C2" library="resistor" library_urn="urn:adsk.eagle:library:348" deviceset="CPOL-US" device="085CS-1AR" package3d_urn="urn:adsk.eagle:package:25875/1" value="1uF"/>
-<part name="C3" library="resistor" library_urn="urn:adsk.eagle:library:348" deviceset="CPOL-US" device="085CS-1AR" package3d_urn="urn:adsk.eagle:package:25875/1" value="10uF"/>
+<part name="C2" library="resistor" library_urn="urn:adsk.eagle:library:348" deviceset="CPOL-US" device="085CS-1AR" package3d_urn="urn:adsk.eagle:package:23396/1" value="1uF"/>
+<part name="C3" library="resistor" library_urn="urn:adsk.eagle:library:348" deviceset="CPOL-US" device="085CS-1AR" package3d_urn="urn:adsk.eagle:package:23396/1" value="10uF"/>
 <part name="D1" library="diode" deviceset="1N4004" device="" package3d_urn="urn:adsk.eagle:package:43336/1" value="1N4002"/>
 <part name="D2" library="diode" deviceset="1N4004" device="" package3d_urn="urn:adsk.eagle:package:43336/1" value="1N4002"/>
 <part name="SUPPLY3" library="supply1" library_urn="urn:adsk.eagle:library:371" deviceset="GND" device=""/>
-<part name="R2" library="resistor" library_urn="urn:adsk.eagle:library:348" deviceset="R-US_" device="M0805" package3d_urn="urn:adsk.eagle:package:26079/1" value="2.1K"/>
+<part name="R2" library="resistor" library_urn="urn:adsk.eagle:library:348" deviceset="R-US_" device="M0805" package3d_urn="urn:adsk.eagle:package:23556/1" value="2.1K"/>
 <part name="SUPPLY1" library="supply1" library_urn="urn:adsk.eagle:library:371" deviceset="GND" device=""/>
 <part name="SUPPLY2" library="supply1" library_urn="urn:adsk.eagle:library:371" deviceset="GND" device=""/>
 <part name="SUPPLY4" library="supply1" library_urn="urn:adsk.eagle:library:371" deviceset="GND" device=""/>
-<part name="R3" library="resistor" library_urn="urn:adsk.eagle:library:348" deviceset="R-US_" device="M0805" package3d_urn="urn:adsk.eagle:package:26079/1" value="10K"/>
-<part name="R4" library="resistor" library_urn="urn:adsk.eagle:library:348" deviceset="R-US_" device="M0805" package3d_urn="urn:adsk.eagle:package:26079/1" value="9K"/>
-<part name="R5" library="resistor" library_urn="urn:adsk.eagle:library:348" deviceset="R-US_" device="M0805" package3d_urn="urn:adsk.eagle:package:26079/1" value="1K"/>
+<part name="R3" library="resistor" library_urn="urn:adsk.eagle:library:348" deviceset="R-US_" device="M0805" package3d_urn="urn:adsk.eagle:package:23556/1" value="10K"/>
+<part name="R4" library="resistor" library_urn="urn:adsk.eagle:library:348" deviceset="R-US_" device="M0805" package3d_urn="urn:adsk.eagle:package:23556/1" value="9K"/>
+<part name="R5" library="resistor" library_urn="urn:adsk.eagle:library:348" deviceset="R-US_" device="M0805" package3d_urn="urn:adsk.eagle:package:23556/1" value="1K"/>
 <part name="ZENER1" library="diode" library_urn="urn:adsk.eagle:library:210" deviceset="ZENER-DIODE" device="C1702-15" package3d_urn="urn:adsk.eagle:package:43351/1" value="3.3V"/>
 <part name="SUPPLY5" library="supply1" library_urn="urn:adsk.eagle:library:371" deviceset="GND" device=""/>
 <part name="SUPPLY6" library="supply1" library_urn="urn:adsk.eagle:library:371" deviceset="GND" device=""/>
 <part name="U$2" library="Teensy356" deviceset="TEENSY_3.5/3.6" device=""/>
+<part name="U1" library="SnapEDA-Library" deviceset="ADA4091-2ARZ-RL" device=""/>
+<part name="SUPPLY7" library="supply1" library_urn="urn:adsk.eagle:library:371" deviceset="GND" device=""/>
+<part name="U2" library="SnapEDA-Library" deviceset="ADA4091-2ARZ-RL" device=""/>
+<part name="R6" library="resistor" library_urn="urn:adsk.eagle:library:348" deviceset="R-US_" device="M0805" package3d_urn="urn:adsk.eagle:package:23556/1" value="100K"/>
+<part name="VAR-RESISTOR" library="SnapEDA-Library" deviceset="MCP4011T-503E/SN" device=""/>
 </parts>
 <sheets>
@@
 <attribute name="VALUE" x="50.292" y="179.07" size="1.778" layer="96" rot="R180"/>
 </instance>
-<instance part="R4" gate="G$1" x="73.66" y="165.1" smashed="yes" rot="R90">
-<attribute name="NAME" x="78.1614" y="169.29" size="1.778" layer="95" rot="R180"/>
-<attribute name="VALUE" x="80.772" y="166.37" size="1.778" layer="96" rot="R180"/>
-</instance>
-<instance part="R5" gate="G$1" x="73.66" y="152.4" smashed="yes" rot="R90">
-<attribute name="NAME" x="78.1614" y="156.59" size="1.778" layer="95" rot="R180"/>
-<attribute name="VALUE" x="80.772" y="153.67" size="1.778" layer="96" rot="R180"/>
+<instance part="R4" gate="G$1" x="66.04" y="165.1" smashed="yes" rot="R90">
+<attribute name="NAME" x="70.5414" y="169.29" size="1.778" layer="95" rot="R180"/>
+<attribute name="VALUE" x="73.152" y="166.37" size="1.778" layer="96" rot="R180"/>
+</instance>
+<instance part="R5" gate="G$1" x="66.04" y="152.4" smashed="yes" rot="R90">
+<attribute name="NAME" x="70.5414" y="156.59" size="1.778" layer="95" rot="R180"/>
+<attribute name="VALUE" x="73.152" y="153.67" size="1.778" layer="96" rot="R180"/>
 </instance>
 <instance part="ZENER1" gate="G$1" x="43.18" y="165.1" rot="R90"/>
 <instance part="SUPPLY5" gate="1" x="43.18" y="160.02"/>
-<instance part="SUPPLY6" gate="1" x="73.66" y="144.78"/>
+<instance part="SUPPLY6" gate="1" x="66.04" y="144.78"/>
 <instance part="U$2" gate="G$1" x="-38.1" y="96.52"/>
+<instance part="U1" gate="A" x="129.54" y="157.48"/>
+<instance part="SUPPLY7" gate="1" x="111.76" y="142.24"/>
+<instance part="U2" gate="A" x="215.9" y="134.62"/>
+<instance part="R6" gate="G$1" x="180.34" y="165.1" smashed="yes" rot="R180">
+<attribute name="NAME" x="176.15" y="169.6014" size="1.778" layer="95" rot="R270"/>
+<attribute name="VALUE" x="179.07" y="172.212" size="1.778" layer="96" rot="R270"/>
+</instance>
+<instance part="VAR-RESISTOR" gate="A" x="81.28" y="106.68" rot="R90"/>
 </instances>
 <busses>
@@
 <pinref part="R5" gate="G$1" pin="1"/>
 <pinref part="SUPPLY6" gate="1" pin="GND"/>
+<wire x1="66.04" y1="147.32" x2="81.28" y2="147.32" width="0.1524" layer="91"/>
+<junction x="66.04" y="147.32"/>
+<pinref part="VAR-RESISTOR" gate="A" pin="A"/>
+<wire x1="81.28" y1="147.32" x2="81.28" y2="142.24" width="0.1524" layer="91"/>
+</segment>
+<segment>
+<pinref part="U1" gate="A" pin="V-"/>
+<pinref part="SUPPLY7" gate="1" pin="GND"/>
 </segment>
 </net>
@@
 </segment>
 </net>
-<net name="VO" class="0">
+<net name="12VOLT" class="0">
 <segment>
 <pinref part="D2" gate="1" pin="C"/>
@@
 <junction x="10.16" y="182.88"/>
 <pinref part="R3" gate="G$1" pin="2"/>
-<wire x1="10.16" y1="182.88" x2="35.56" y2="182.88" width="0.1524" layer="91"/>
+<wire x1="10.16" y1="182.88" x2="20.32" y2="182.88" width="0.1524" layer="91"/>
+<wire x1="20.32" y1="182.88" x2="35.56" y2="182.88" width="0.1524" layer="91"/>
 <wire x1="35.56" y1="182.88" x2="43.18" y2="182.88" width="0.1524" layer="91"/>
+<pinref part="U1" gate="A" pin="V+"/>
+<wire x1="20.32" y1="182.88" x2="111.76" y2="182.88" width="0.1524" layer="91"/>
+<wire x1="111.76" y1="182.88" x2="111.76" y2="165.1" width="0.1524" layer="91"/>
+<junction x="20.32" y="182.88"/>
 </segment>
 </net>
@@
 <wire x1="43.18" y1="170.18" x2="43.18" y2="167.64" width="0.1524" layer="91"/>
 <pinref part="R4" gate="G$1" pin="2"/>
-<wire x1="43.18" y1="170.18" x2="73.66" y2="170.18" width="0.1524" layer="91"/>
+<wire x1="43.18" y1="170.18" x2="66.04" y2="170.18" width="0.1524" layer="91"/>
 <junction x="43.18" y="170.18"/>
 </segment>
@@
 <pinref part="R4" gate="G$1" pin="1"/>
 <pinref part="R5" gate="G$1" pin="2"/>
-<wire x1="73.66" y1="157.48" x2="73.66" y2="160.02" width="0.1524" layer="91"/>
+<wire x1="66.04" y1="157.48" x2="66.04" y2="160.02" width="0.1524" layer="91"/>
+<pinref part="U1" gate="A" pin="INA+"/>
+<wire x1="66.04" y1="160.02" x2="83.82" y2="160.02" width="0.1524" layer="91"/>
+<wire x1="83.82" y1="160.02" x2="91.44" y2="160.02" width="0.1524" layer="91"/>
+<wire x1="91.44" y1="160.02" x2="101.6" y2="160.02" width="0.1524" layer="91"/>
+<wire x1="101.6" y1="160.02" x2="111.76" y2="160.02" width="0.1524" layer="91"/>
+<junction x="66.04" y="160.02"/>
+<pinref part="VAR-RESISTOR" gate="A" pin="W"/>
+<wire x1="83.82" y1="142.24" x2="83.82" y2="160.02" width="0.1524" layer="91"/>
+<junction x="83.82" y="160.02"/>
+</segment>
+</net>
+<net name="N$4" class="0">
+<segment>
+<pinref part="U1" gate="A" pin="OUTA"/>
+<pinref part="U1" gate="A" pin="INA-"/>
+<wire x1="147.32" y1="165.1" x2="162.56" y2="165.1" width="0.1524" layer="91"/>
+<wire x1="162.56" y1="165.1" x2="162.56" y2="157.48" width="0.1524" layer="91"/>
+<junction x="162.56" y="165.1"/>
+<junction x="162.56" y="157.48"/>
+<wire x1="162.56" y1="157.48" x2="111.76" y2="157.48" width="0.1524" layer="91"/>
 </segment>
 </net>
@@
 packages will not be understood (or retained) with this version.
 </note>
+<note version="8.4" severity="warning">
+Since Version 8.4, EAGLE supports properties for SPICE simulation.
+Probes in schematics and SPICE mapping objects found in parts and library devices
+will not be understood with this version. Update EAGLE to the latest version
+for full support of SPICE simulation.
+</note>
 </compatibility>

Commit message: Eagle work- niall
Parts:
- removed VAR-RESISTOR: MCP4011T-503E/SN, SnapEDA-Library:MCP4011T-503E/SN
- added C35: 100nF, resistor:C-EUC0805
- added Q1: 2N7000G, SnapEDA-Library:2N7000G
- added R10: 1.2k, resistor:R-US_M0805
- added R11: 330, resistor:R-US_M0805
- added R12: 1M, resistor:R-US_M0805
- added R13: 100, resistor:R-US_M0805
- added R14: 10k, resistor:R-US_M0805
- added R7: 100K, resistor:R-US_M0805
- added R8: 33K, resistor:R-US_M0805
- added R9: 1K, resistor:R-US_M0805
- added T3: MA40S4S, Parts:MA40S4S
- added U35: TC4427AEOA, Parts:TC4427AEOA
- R4: value 9K -> 10K
Connections:
- removed net 12VOLT: C2.+, D1.A, D2.C, IC1.OUT, R1.2, R3.2, U1.V+
- new net N$10: R12.2, R13.2, U$2.35/A16
- new net N$11: Q1.GATE, R13.1
- new net N$12: R14.2, T3.1
- new net N$13: U$2.36/A17, U35.IN_B
- new net N$5: R6.1, R7.2, U2.INA+
- new net N$6: Q1.DRN, R6.2
- new net N$7: R10.2, R8.1, U2.OUTA
- new net N$72: R14.1, T3.2, U35.*OUT_B
- new net N$8: R8.2, R9.1, U2.INA-
- new net N$9: R10.1, R11.2, U$2.23/A9
- new net VDD: C2.+, D1.A, D2.C, IC1.OUT, R1.2, R3.2, U1.V+, U2.V+
- net GND: now also C35.1, Q1.SRC, R11.1, R12.1, R9.2, U2.V-, U35.GND; no longer VAR-RESISTOR.A
- net N$2: no longer VAR-RESISTOR.W
- net N$4: now also R7.1
- net VIN: now also C35.2, U35.VDD
Other:
- moved on the sheet: R3, R4, R5, R6, U1, U2, ZENER1

Commit message: Niall bord edits
Parts:
- added C4, C5: 100nF, resistor:C-EUC0805
- added R15, R16: (no value), pot:TRIM_EU-CA6V
Connections:
- removed net N$8: R8.2, R9.1, U2.INA-
- new net N$14: R16.A, R8.2, R9.1, U2.INA-
- net GND: now also C4.2, C5.2
- net N$2: now also R15.S
- net N$3: now also R15.A
- net N$7: now also R16.S
- net VDD: now also C4.1, C5.1
Other:
- moved on the sheet: R8
Changed lines of the file:
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@@
 <part name="SUPPLY13" library="SparkFun-PowerSymbols" library_urn="urn:adsk.eagle:library:530" deviceset="VDD" device=""/>
 <part name="SUPPLY14" library="SparkFun-PowerSymbols" library_urn="urn:adsk.eagle:library:530" deviceset="VDD" device=""/>
+<part name="R15" library="pot" library_urn="urn:adsk.eagle:library:331" deviceset="TRIM_EU-" device="CA6V" package3d_urn="urn:adsk.eagle:package:22691/1"/>
+<part name="R16" library="pot" library_urn="urn:adsk.eagle:library:331" deviceset="TRIM_EU-" device="CA6V" package3d_urn="urn:adsk.eagle:package:22691/1"/>
+<part name="C4" library="resistor" library_urn="urn:adsk.eagle:library:348" deviceset="C-EU" device="C0805" package3d_urn="urn:adsk.eagle:package:26137/1" value="100nF"/>
+<part name="SUPPLY15" library="supply1" library_urn="urn:adsk.eagle:library:371" deviceset="GND" device=""/>
+<part name="C5" library="resistor" library_urn="urn:adsk.eagle:library:348" deviceset="C-EU" device="C0805" package3d_urn="urn:adsk.eagle:package:26137/1" value="100nF"/>
+<part name="SUPPLY17" library="supply1" library_urn="urn:adsk.eagle:library:371" deviceset="GND" device=""/>
 </parts>
 <sheets>
@@
 <attribute name="VALUE" x="159.512" y="156.21" size="1.778" layer="96" rot="R180"/>
 </instance>
-<instance part="R8" gate="G$1" x="167.64" y="139.7" smashed="yes" rot="R180">
-<attribute name="NAME" x="165.6786" y="143.13" size="1.778" layer="95"/>
-<attribute name="VALUE" x="165.608" y="140.97" size="1.778" layer="96"/>
+<instance part="R8" gate="G$1" x="172.72" y="139.7" smashed="yes" rot="R180">
+<attribute name="NAME" x="170.7586" y="143.13" size="1.778" layer="95"/>
+<attribute name="VALUE" x="170.688" y="140.97" size="1.778" layer="96"/>
 </instance>
 <instance part="SUPPLY8" gate="1" x="162.56" y="127"/>
@@
 <instance part="SUPPLY13" gate="VDD" x="83.82" y="165.1" rot="R90"/>
 <instance part="SUPPLY14" gate="VDD" x="175.26" y="170.18" rot="R90"/>
+<instance part="R15" gate="1" x="63.5" y="175.26" rot="R270"/>
+<instance part="R16" gate="1" x="180.34" y="129.54" rot="R270"/>
+<instance part="C4" gate="G$1" x="83.82" y="172.72" rot="R180"/>
+<instance part="SUPPLY15" gate="1" x="83.82" y="182.88" rot="R180"/>
+<instance part="C5" gate="G$1" x="175.26" y="177.8" rot="R180"/>
+<instance part="SUPPLY17" gate="1" x="175.26" y="187.96" rot="R180"/>
 </instances>
 <busses>
@@
 <wire x1="121.92" y1="281.94" x2="121.92" y2="284.48" width="0.1524" layer="91"/>
 <junction x="121.92" y="281.94"/>
+</segment>
+<segment>
+<pinref part="C4" gate="G$1" pin="2"/>
+<wire x1="83.82" y1="177.8" x2="83.82" y2="180.34" width="0.1524" layer="91"/>
+<pinref part="SUPPLY15" gate="1" pin="GND"/>
+</segment>
+<segment>
+<pinref part="C5" gate="G$1" pin="2"/>
+<wire x1="175.26" y1="182.88" x2="175.26" y2="185.42" width="0.1524" layer="91"/>
+<pinref part="SUPPLY17" gate="1" pin="GND"/>
 </segment>
 </net>
@@
 <pinref part="R4" gate="G$1" pin="2"/>
 <wire x1="48.26" y1="170.18" x2="55.88" y2="170.18" width="0.1524" layer="91"/>
+<wire x1="55.88" y1="170.18" x2="55.88" y2="175.26" width="0.1524" layer="91"/>
+<junction x="55.88" y="170.18"/>
+<pinref part="R15" gate="1" pin="A"/>
+<wire x1="55.88" y1="175.26" x2="58.42" y2="175.26" width="0.1524" layer="91"/>
 </segment>
 </net>
@@
 <pinref part="R5" gate="G$1" pin="2"/>
 <pinref part="U1" gate="A" pin="INA+"/>
-<wire x1="55.88" y1="160.02" x2="78.74" y2="160.02" width="0.1524" layer="91"/>
-<wire x1="78.74" y1="160.02" x2="63.5" y2="160.02" width="0.1524" layer="91"/>
-<wire x1="63.5" y1="160.02" x2="73.66" y2="160.02" width="0.1524" layer="91"/>
+<wire x1="55.88" y1="160.02" x2="66.04" y2="160.02" width="0.1524" layer="91"/>
+<wire x1="66.04" y1="160.02" x2="78.74" y2="160.02" width="0.1524" layer="91"/>
+<wire x1="78.74" y1="160.02" x2="66.04" y2="160.02" width="0.1524" layer="91"/>
+<wire x1="66.04" y1="160.02" x2="63.5" y2="160.02" width="0.1524" layer="91"/>
+<wire x1="63.5" y1="160.02" x2="66.04" y2="160.02" width="0.1524" layer="91"/>
+<wire x1="66.04" y1="160.02" x2="73.66" y2="160.02" width="0.1524" layer="91"/>
 <wire x1="73.66" y1="160.02" x2="83.82" y2="160.02" width="0.1524" layer="91"/>
 <junction x="55.88" y="160.02"/>
+<pinref part="R15" gate="1" pin="S"/>
+<wire x1="63.5" y1="170.18" x2="66.04" y2="170.18" width="0.1524" layer="91"/>
+<wire x1="66.04" y1="170.18" x2="66.04" y2="167.64" width="0.1524" layer="91"/>
+<wire x1="66.04" y1="167.64" x2="66.04" y2="160.02" width="0.1524" layer="91"/>
+<junction x="66.04" y="160.02"/>
 </segment>
 </net>
@@
 <pinref part="R8" gate="G$1" pin="1"/>
 <wire x1="223.52" y1="139.7" x2="223.52" y2="116.84" width="0.1524" layer="91"/>
-<wire x1="172.72" y1="139.7" x2="175.26" y2="139.7" width="0.1524" layer="91"/>
+<wire x1="177.8" y1="139.7" x2="175.26" y2="139.7" width="0.1524" layer="91"/>
 <wire x1="175.26" y1="139.7" x2="177.8" y2="139.7" width="0.1524" layer="91"/>
 <wire x1="177.8" y1="139.7" x2="185.42" y2="139.7" width="0.1524" layer="91"/>
-<wire x1="185.42" y1="139.7" x2="223.52" y2="139.7" width="0.1524" layer="91"/>
+<wire x1="185.42" y1="139.7" x2="193.04" y2="139.7" width="0.1524" layer="91"/>
 <junction x="223.52" y="139.7"/>
-</segment>
-</net>
-<net name="N$8" class="0">
-<segment>
-<pinref part="R8" gate="G$1" pin="2"/>
-<wire x1="162.56" y1="139.7" x2="162.56" y2="162.56" width="0.1524" layer="91"/>
-<pinref part="R9" gate="G$1" pin="1"/>
-<junction x="162.56" y="139.7"/>
-<pinref part="U2" gate="A" pin="INA-"/>
-<wire x1="162.56" y1="162.56" x2="175.26" y2="162.56" width="0.1524" layer="91"/>
+<pinref part="R16" gate="1" pin="S"/>
+<wire x1="193.04" y1="139.7" x2="223.52" y2="139.7" width="0.1524" layer="91"/>
+<wire x1="180.34" y1="124.46" x2="193.04" y2="124.46" width="0.1524" layer="91"/>
+<wire x1="193.04" y1="124.46" x2="193.04" y2="139.7" width="0.1524" layer="91"/>
+<junction x="193.04" y="139.7"/>
 </segment>
 </net>
@@
 <pinref part="U1" gate="A" pin="V+"/>
 <pinref part="SUPPLY13" gate="VDD" pin="VDD"/>
+<pinref part="C4" gate="G$1" pin="1"/>
+<wire x1="83.82" y1="165.1" x2="83.82" y2="170.18" width="0.1524" layer="91"/>
+<junction x="83.82" y="165.1"/>
 </segment>
 <segment>
@@
 <label x="175.26" y="172.72" size="1.778" layer="95"/>
 <pinref part="SUPPLY14" gate="VDD" pin="VDD"/>
+<pinref part="C5" gate="G$1" pin="1"/>
+<wire x1="175.26" y1="175.26" x2="175.26" y2="170.18" width="0.1524" layer="91"/>
+<junction x="175.26" y="170.18"/>
 </segment>
 </net>
@@
 </segment>
 </net>
+<net name="N$14" class="0">
+<segment>
+<pinref part="R9" gate="G$1" pin="1"/>
+<pinref part="R8" gate="G$1" pin="2"/>
+<wire x1="167.64" y1="139.7" x2="162.56" y2="139.7" width="0.1524" layer="91"/>
+<pinref part="U2" gate="A" pin="INA-"/>
+<wire x1="175.26" y1="162.56" x2="162.56" y2="162.56" width="0.1524" layer="91"/>
+<wire x1="162.56" y1="162.56" x2="162.56" y2="139.7" width="0.1524" layer="91"/>
+<junction x="162.56" y="139.7"/>
+<wire x1="167.64" y1="139.7" x2="167.64" y2="129.54" width="0.1524" layer="91"/>
+<wire x1="167.64" y1="129.54" x2="170.18" y2="129.54" width="0.1524" layer="91"/>
+<junction x="167.64" y="139.7"/>
+<pinref part="R16" gate="1" pin="A"/>
+<wire x1="170.18" y1="129.54" x2="175.26" y2="129.54" width="0.1524" layer="91"/>
+</segment>
+</net>

Commit message: Niall Board layout first attempt
Parts:
- removed ZENER1: 3.3V, diode:ZENER-DIODEC1702-15
- added J1: 694102303002, SnapEDA-Library:694102303002
- added ZENER: 3.3V, diode:ZENER-DIODEDO34-7
Connections:
- net VDD renamed $VDD
- removed net GND: C1.2, C2.-, C3.-, C35.1, C4.2, C5.2, Q1.SRC, R11.1, R12.1, R2.1, R5.1, R9.2, U1.V-, U2.V-, U35.GND, ZENER1.A
- removed net N$6: Q1.DRN, R6.2
- removed net VIN: C1.1, C35.2, D1.C, IC1.IN, U35.VDD
- new net $GND: C1.2, C2.-, C3.-, C35.1, C4.2, C5.2, J1.2, Q1.SRC, R11.1, R12.1, R2.1, R5.1, R9.2, U$2.GND, U1.V-, U2.V-, U35.GND, ZENER.A
- new net $VIN: C1.1, C35.2, D1.C, IC1.IN, J1.1, U35.VDD
- net N$12: now also Q1.DRN, R6.2
- net N$3: now also ZENER.C; no longer ZENER1.C

Commit message: Niall Board layout first attempt
Changed lines of the file:
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@@
 <wire x1="152.4" y1="149.86" x2="134.62" y2="149.86" width="0.1524" layer="91"/>
 <junction x="134.62" y="149.86"/>
+<label x="66.04" y="132.08" size="1.778" layer="95"/>
 </segment>
 </net>
@@
 <wire x1="193.04" y1="124.46" x2="193.04" y2="139.7" width="0.1524" layer="91"/>
 <junction x="193.04" y="139.7"/>
+<junction x="177.8" y="139.7"/>
 </segment>
 </net>
@@
 </sheet>
 </sheets>
+<errors>
+</errors>
 </schematic>
 </drawing>
