File: eagle/ProjectX/Driver_Board_Niall.sch (EAGLE design)
At the start: 33 parts, among them IC1 LM317MBSTT3, J1 694102303002, Q1 2N7000G, T3 MA40S4S, U1 ADA4091-2ARZ-RL, U2 ADA4091-2ARZ-RL, U35 TC4427AEOA

Commit message: Nialls slightly better board atempt 2
Parts:
- removed T3: MA40S4S, Parts:MA40S4S
- added SL1: (no value), con-amp-quick:M08
Connections:
- net N$12: now also SL1.7; no longer T3.1
- net N$72: now also SL1.8; no longer T3.2
Changed lines of the file:
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@@
 <part name="R12" library="resistor" library_urn="urn:adsk.eagle:library:348" deviceset="R-US_" device="M0805" package3d_urn="urn:adsk.eagle:package:23556/1" value="1M"/>
 <part name="R13" library="resistor" library_urn="urn:adsk.eagle:library:348" deviceset="R-US_" device="M0805" package3d_urn="urn:adsk.eagle:package:23556/1" value="100"/>
-<part name="T3" library="Parts" deviceset="MA40S4S" device=""/>
 <part name="U35" library="Parts" deviceset="TC4427AEOA" device=""/>
 <part name="GND74" library="supply1" library_urn="urn:adsk.eagle:library:371" deviceset="GND" device=""/>
@@
 <part name="SUPPLY16" library="supply1" library_urn="urn:adsk.eagle:library:371" deviceset="GND" device=""/>
 <part name="SUPPLY18" library="supply1" library_urn="urn:adsk.eagle:library:371" deviceset="GND" device=""/>
+<part name="SL1" library="con-amp-quick" library_urn="urn:adsk.eagle:library:125" deviceset="M08" device="" package3d_urn="urn:adsk.eagle:package:5962/1"/>
 </parts>
 <sheets>
@@
 <attribute name="VALUE" x="107.95" y="225.552" size="1.778" layer="96" rot="R270"/>
 </instance>
-<instance part="T3" gate="G$1" x="132.08" y="238.76" rot="R90"/>
 <instance part="U35" gate="A" x="134.62" y="264.16" rot="R270"/>
 <instance part="GND74" gate="1" x="119.38" y="281.94" rot="R270"/>
@@
 <instance part="SUPPLY16" gate="1" x="-81.28" y="170.18"/>
 <instance part="SUPPLY18" gate="1" x="-66.04" y="111.76"/>
+<instance part="SL1" gate="G$1" x="111.76" y="241.3"/>
 </instances>
 <busses>
@@
 <pinref part="U$2" gate="G$1" pin="23/A9"/>
 <wire x1="-7.62" y1="106.68" x2="-15.24" y2="106.68" width="0.1524" layer="91"/>
+<label x="20.32" y="99.06" size="1.778" layer="95"/>
 </segment>
 </net>
@@
 <pinref part="U$2" gate="G$1" pin="35/A16"/>
 <wire x1="-7.62" y1="60.96" x2="-15.24" y2="60.96" width="0.1524" layer="91"/>
+<label x="38.1" y="226.06" size="1.778" layer="95"/>
 </segment>
 </net>
@@
 <net name="N$72" class="0">
 <segment>
-<pinref part="T3" gate="G$1" pin="2"/>
-<wire x1="132.08" y1="243.84" x2="132.08" y2="248.92" width="0.1524" layer="91"/>
 <pinref part="U35" gate="A" pin="*OUT_B"/>
 <wire x1="132.08" y1="248.92" x2="132.08" y2="251.46" width="0.1524" layer="91"/>
@@
 <pinref part="R14" gate="G$1" pin="1"/>
 <wire x1="144.78" y1="248.92" x2="144.78" y2="243.84" width="0.1524" layer="91"/>
+<pinref part="SL1" gate="G$1" pin="8"/>
+<wire x1="116.84" y1="251.46" x2="121.92" y2="251.46" width="0.1524" layer="91"/>
+<wire x1="121.92" y1="251.46" x2="121.92" y2="248.92" width="0.1524" layer="91"/>
+<wire x1="121.92" y1="248.92" x2="132.08" y2="248.92" width="0.1524" layer="91"/>
 </segment>
 </net>
 <net name="N$12" class="0">
 <segment>
-<pinref part="T3" gate="G$1" pin="1"/>
-<wire x1="132.08" y1="233.68" x2="132.08" y2="228.6" width="0.1524" layer="91"/>
 <pinref part="R14" gate="G$1" pin="2"/>
 <wire x1="132.08" y1="228.6" x2="132.08" y2="226.06" width="0.1524" layer="91"/>
@@
 <wire x1="132.08" y1="226.06" x2="132.08" y2="223.52" width="0.1524" layer="91"/>
 <junction x="132.08" y="223.52"/>
+<pinref part="SL1" gate="G$1" pin="7"/>
+<wire x1="116.84" y1="248.92" x2="119.38" y2="248.92" width="0.1524" layer="91"/>
+<wire x1="119.38" y1="248.92" x2="119.38" y2="228.6" width="0.1524" layer="91"/>
+<wire x1="119.38" y1="228.6" x2="132.08" y2="228.6" width="0.1524" layer="91"/>
 </segment>
 </net>
@@
 <wire x1="-15.24" y1="63.5" x2="-5.08" y2="63.5" width="0.1524" layer="91"/>
 <wire x1="-5.08" y1="63.5" x2="-5.08" y2="58.42" width="0.1524" layer="91"/>
-</segment>
-</net>
+<label x="10.16" y="43.18" size="1.778" layer="95"/>
+</segment>
+</net>

Commit message: Nialls boards
Parts:
- removed C1: 0.1uF, rcl:C-EU075-052X106
- removed C2: 1uF, resistor:CPOL-US085CS-1AR
- removed C3: 10uF, resistor:CPOL-US085CS-1AR
- removed C4: 100nF, resistor:C-EUC0805
- removed D1, D2: 1N4002, diode:1N4004
- removed IC1: LM317MBSTT3, v-reg:LM317MBSTT3
- removed Q1: 2N7000G, SnapEDA-Library:2N7000G
- removed R1: 240Ω, resistor:R-US_M0805
- removed R15, R16: (no value), pot:TRIM_EU-CA6V
- removed R2: 2.1K, resistor:R-US_M0805
- removed R3: 10K, resistor:R-US_M0805
- removed U1: ADA4091-2ARZ-RL, SnapEDA-Library:ADA4091-2ARZ-RL
- removed ZENER: 3.3V, diode:ZENER-DIODEDO34-7
- added IC2: NCV78M05BDTRKG, linear:NCV78M05BDTRKG
- added Q2: 2N7002, SnapEDA-Library:2N7002
- added REFULATOR_TANTALUM: 0.33 uF, rcl:C-USC1206
- R4: value 10K -> 8.2k
- R5: value 1K -> Not Sure
- R8: value 33K -> Not Sure
Connections:
- removed net N$1: C3.+, D2.A, IC1.ADJ, R1.1, R2.2
- removed net N$3: R15.A, R3.1, R4.2, ZENER.C
- removed net N$4: R7.1, U1.INA-, U1.OUTA
- net $GND: now also IC2.GND, Q2.S, R5.2, REFULATOR_TANTALUM.2; no longer C1.2, C2.-, C3.-, C4.2, Q1.SRC, R2.1, R5.1, U1.V-, ZENER.A
- net $VDD: now also IC2.VO, R4.2; no longer C2.+, C4.1, D1.A, D2.C, IC1.OUT, R1.2, R3.2, U1.V+
- net $VIN: now also IC2.VI, REFULATOR_TANTALUM.1; no longer C1.1, D1.C, IC1.IN
- net N$11: now also Q2.G; no longer Q1.GATE
- net N$12: now also Q2.D; no longer Q1.DRN
- net N$14: no longer R16.A
- net N$2: now also R5.1, R7.1; no longer R15.S, R5.2, U1.INA+
- net N$7: no longer R16.S
Other:
- note removed: "C2 of 1 µF tantalum capacitor on the output helps to improve transient response"
- note removed: "C3 helps in ripple rejection upto 15dB"
- note removed: "D1 protect the device against input short circuit"
- note removed: "D2 protect against output short circuit for capacitance discharging"
- note removed: "Useful Notes"
- note removed: "Vref = 1.25V"
- moved on the sheet: R5

Commit message: Nialls's boards
Parts:
- added DIP1: CORE3S500ESMT, Parts:CORE3S500ESMT
- added U1: CD74HC4067SM96, SnapEDA-Library (3):CD74HC4067SM96
- added X1, X2: 1296-T50, con-leotronics:1296-T50
Connections:
- removed net N$5: R6.1, R7.2, U2.INA+
- new net N$1: R6.1, U1.S0
- new net N$3: R7.2, U1.COMMON_IN/OUT, U2.INA+
- net $GND: now also U1.GND
Other:
- note removed: "3V - 40V DC"
- moved on the sheet: C5, IC2, J1, R10, R11, R6, R7, R8, R9, REFULATOR_TANTALUM, U2
