File: eagle/ProjectX/Driver_Board_Niall.sch (EAGLE design)
At the start: 25 parts, among them IC2 NCV78M05BDTRKG, J1 694102303002, Q2 2N7002, U1 CD74HC4067SM96, U2 ADA4091-2ARZ-RL, U35 TC4427AEOA, X1 1296-T50, X2 1296-T50

Commit message: Niall board edits
Parts:
- removed X1, X2: 1296-T50, con-leotronics:1296-T50
Changed lines of the file:
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@@
 <part name="U1" library="SnapEDA-Library (3)" deviceset="CD74HC4067SM96" device=""/>
 <part name="SUPPLY2" library="supply1" library_urn="urn:adsk.eagle:library:371" deviceset="GND" device=""/>
-<part name="X1" library="con-leotronics" library_urn="urn:adsk.eagle:library:160" deviceset="1296-T50" device="" package3d_urn="urn:adsk.eagle:package:7940/1"/>
-<part name="X2" library="con-leotronics" library_urn="urn:adsk.eagle:library:160" deviceset="1296-T50" device="" package3d_urn="urn:adsk.eagle:package:7940/1"/>
 </parts>
 <sheets>
@@
 <instance part="U1" gate="A" x="213.36" y="233.68"/>
 <instance part="SUPPLY2" gate="1" x="187.96" y="190.5" rot="MR0"/>
-<instance part="X1" gate="-1" x="-287.02" y="38.1"/>
-<instance part="X1" gate="-2" x="-256.54" y="38.1"/>
-<instance part="X1" gate="-3" x="-287.02" y="35.56"/>
-<instance part="X1" gate="-4" x="-256.54" y="35.56"/>
-<instance part="X1" gate="-5" x="-287.02" y="33.02"/>
-<instance part="X1" gate="-6" x="-256.54" y="33.02"/>
-<instance part="X1" gate="-7" x="-287.02" y="30.48"/>
-<instance part="X1" gate="-8" x="-256.54" y="30.48"/>
-<instance part="X1" gate="-9" x="-287.02" y="27.94"/>
-<instance part="X1" gate="-10" x="-256.54" y="27.94"/>
-<instance part="X1" gate="-11" x="-287.02" y="25.4"/>
-<instance part="X1" gate="-12" x="-256.54" y="25.4"/>
-<instance part="X1" gate="-13" x="-287.02" y="22.86"/>
-<instance part="X1" gate="-14" x="-256.54" y="22.86"/>
-<instance part="X1" gate="-15" x="-287.02" y="20.32"/>
-<instance part="X1" gate="-16" x="-256.54" y="20.32"/>
-<instance part="X1" gate="-17" x="-287.02" y="17.78"/>
-<instance part="X1" gate="-18" x="-256.54" y="17.78"/>
-<instance part="X1" gate="-19" x="-287.02" y="15.24"/>
-<instance part="X1" gate="-20" x="-256.54" y="15.24"/>
-<instance part="X1" gate="-21" x="-287.02" y="12.7"/>
-<instance part="X1" gate="-22" x="-256.54" y="12.7"/>
-<instance part="X1" gate="-23" x="-287.02" y="10.16"/>
-<instance part="X1" gate="-24" x="-256.54" y="10.16"/>
-<instance part="X1" gate="-25" x="-287.02" y="7.62"/>
-<instance part="X1" gate="-26" x="-256.54" y="7.62"/>
-<instance part="X1" gate="-27" x="-287.02" y="5.08"/>
-<instance part="X1" gate="-28" x="-256.54" y="5.08"/>
-<instance part="X1" gate="-29" x="-287.02" y="2.54"/>
-<instance part="X1" gate="-30" x="-256.54" y="2.54"/>
-<instance part="X1" gate="-31" x="-287.02" y="0"/>
-<instance part="X1" gate="-32" x="-256.54" y="0"/>
-<instance part="X1" gate="-33" x="-287.02" y="-2.54"/>
-<instance part="X1" gate="-34" x="-256.54" y="-2.54"/>
-<instance part="X1" gate="-35" x="-287.02" y="-5.08"/>
-<instance part="X1" gate="-36" x="-256.54" y="-5.08"/>
-<instance part="X1" gate="-37" x="-287.02" y="-7.62"/>
-<instance part="X1" gate="-38" x="-256.54" y="-7.62"/>
-<instance part="X1" gate="-39" x="-287.02" y="-10.16"/>
-<instance part="X1" gate="-40" x="-256.54" y="-10.16"/>
-<instance part="X1" gate="-41" x="-287.02" y="-12.7"/>
-<instance part="X1" gate="-42" x="-256.54" y="-12.7"/>
-<instance part="X1" gate="-43" x="-287.02" y="-15.24"/>
-<instance part="X1" gate="-44" x="-256.54" y="-15.24"/>
-<instance part="X1" gate="-45" x="-287.02" y="-17.78"/>
-<instance part="X1" gate="-46" x="-256.54" y="-17.78"/>
-<instance part="X1" gate="-47" x="-287.02" y="-20.32"/>
-<instance part="X1" gate="-48" x="-256.54" y="-20.32"/>
-<instance part="X1" gate="-49" x="-287.02" y="-22.86"/>
-<instance part="X1" gate="-50" x="-256.54" y="-22.86"/>
-<instance part="X2" gate="-1" x="-228.6" y="38.1"/>
-<instance part="X2" gate="-2" x="-198.12" y="38.1"/>
-<instance part="X2" gate="-3" x="-228.6" y="35.56"/>
-<instance part="X2" gate="-4" x="-198.12" y="35.56"/>
-<instance part="X2" gate="-5" x="-228.6" y="33.02"/>
-<instance part="X2" gate="-6" x="-198.12" y="33.02"/>
-<instance part="X2" gate="-7" x="-228.6" y="30.48"/>
-<instance part="X2" gate="-8" x="-198.12" y="30.48"/>
-<instance part="X2" gate="-9" x="-228.6" y="27.94"/>
-<instance part="X2" gate="-10" x="-198.12" y="27.94"/>
-<instance part="X2" gate="-11" x="-228.6" y="25.4"/>
-<instance part="X2" gate="-12" x="-198.12" y="25.4"/>
-<instance part="X2" gate="-13" x="-228.6" y="22.86"/>
-<instance part="X2" gate="-14" x="-198.12" y="22.86"/>
-<instance part="X2" gate="-15" x="-228.6" y="20.32"/>
-<instance part="X2" gate="-16" x="-198.12" y="20.32"/>
-<instance part="X2" gate="-17" x="-228.6" y="17.78"/>
-<instance part="X2" gate="-18" x="-198.12" y="17.78"/>
-<instance part="X2" gate="-19" x="-228.6" y="15.24"/>
-<instance part="X2" gate="-20" x="-198.12" y="15.24"/>
-<instance part="X2" gate="-21" x="-228.6" y="12.7"/>
-<instance part="X2" gate="-22" x="-198.12" y="12.7"/>
-<instance part="X2" gate="-23" x="-228.6" y="10.16"/>
-<instance part="X2" gate="-24" x="-198.12" y="10.16"/>
-<instance part="X2" gate="-25" x="-228.6" y="7.62"/>
-<instance part="X2" gate="-26" x="-198.12" y="7.62"/>
-<instance part="X2" gate="-27" x="-228.6" y="5.08"/>
-<instance part="X2" gate="-28" x="-198.12" y="5.08"/>
-<instance part="X2" gate="-29" x="-228.6" y="2.54"/>
-<instance part="X2" gate="-30" x="-198.12" y="2.54"/>
-<instance part="X2" gate="-31" x="-228.6" y="0"/>
-<instance part="X2" gate="-32" x="-198.12" y="0"/>
-<instance part="X2" gate="-33" x="-228.6" y="-2.54"/>
-<instance part="X2" gate="-34" x="-198.12" y="-2.54"/>
-<instance part="X2" gate="-35" x="-228.6" y="-5.08"/>
-<instance part="X2" gate="-36" x="-198.12" y="-5.08"/>
-<instance part="X2" gate="-37" x="-228.6" y="-7.62"/>
-<instance part="X2" gate="-38" x="-198.12" y="-7.62"/>
-<instance part="X2" gate="-39" x="-228.6" y="-10.16"/>
-<instance part="X2" gate="-40" x="-198.12" y="-10.16"/>
-<instance part="X2" gate="-41" x="-228.6" y="-12.7"/>
-<instance part="X2" gate="-42" x="-198.12" y="-12.7"/>
-<instance part="X2" gate="-43" x="-228.6" y="-15.24"/>
-<instance part="X2" gate="-44" x="-198.12" y="-15.24"/>
-<instance part="X2" gate="-45" x="-228.6" y="-17.78"/>
-<instance part="X2" gate="-46" x="-198.12" y="-17.78"/>
-<instance part="X2" gate="-47" x="-228.6" y="-20.32"/>
-<instance part="X2" gate="-48" x="-198.12" y="-20.32"/>
-<instance part="X2" gate="-49" x="-228.6" y="-22.86"/>
-<instance part="X2" gate="-50" x="-198.12" y="-22.86"/>
 </instances>
 <busses>

Commit message: Nialls board changes
Parts:
- removed U$2: TEENSY_3.5/3.6, Teensy356:TEENSY_3.5/3.6
- added U$1: TEENSY_SMD, Parts:TEENSY_SMD
- added X1, X2, X3, X4, X5, X6: 87758-2016, con-molex:87758-2016
Connections:
- removed net N$4: R10.1, R11.2, U$2.23/A9
- new net GND: U$1.GND
- new net N$5: R10.1, R11.2, U$1.23/A9
- net $GND: no longer U$2.GND
- net N$10: now also U$1.35/A16; no longer U$2.35/A16
- net N$13: now also U$1.36/A17; no longer U$2.36/A17

Commit message: Niall's work in progress board
Parts:
- removed DIP1: CORE3S500ESMT, Parts:CORE3S500ESMT
- removed SL1: (no value), con-amp-quick:M08
- removed X1, X2, X3, X4, X5, X6: 87758-2016, con-molex:87758-2016
- added 5V-REG: OKI-78SR, Parts:OKI-78SR
- added C1, C10, C11, C12, C13, C14, C15, C16, C17, C18, C19, C2, C20, C21, C22, C23, C24, C25, C26, C27, C28, C29, C3, C30, C31, C32, C33, C34, C36, C37, C38, C39, C4, C40, C41, C42, C43, C44, C45, C46, C47, C48, C49, C50, C6, C7, C8, C9, C90, C905: 100nF, resistor:C-EUC0805
- added DATA: Data, SparkFun-Connectors:CONN_11
- added DIP2: CORE3S500ESMT, Parts:CORE3S500ESMT
- added JP1, JP2, JP3: (no value), pinhead:PINHD-2X20
- added U10, U11, U12, U13, U14, U15, U16, U17, U18, U19, U20, U21, U22, U23, U24, U25, U26, U27, U28, U29, U3, U30, U31, U32, U33, U34, U36, U37, U38, U39, U4, U40, U41, U42, U43, U44, U45, U46, U47, U48, U49, U5, U50, U6, U7, U8, U9, U900: TC4427AEOA, Parts:TC4427AEOA
- added U1200: CD74HC4067SM96, SnapEDA-Library (3):CD74HC4067SM96
- added U200: ADA4091-2ARZ-RL, SnapEDA-Library:ADA4091-2ARZ-RL
- U1: value CD74HC4067SM96 -> TC4427AEOA; device SnapEDA-Library (3):CD74HC4067SM96 -> Parts:TC4427AEOA
- U2: value ADA4091-2ARZ-RL -> TC4427AEOA; device SnapEDA-Library:ADA4091-2ARZ-RL -> Parts:TC4427AEOA
Connections:
- removed net $GND: C35.1, C5.2, IC2.GND, J1.2, Q2.S, R11.1, R12.1, R5.2, R9.2, REFULATOR_TANTALUM.2, U1.GND, U2.V-, U35.GND
- removed net $VDD: C5.1, IC2.VO, R4.2, U2.V+
- removed net $VIN: C35.2, IC2.VI, J1.1, REFULATOR_TANTALUM.1, U35.VDD
- new net +12V: C905.1, IC2.VO, R4.2, U200.V+
- new net +5V: 5V-REG.OUT, DIP2.5V@1, DIP2.5V@2
- new net 1: U1.IN_A
- new net 100: U50.IN_B, U7.IN_B
- new net 101: U8.IN_A
- new net 102: U8.IN_B
- new net 103: U9.IN_A
- new net 104: U9.IN_B
- new net 105: U10.IN_A
- new net 106: U10.IN_B
- new net 107: U11.IN_A
- new net 108: U11.IN_B
- new net 109: U12.IN_A
- new net 110: U12.IN_B
- new net 111: U13.IN_A
- new net 112: U13.IN_B
- new net 113: U14.IN_A
- new net 114: U14.IN_B
- new net 115: U15.IN_A
- new net 116: U15.IN_B
- new net 117: U16.IN_A
- new net 118: U16.IN_B
- new net 119: U17.IN_A
- new net 120: U17.IN_B
- new net 121: U18.IN_A
- new net 122: U18.IN_B
- new net 123: U19.IN_A
- new net 124: U19.IN_B
- new net 125: U20.IN_A
- new net 126: U20.IN_B
- new net 127: U21.IN_A
- new net 128: U21.IN_B
- new net 129: U22.IN_A
- new net 130: U22.IN_B
- new net 131: U23.IN_A
- new net 132: U23.IN_B
- new net 133: U24.IN_A
- new net 134: U24.IN_B
- new net 135: U25.IN_A
- new net 136: U25.IN_B
- new net 137: U26.IN_A
- new net 138: U26.IN_B
- new net 139: U27.IN_A
- new net 140: U27.IN_B
- new net 141: U28.IN_A
- new net 142: U28.IN_B
- new net 143: U29.IN_A
- new net 144: U29.IN_B
- new net 145: U30.IN_A
- new net 146: U30.IN_B
- new net 147: U31.IN_A
- new net 148: U31.IN_B
- new net 149: U32.IN_A
- new net 150: U32.IN_B
- new net 151: U33.IN_A
- new net 152: U33.IN_B
- new net 153: U34.IN_A
- new net 154: U34.IN_B
- new net 155: U35.IN_A
- new net 156: U35.IN_B
- new net 157: U36.IN_A
- new net 158: U36.IN_B
- new net 159: U37.IN_A
- new net 160: U37.IN_B
- new net 161: U38.IN_A
- new net 162: U38.IN_B
- new net 163: U39.IN_A
- new net 164: U39.IN_B
- new net 165: U40.IN_A
- new net 166: U40.IN_B
- new net 167: U41.IN_A
- new net 168: U41.IN_B
- new net 169: U42.IN_A
- new net 170: U42.IN_B
- new net 171: U43.IN_A
- new net 172: U43.IN_B
- new net 173: U44.IN_A
- new net 174: U44.IN_B
- new net 175: U45.IN_A
- new net 176: U45.IN_B
- new net 2: U1.IN_B
- new net 89: U2.IN_A
- new net 90: U2.IN_B
- new net 91: U3.IN_A, U46.IN_A
- new net 92: U3.IN_B, U46.IN_B
- new net 93: U4.IN_A, U47.IN_A
- new net 94: U4.IN_B, U47.IN_B
- new net 95: U48.IN_A, U5.IN_A
- new net 96: U48.IN_B, U5.IN_B
- new net 97: U49.IN_A, U6.IN_A
- new net 98: U49.IN_B, U6.IN_B
- new net 99: U50.IN_A, U7.IN_A
- new net DRIVE_1: U1.*OUT_B
- new net DRIVE_10: U10.*OUT_B
- new net DRIVE_11: U11.*OUT_B
- new net DRIVE_12: U12.*OUT_B
- new net DRIVE_13: U13.*OUT_B
- new net DRIVE_14: U14.*OUT_B
- new net DRIVE_15: U15.*OUT_B
- new net DRIVE_16: U16.*OUT_B
- new net DRIVE_17: U17.*OUT_B
- new net DRIVE_18: U18.*OUT_B
- new net DRIVE_19: U19.*OUT_B
- new net DRIVE_2: U2.*OUT_B
- new net DRIVE_20: U20.*OUT_B
- new net DRIVE_21: U21.*OUT_B
- new net DRIVE_22: U22.*OUT_B
- new net DRIVE_23: U23.*OUT_B
- new net DRIVE_24: U24.*OUT_B
- new net DRIVE_25: U25.*OUT_B
- new net DRIVE_26: U26.*OUT_B
- new net DRIVE_27: U27.*OUT_B
- new net DRIVE_28: U28.*OUT_B
- new net DRIVE_29: U29.*OUT_B
- new net DRIVE_3: U3.*OUT_B
- new net DRIVE_30: U30.*OUT_B
- new net DRIVE_31: U31.*OUT_B
- new net DRIVE_32: U32.*OUT_B
- new net DRIVE_33: U33.*OUT_B
- new net DRIVE_34: U34.*OUT_B
- new net DRIVE_35: U35.*OUT_B
- new net DRIVE_36: U36.*OUT_B
- new net DRIVE_37: U37.*OUT_B
- new net DRIVE_38: U38.*OUT_B
- new net DRIVE_39: U39.*OUT_B
- new net DRIVE_4: U4.*OUT_B
- new net DRIVE_40: U40.*OUT_B
- new net DRIVE_41: U41.*OUT_B
- new net DRIVE_42: U42.*OUT_B
- new net DRIVE_43: U43.*OUT_B
- new net DRIVE_44: U44.*OUT_B
- new net DRIVE_45: U45.*OUT_B
- new net DRIVE_5: U5.*OUT_B
- new net DRIVE_6: U6.*OUT_B
- new net DRIVE_7: U7.*OUT_B
- new net DRIVE_8: U8.*OUT_B
- new net DRIVE_9: U9.*OUT_B
- new net N$130: U1.*OUT_A
- new net N$15: U7.*OUT_A
- new net N$16: U8.*OUT_A
- new net N$17: U9.*OUT_A
- new net N$18: U10.*OUT_A
- new net N$19: U11.*OUT_A
- new net N$20: U12.*OUT_A
- new net N$21: U13.*OUT_A
- new net N$22: U14.*OUT_A
- new net N$23: U15.*OUT_A
- new net N$24: U16.*OUT_A
- new net N$25: U17.*OUT_A
- new net N$26: U18.*OUT_A
- new net N$27: U19.*OUT_A
- new net N$28: U20.*OUT_A
- new net N$29: U21.*OUT_A
- new net N$39: U22.*OUT_A
- new net N$4: U2.*OUT_A
- new net N$40: U23.*OUT_A
- new net N$41: U24.*OUT_A
- new net N$42: U25.*OUT_A
- new net N$43: U26.*OUT_A
- new net N$44: U27.*OUT_A
- new net N$45: U28.*OUT_A
- new net N$46: U29.*OUT_A
- new net N$47: U30.*OUT_A
- new net N$48: U31.*OUT_A
- new net N$49: U32.*OUT_A
- new net N$50: U33.*OUT_A
- new net N$51: U34.*OUT_A
- new net N$52: U35.*OUT_A
- new net N$53: U36.*OUT_A
- new net N$54: U37.*OUT_A
- new net N$55: U38.*OUT_A
- new net N$56: U39.*OUT_A
- new net N$57: U40.*OUT_A
- new net N$58: U41.*OUT_A
- new net N$59: U42.*OUT_A
- new net N$6: U3.*OUT_A
- new net N$60: U43.*OUT_A
- new net N$61: U44.*OUT_A
- new net N$62: U45.*OUT_A
- new net N$8: U4.*OUT_A
- new net N$9: U5.*OUT_A
- new net TO_TRAN_100: JP1.2, U50.*OUT_B
- new net TO_TRAN_85: JP1.32
- new net TO_TRAN_86: JP1.30
- new net TO_TRAN_87: JP1.28
- new net TO_TRAN_88: JP1.26
- new net TO_TRAN_89: JP1.24
- new net TO_TRAN_90: JP1.22
- new net TO_TRAN_91: JP1.20, U46.*OUT_A
- new net TO_TRAN_92: JP1.18, U46.*OUT_B
- new net TO_TRAN_93: JP1.16, U47.*OUT_A
- new net TO_TRAN_94: JP1.14, U47.*OUT_B
- new net TO_TRAN_95: JP1.12, U48.*OUT_A
- new net TO_TRAN_96: JP1.10, U48.*OUT_B
- new net TO_TRAN_97: JP1.8, U49.*OUT_A
- new net TO_TRAN_98: JP1.6, U49.*OUT_B
- new net TO_TRAN_99: JP1.4, U50.*OUT_A
- new net TRANSIVER_DRIVE_1: U900.IN_A
- new net TRANSIVER_DRIVE_2: U900.IN_B
- new net VDD: 5V-REG.IN, C1.2, C10.2, C11.2, C12.2, C13.2, C14.2, C15.2, C16.2, C17.2, C18.2, C19.2, C2.2, C20.2, C21.2, C22.2, C23.2, C24.2, C25.2, C26.2, C27.2, C28.2, C29.2, C3.2, C30.2, C31.2, C32.2, C33.2, C34.2, C35.2, C36.2, C37.2, C38.2, C39.2, C4.2, C40.2, C41.2, C42.2, C43.2, C44.2, C45.2, C46.2, C47.2, C48.2, C49.2, C5.2, C50.2, C6.2, C7.2, C8.2, C9.2, C90.2, IC2.VI, J1.1, REFULATOR_TANTALUM.1, U1.VDD, U10.VDD, U11.VDD, U12.VDD, U13.VDD, U14.VDD, U15.VDD, U16.VDD, U17.VDD, U18.VDD, U19.VDD, U2.VDD, U20.VDD, U21.VDD, U22.VDD, U23.VDD, U24.VDD, U25.VDD, U26.VDD, U27.VDD, U28.VDD, U29.VDD, U3.VDD, U30.VDD, U31.VDD, U32.VDD, U33.VDD, U34.VDD, U35.VDD, U36.VDD, U37.VDD, U38.VDD, U39.VDD, U4.VDD, U40.VDD, U41.VDD, U42.VDD, U43.VDD, U44.VDD, U45.VDD, U46.VDD, U47.VDD, U48.VDD, U49.VDD, U5.VDD, U50.VDD, U6.VDD, U7.VDD, U8.VDD, U9.VDD, U900.VDD
- net GND: now also 5V-REG.GND, C1.1, C10.1, C11.1, C12.1, C13.1, C14.1, C15.1, C16.1, C17.1, C18.1, C19.1, C2.1, C20.1, C21.1, C22.1, C23.1, C24.1, C25.1, C26.1, C27.1, C28.1, C29.1, C3.1, C30.1, C31.1, C32.1, C33.1, C34.1, C35.1, C36.1, C37.1, C38.1, C39.1, C4.1, C40.1, C41.1, C42.1, C43.1, C44.1, C45.1, C46.1, C47.1, C48.1, C49.1, C5.1, C50.1, C6.1, C7.1, C8.1, C9.1, C90.1, C905.2, DATA.11, DIP2.GND@1, DIP2.GND@2, DIP2.GND@3, DIP2.GND@4, IC2.GND, J1.2, Q2.S, R11.1, R12.1, R5.2, R9.2, REFULATOR_TANTALUM.2, U1.GND, U10.GND, U11.GND, U12.GND, U1200.GND, U13.GND, U14.GND, U15.GND, U16.GND, U17.GND, U18.GND, U19.GND, U2.GND, U20.GND, U200.V-, U21.GND, U22.GND, U23.GND, U24.GND, U25.GND, U26.GND, U27.GND, U28.GND, U29.GND, U3.GND, U30.GND, U31.GND, U32.GND, U33.GND, U34.GND, U35.GND, U36.GND, U37.GND, U38.GND, U39.GND, U4.GND, U40.GND, U41.GND, U42.GND, U43.GND, U44.GND, U45.GND, U46.GND, U47.GND, U48.GND, U49.GND, U5.GND, U50.GND, U6.GND, U7.GND, U8.GND, U9.GND, U900.GND
- net N$1: now also U1200.I0; no longer U1.S0
- net N$12: no longer SL1.7
- net N$13: now also U6.*OUT_A; no longer U$1.36/A17, U35.IN_B
- net N$14: now also U200.INA-; no longer U2.INA-
- net N$3: now also U1200.COMMON_IN/OUT, U200.INA+; no longer U1.COMMON_IN/OUT, U2.INA+
- net N$7: now also U200.OUTA; no longer U2.OUTA
- net N$72: now also U900.*OUT_B; no longer SL1.8, U35.*OUT_B
Other:
- moved on the sheet: C35, C5, J1, R6, U2, U35

Commit message: Niall's board work
Parts:
- removed C90: 100nF, resistor:C-EUC0805
- removed Q2: 2N7002, SnapEDA-Library:2N7002
- removed R12: 1M, resistor:R-US_M0805
- removed R13: 100, resistor:R-US_M0805
- removed R14: 10k, resistor:R-US_M0805
- removed R6: 100K, resistor:R-US_M0805
- removed U900: TC4427AEOA, Parts:TC4427AEOA
- added NPN_1, NPN_10, NPN_11, NPN_12, NPN_13, NPN_14, NPN_15, NPN_16, NPN_2, NPN_3, NPN_4, NPN_5, NPN_6, NPN_7, NPN_8, NPN_9: 2N7002, SnapEDA-Library:2N7002
- added PROTECT_R_1, PROTECT_R_10, PROTECT_R_11, PROTECT_R_12, PROTECT_R_13, PROTECT_R_14, PROTECT_R_15, PROTECT_R_16, PROTECT_R_2, PROTECT_R_3, PROTECT_R_4, PROTECT_R_5, PROTECT_R_6, PROTECT_R_7, PROTECT_R_8, PROTECT_R_9: 100K, resistor:R-US_M0805
- added R-TRANS-100, R-TRANS-85, R-TRANS-86, R-TRANS-87, R-TRANS-88, R-TRANS-89, R-TRANS-90, R-TRANS-91, R-TRANS-92, R-TRANS-93, R-TRANS-94, R-TRANS-95, R-TRANS-96, R-TRANS-97, R-TRANS-98, R-TRANS-99: 10k, resistor:R-US_M0805
- added T_S-R1.1, T_S-R10.1, T_S-R11.1, T_S-R12.1, T_S-R13.1, T_S-R14.1, T_S-R15.1, T_S-R16.1, T_S-R2.1, T_S-R3.1, T_S-R4.1, T_S-R5.1, T_S-R6.1, T_S-R7.1, T_S-R8.1, T_S-R9.1: 1M, resistor:R-US_M0805
- added T_S-R1.2, T_S-R10.2, T_S-R11.2, T_S-R12.2, T_S-R13.2, T_S-R14.2, T_S-R15.2, T_S-R16.2, T_S-R2.2, T_S-R3.2, T_S-R4.2, T_S-R5.2, T_S-R6.2, T_S-R7.2, T_S-R8.2, T_S-R9.2: 100, resistor:R-US_M0805
Connections:
- net 89 renamed 3
- net 90 renamed 4
- net DRIVE_1 renamed TO_TRAN_2
- net DRIVE_2 renamed TO_TRAN_4
- net DRIVE_3 renamed TO_TRAN_6
- net DRIVE_4 renamed TO_TRAN_8
- net N$130 renamed TO_TRAN_1
- net N$4 renamed TO_TRAN_3
- net N$6 renamed TO_TRAN_5
- net N$8 renamed TO_TRAN_7
- removed net N$72: R14.1, U900.*OUT_B
- removed net TRANSIVER_DRIVE_1: U900.IN_A
- removed net TRANSIVER_DRIVE_2: U900.IN_B
- new net 5: U3.IN_A
- new net 6: U3.IN_B
- new net 7: U4.IN_A
- new net 8: U4.IN_B
- new net FROM_TRANS_100: JP1.1, NPN_1.D, PROTECT_R_1.2, R-TRANS-100.1
- new net FROM_TRANS_85: JP1.31, NPN_16.D, PROTECT_R_16.2, R-TRANS-85.1
- new net FROM_TRANS_86: JP1.29, NPN_15.D, PROTECT_R_15.2, R-TRANS-86.1
- new net FROM_TRANS_87: JP1.27, NPN_14.D, PROTECT_R_14.2, R-TRANS-87.1
- new net FROM_TRANS_88: JP1.25, NPN_13.D, PROTECT_R_13.2, R-TRANS-88.1
- new net FROM_TRANS_89: JP1.23, NPN_12.D, PROTECT_R_12.2, R-TRANS-89.1
- new net FROM_TRANS_90: JP1.21, NPN_11.D, PROTECT_R_11.2, R-TRANS-90.1
- new net FROM_TRANS_91: JP1.19, NPN_10.D, PROTECT_R_10.2, R-TRANS-91.1
- new net FROM_TRANS_92: JP1.17, NPN_9.D, PROTECT_R_9.2, R-TRANS-92.1
- new net FROM_TRANS_93: JP1.15, NPN_8.D, PROTECT_R_8.2, R-TRANS-93.1
- new net FROM_TRANS_94: JP1.13, NPN_7.D, PROTECT_R_7.2, R-TRANS-94.1
- new net FROM_TRANS_95: JP1.11, NPN_6.D, PROTECT_R_6.2, R-TRANS-95.1
- new net FROM_TRANS_96: JP1.9, NPN_5.D, PROTECT_R_5.2, R-TRANS-96.1
- new net FROM_TRANS_97: JP1.7, NPN_4.D, PROTECT_R_4.2, R-TRANS-97.1
- new net FROM_TRANS_98: JP1.5, NPN_3.D, PROTECT_R_3.2, R-TRANS-98.1
- new net FROM_TRANS_99: JP1.3, NPN_2.D, PROTECT_R_2.2, R-TRANS-99.1
- new net N$101: NPN_16.G, T_S-R16.2.1
- new net N$3: PROTECT_R_2.1, U1200.I1
- new net N$30: U$1.38/A19, U1200.S0
- new net N$31: NPN_1.G, T_S-R1.2.1
- new net N$34: NPN_2.G, T_S-R2.2.1
- new net N$35: PROTECT_R_3.1, U1200.I2
- new net N$36: T_S-R1.1.2, T_S-R1.2.2, T_S-R10.1.2, T_S-R10.2.2, T_S-R11.1.2, T_S-R11.2.2, T_S-R12.1.2, T_S-R12.2.2, T_S-R13.1.2, T_S-R13.2.2, T_S-R14.1.2, T_S-R14.2.2, T_S-R15.1.2, T_S-R15.2.2, T_S-R16.1.2, T_S-R16.2.2, T_S-R2.1.2, T_S-R2.2.2, T_S-R3.1.2, T_S-R3.2.2, T_S-R4.1.2, T_S-R4.2.2, T_S-R5.1.2, T_S-R5.2.2, T_S-R6.1.2, T_S-R6.2.2, T_S-R7.1.2, T_S-R7.2.2, T_S-R8.1.2, T_S-R8.2.2, T_S-R9.1.2, T_S-R9.2.2, U$1.28
- new net N$37: NPN_3.G, T_S-R3.2.1
- new net N$38: PROTECT_R_4.1, U1200.I3
- new net N$64: NPN_4.G, T_S-R4.2.1
- new net N$65: PROTECT_R_5.1, U1200.I4
- new net N$67: NPN_5.G, T_S-R5.2.1
- new net N$68: PROTECT_R_6.1, U1200.I5
- new net N$70: NPN_6.G, T_S-R6.2.1
- new net N$71: PROTECT_R_7.1, U1200.I6
- new net N$74: NPN_7.G, T_S-R7.2.1
- new net N$75: PROTECT_R_8.1, U1200.I7
- new net N$77: NPN_8.G, T_S-R8.2.1
- new net N$78: PROTECT_R_9.1, U1200.I8
- new net N$80: NPN_9.G, T_S-R9.2.1
- new net N$81: PROTECT_R_10.1, U1200.I9
- new net N$83: NPN_10.G, T_S-R10.2.1
- new net N$84: PROTECT_R_11.1, U1200.I10
- new net N$86: NPN_11.G, T_S-R11.2.1
- new net N$87: PROTECT_R_12.1, U1200.I11
- new net N$89: NPN_12.G, T_S-R12.2.1
- new net N$90: PROTECT_R_13.1, U1200.I12
- new net N$92: NPN_13.G, T_S-R13.2.1
- new net N$93: PROTECT_R_14.1, U1200.I13
- new net N$95: NPN_14.G, T_S-R14.2.1
- new net N$96: PROTECT_R_15.1, U1200.I14
- new net N$98: NPN_15.G, T_S-R15.2.1
- new net N$99: PROTECT_R_16.1, U1200.I15
- net +5V: now also U1200.VCC
- net 91: no longer U3.IN_A
- net 92: no longer U3.IN_B
- net 93: no longer U4.IN_A
- net 94: no longer U4.IN_B
- net GND: now also NPN_1.S, NPN_10.S, NPN_11.S, NPN_12.S, NPN_13.S, NPN_14.S, NPN_15.S, NPN_16.S, NPN_2.S, NPN_3.S, NPN_4.S, NPN_5.S, NPN_6.S, NPN_7.S, NPN_8.S, NPN_9.S, T_S-R1.1.1, T_S-R10.1.1, T_S-R11.1.1, T_S-R12.1.1, T_S-R13.1.1, T_S-R14.1.1, T_S-R15.1.1, T_S-R16.1.1, T_S-R2.1.1, T_S-R3.1.1, T_S-R4.1.1, T_S-R5.1.1, T_S-R6.1.1, T_S-R7.1.1, T_S-R8.1.1, T_S-R9.1.1, U1200.~E; no longer C90.1, Q2.S, R12.1, U900.GND
- net N$1: now also PROTECT_R_1.1; no longer R6.1
- net N$10: now also U1200.S3; no longer R12.2, R13.2
- net N$11: now also U$1.36/A17, U1200.S2; no longer Q2.G, R13.1
- net N$12: now also U$1.37/A18, U1200.S1; no longer Q2.D, R14.2, R6.2
- net TO_TRAN_100: now also R-TRANS-100.2
- net TO_TRAN_85: now also R-TRANS-85.2
- net TO_TRAN_86: now also R-TRANS-86.2
- net TO_TRAN_87: now also R-TRANS-87.2
- net TO_TRAN_88: now also R-TRANS-88.2
- net TO_TRAN_89: now also R-TRANS-89.2
- net TO_TRAN_90: now also R-TRANS-90.2
- net TO_TRAN_91: now also R-TRANS-91.2
- net TO_TRAN_92: now also R-TRANS-92.2
- net TO_TRAN_93: now also R-TRANS-93.2
- net TO_TRAN_94: now also R-TRANS-94.2
- net TO_TRAN_95: now also R-TRANS-95.2
- net TO_TRAN_96: now also R-TRANS-96.2
- net TO_TRAN_97: now also R-TRANS-97.2
- net TO_TRAN_98: now also R-TRANS-98.2
- net TO_TRAN_99: now also R-TRANS-99.2
- net VDD: no longer C90.2, U900.VDD
Other:
- note added: "5 Volt regulator"
- moved on the sheet: 5V-REG, JP1, JP2, JP3, R11, U1200

Commit message: Niall board update
Parts:
- added DATA1: Data, SparkFun-Connectors:CONN_11
Changed lines of the file:
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@@
 <part name="SUPPLY11" library="supply1" library_urn="urn:adsk.eagle:library:371" deviceset="GND" device=""/>
 <part name="SUPPLY82" library="supply2" library_urn="urn:adsk.eagle:library:372" deviceset="+5V" device=""/>
+<part name="DATA1" library="SparkFun-Connectors" library_urn="urn:adsk.eagle:library:513" deviceset="CONN_11" device="" package3d_urn="urn:adsk.eagle:package:38251/1" value="Data"/>
 </parts>
 <sheets>
@@
 <instance part="SUPPLY11" gate="1" x="-30.48" y="27.94" rot="R270"/>
 <instance part="SUPPLY82" gate="+5V" x="-30.48" y="33.02" rot="R90"/>
+<instance part="DATA1" gate="G$1" x="-27.94" y="497.84" rot="R270"/>
 </instances>
 <busses>

Commit message: Niall board edits
Connections:
- net 101 renamed 15
- net 102 renamed 16
- net 103 renamed 17
- net 104 renamed 18
- net 105 renamed 19
- net 106 renamed 20
- net 107 renamed 21
- net 108 renamed 22
- net 109 renamed 23
- net 110 renamed 24
- net 111 renamed 25
- net 112 renamed 26
- net 113 renamed 27
- net 114 renamed 28
- net 115 renamed 29
- net 116 renamed 30
- net 117 renamed 31
- net 118 renamed 32
- net 119 renamed 33
- net 120 renamed 34
- net 121 renamed 35
- net 122 renamed 36
- net 123 renamed 37
- net 124 renamed 38
- net 125 renamed 40
- net 126 renamed 39
- net 127 renamed 41
- net 128 renamed 42
- net 129 renamed 43
- net 130 renamed 44
- net 131 renamed 45
- net 132 renamed 46
- net DRIVE_10 renamed TO_TRAN_20
- net DRIVE_11 renamed TO_TRAN_22
- net DRIVE_12 renamed TO_TRAN_24
- net DRIVE_13 renamed TO_TRAN_26
- net DRIVE_14 renamed TO_TRAN_28
- net DRIVE_15 renamed TO_TRAN_30
- net DRIVE_16 renamed TO_TRAN_32
- net DRIVE_17 renamed TO_TRAN_34
- net DRIVE_18 renamed TO_TRAN_36
- net DRIVE_19 renamed TO_TRAN_38
- net DRIVE_20 renamed TO_TRAN_39
- net DRIVE_21 renamed TO_TRAN_42
- net DRIVE_22 renamed TO_TRAN_44
- net DRIVE_23 renamed TO_TRAN_46
- net DRIVE_5 renamed TO_TRAN_10
- net DRIVE_6 renamed TO_TRAN_12
- net DRIVE_7 renamed TO_TRAN_14
- net DRIVE_8 renamed TO_TRAN_16
- net DRIVE_9 renamed TO_TRAN_18
- net N$13 renamed TO_TRAN_11
- net N$15 renamed TO_TRAN_13
- net N$16 renamed TO_TRAN_15
- net N$17 renamed TO_TRAN_17
- net N$18 renamed TO_TRAN_19
- net N$19 renamed TO_TRAN_21
- net N$20 renamed TO_TRAN_23
- net N$21 renamed TO_TRAN_25
- net N$22 renamed TO_TRAN_27
- net N$23 renamed TO_TRAN_29
- net N$24 renamed TO_TRAN_31
- net N$25 renamed TO_TRAN_33
- net N$26 renamed TO_TRAN_35
- net N$27 renamed TO_TRAN_37
- net N$28 renamed TO_TRAN_40
- net N$29 renamed TO_TRAN_41
- net N$39 renamed TO_TRAN_43
- net N$40 renamed TO_TRAN_45
- net N$9 renamed TO_TRAN_9
- new net 10: U5.IN_B
- new net 11: U6.IN_A
- new net 12: U6.IN_B
- new net 13: U7.IN_A
- new net 14: U7.IN_B
- new net 9: U5.IN_A
- net 100: no longer U7.IN_B
- net 95: no longer U5.IN_A
- net 96: no longer U5.IN_B
- net 97: no longer U6.IN_A
- net 98: no longer U6.IN_B
- net 99: no longer U7.IN_A

Commit message: Niall's amazing masterpeice
Parts:
- removed T_S-R1.1, T_S-R2.1: 1M, resistor:R-US_M0805
- removed T_S-R1.2, T_S-R2.2: 100, resistor:R-US_M0805
- added R_PROTECT: 100, resistor:R-US_M0805
- added R_TO_GND: 1M, resistor:R-US_M0805
Connections:
- removed net N$36: T_S-R1.1.2, T_S-R1.2.2, T_S-R10.1.2, T_S-R10.2.2, T_S-R11.1.2, T_S-R11.2.2, T_S-R12.1.2, T_S-R12.2.2, T_S-R13.1.2, T_S-R13.2.2, T_S-R14.1.2, T_S-R14.2.2, T_S-R15.1.2, T_S-R15.2.2, T_S-R16.1.2, T_S-R16.2.2, T_S-R2.1.2, T_S-R2.2.2, T_S-R3.1.2, T_S-R3.2.2, T_S-R4.1.2, T_S-R4.2.2, T_S-R5.1.2, T_S-R5.2.2, T_S-R6.1.2, T_S-R6.2.2, T_S-R7.1.2, T_S-R7.2.2, T_S-R8.1.2, T_S-R8.2.2, T_S-R9.1.2, T_S-R9.2.2, U$1.28
- new net N$8: R_PROTECT.1, U$1.28
- new net N$9: R_PROTECT.2, R_TO_GND.2, T_S-R10.1.2, T_S-R10.2.2, T_S-R11.1.2, T_S-R11.2.2, T_S-R12.1.2, T_S-R12.2.2, T_S-R13.1.2, T_S-R13.2.2, T_S-R14.1.2, T_S-R14.2.2, T_S-R15.1.2, T_S-R15.2.2, T_S-R16.1.2, T_S-R16.2.2, T_S-R3.1.2, T_S-R3.2.2, T_S-R4.1.2, T_S-R4.2.2, T_S-R5.1.2, T_S-R5.2.2, T_S-R6.1.2, T_S-R6.2.2, T_S-R7.1.2, T_S-R7.2.2, T_S-R8.1.2, T_S-R8.2.2, T_S-R9.1.2, T_S-R9.2.2
- net +5V: now also U$1.VIN
- net GND: now also R_TO_GND.1; no longer T_S-R1.1.1, T_S-R2.1.1
- net N$10: now also U$1.37/A18; no longer U$1.35/A16
- net N$11: now also U$1.35/A16; no longer U$1.36/A17
- net N$12: now also U$1.36/A17; no longer U$1.37/A18
- net N$31: no longer T_S-R1.2.1
- net N$34: no longer T_S-R2.2.1
- net N$5: now also U$1.39/A20; no longer U$1.23/A9
