File: eagle/ProjectX/Driver_Board_Niall.sch (EAGLE design)
At the start: 199 parts, among them IC2 NCV78M05BDTRKG, J1 694102303002, U1 TC4427AEOA, U10 TC4427AEOA, U11 TC4427AEOA, U12 TC4427AEOA, U1200 CD74HC4067SM96, U13 TC4427AEOA, U14 TC4427AEOA, U15 TC4427AEOA, U16 TC4427AEOA, U17 TC4427AEOA, U18 TC4427AEOA, U19 TC4427AEOA, U2 TC4427AEOA, U20 TC4427AEOA, U200 ADA4091-2ARZ-RL, U21 TC4427AEOA, U22 TC4427AEOA, U23 TC4427AEOA, U24 TC4427AEOA, U25 TC4427AEOA, U26 TC4427AEOA, U27 TC4427AEOA, U28 TC4427AEOA, U29 TC4427AEOA, U3 TC4427AEOA, U30 TC4427AEOA, U31 TC4427AEOA, U32 TC4427AEOA, U33 TC4427AEOA, U34 TC4427AEOA, U35 TC4427AEOA, U36 TC4427AEOA, U37 TC4427AEOA, U38 TC4427AEOA, U39 TC4427AEOA, U4 TC4427AEOA, U40 TC4427AEOA, U41 TC4427AEOA, U42 TC4427AEOA, U43 TC4427AEOA, U44 TC4427AEOA, U45 TC4427AEOA, U46 TC4427AEOA, U47 TC4427AEOA, U48 TC4427AEOA, U49 TC4427AEOA, U5 TC4427AEOA, U50 TC4427AEOA, U6 TC4427AEOA, U7 TC4427AEOA, U8 TC4427AEOA, U9 TC4427AEOA

Commit message: Niall board edits
Parts:
- removed JP2, JP3: (no value), pinhead:PINHD-2X20
- removed T_S-R10.1, T_S-R11.1, T_S-R12.1, T_S-R13.1, T_S-R14.1, T_S-R15.1, T_S-R16.1, T_S-R3.1, T_S-R4.1, T_S-R5.1, T_S-R6.1, T_S-R7.1, T_S-R8.1, T_S-R9.1: 1M, resistor:R-US_M0805
- removed T_S-R10.2, T_S-R11.2, T_S-R12.2, T_S-R13.2, T_S-R14.2, T_S-R15.2, T_S-R16.2, T_S-R3.2, T_S-R4.2, T_S-R5.2, T_S-R6.2, T_S-R7.2, T_S-R8.2, T_S-R9.2: 100, resistor:R-US_M0805
- added U$2, U$3, U$4, U$5: 40_PIN_SMD, Parts:40_PIN_SMD
Connections:
- removed net N$101: NPN_16.G, T_S-R16.2.1
- removed net N$31: NPN_1.G
- removed net N$37: NPN_3.G, T_S-R3.2.1
- removed net N$64: NPN_4.G, T_S-R4.2.1
- removed net N$67: NPN_5.G, T_S-R5.2.1
- removed net N$70: NPN_6.G, T_S-R6.2.1
- removed net N$74: NPN_7.G, T_S-R7.2.1
- removed net N$77: NPN_8.G, T_S-R8.2.1
- removed net N$80: NPN_9.G, T_S-R9.2.1
- removed net N$83: NPN_10.G, T_S-R10.2.1
- removed net N$86: NPN_11.G, T_S-R11.2.1
- removed net N$89: NPN_12.G, T_S-R12.2.1
- removed net N$9: R_PROTECT.2, R_TO_GND.2, T_S-R10.1.2, T_S-R10.2.2, T_S-R11.1.2, T_S-R11.2.2, T_S-R12.1.2, T_S-R12.2.2, T_S-R13.1.2, T_S-R13.2.2, T_S-R14.1.2, T_S-R14.2.2, T_S-R15.1.2, T_S-R15.2.2, T_S-R16.1.2, T_S-R16.2.2, T_S-R3.1.2, T_S-R3.2.2, T_S-R4.1.2, T_S-R4.2.2, T_S-R5.1.2, T_S-R5.2.2, T_S-R6.1.2, T_S-R6.2.2, T_S-R7.1.2, T_S-R7.2.2, T_S-R8.1.2, T_S-R8.2.2, T_S-R9.1.2, T_S-R9.2.2
- removed net N$92: NPN_13.G, T_S-R13.2.1
- removed net N$95: NPN_14.G, T_S-R14.2.1
- removed net N$98: NPN_15.G, T_S-R15.2.1
- net GND: no longer T_S-R10.1.1, T_S-R11.1.1, T_S-R12.1.1, T_S-R13.1.1, T_S-R14.1.1, T_S-R15.1.1, T_S-R16.1.1, T_S-R3.1.1, T_S-R4.1.1, T_S-R5.1.1, T_S-R6.1.1, T_S-R7.1.1, T_S-R8.1.1, T_S-R9.1.1
- net N$34: now also NPN_1.G, NPN_10.G, NPN_11.G, NPN_12.G, NPN_13.G, NPN_14.G, NPN_15.G, NPN_16.G, NPN_3.G, NPN_4.G, NPN_5.G, NPN_6.G, NPN_7.G, NPN_8.G, NPN_9.G, R_PROTECT.2, R_TO_GND.2
Other:
- moved on the sheet: R_PROTECT, R_TO_GND
