File: eagle/ProjectX/Driver_Board_Niall.sch (EAGLE design)
At the start: 183 parts, among them IC2 NCV78M05BDTRKG, J1 694102303002, J2 694102303002, U1 TC4427AEOA, U10 TC4427AEOA, U11 TC4427AEOA, U12 TC4427AEOA, U1200 CD74HC4067SM96, U13 TC4427AEOA, U14 TC4427AEOA, U15 TC4427AEOA, U16 TC4427AEOA, U17 TC4427AEOA, U18 TC4427AEOA, U19 TC4427AEOA, U2 TC4427AEOA, U20 TC4427AEOA, U200 ADA4091-2ARZ-RL, U21 TC4427AEOA, U22 TC4427AEOA, U23 TC4427AEOA, U24 TC4427AEOA, U25 TC4427AEOA, U26 TC4427AEOA, U27 TC4427AEOA, U28 TC4427AEOA, U29 TC4427AEOA, U3 TC4427AEOA, U30 TC4427AEOA, U31 TC4427AEOA, U32 TC4427AEOA, U33 TC4427AEOA, U34 TC4427AEOA, U35 TC4427AEOA, U36 TC4427AEOA, U37 TC4427AEOA, U38 TC4427AEOA, U39 TC4427AEOA, U4 TC4427AEOA, U40 TC4427AEOA, U41 TC4427AEOA, U42 TC4427AEOA, U43 TC4427AEOA, U44 TC4427AEOA, U45 TC4427AEOA, U46 TC4427AEOA, U47 TC4427AEOA, U48 TC4427AEOA, U49 TC4427AEOA, U5 TC4427AEOA, U50 TC4427AEOA, U6 TC4427AEOA, U7 TC4427AEOA, U8 TC4427AEOA, U9 TC4427AEOA

Commit message: Niall almost done
Parts:
- added TP1, TP10, TP11, TP12, TP13, TP14, TP15, TP16, TP17, TP18, TP19, TP2, TP20, TP3, TP4, TP5, TP6, TP7, TP8, TP9: TPSQPAD1-13Y, testpad:TPSQPAD1-13Y
Connections:
- new net N$13: TP2.TP, U$1.23/A9
- new net N$15: TP3.TP, U$1.22/A8
- new net N$16: TP4.TP, U$1.21/A7
- new net N$17: TP5.TP, U$1.20/A6
- new net N$18: TP6.TP, U$1.19/A5/SCL
- new net N$19: TP7.TP, U$1.17/A3
- new net N$20: TP8.TP, U$1.18/A4/SDA
- new net N$21: TP9.TP, U$1.16/A2
- new net N$22: TP10.TP, U$1.15/A1
- new net N$26: TP11.TP, U$1.14/A0
- new net N$27: TP12.TP, U$1.13/SCK
- new net N$28: TP13.TP, U$1.GND2
- new net N$29: TP14.TP, U$1.A22/DAC1
- new net N$30: TP15.TP, U$1.A21/DAC0
- new net N$31: TP16.TP, U$1.3V3
- new net N$33: TP17.TP, U$1.AGND
- new net N$9: TP1.TP, U$1.3V3_LO
- net +5V: now also TP18.TP
- net GND: now also TP19.TP
- net VDD: now also TP20.TP
Changed lines of the file:
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@@
 <part name="SUPPLY170" library="supply2" library_urn="urn:adsk.eagle:library:372" deviceset="+5V" device=""/>
 <part name="SUPPLY171" library="supply2" library_urn="urn:adsk.eagle:library:372" deviceset="+5V" device=""/>
+<part name="TP1" library="testpad" library_urn="urn:adsk.eagle:library:385" deviceset="TPSQ" device="PAD1-13Y" package3d_urn="urn:adsk.eagle:package:27947/1"/>
+<part name="TP2" library="testpad" library_urn="urn:adsk.eagle:library:385" deviceset="TPSQ" device="PAD1-13Y" package3d_urn="urn:adsk.eagle:package:27947/1"/>
+<part name="TP3" library="testpad" library_urn="urn:adsk.eagle:library:385" deviceset="TPSQ" device="PAD1-13Y" package3d_urn="urn:adsk.eagle:package:27947/1"/>
+<part name="TP4" library="testpad" library_urn="urn:adsk.eagle:library:385" deviceset="TPSQ" device="PAD1-13Y" package3d_urn="urn:adsk.eagle:package:27947/1"/>
+<part name="TP5" library="testpad" library_urn="urn:adsk.eagle:library:385" deviceset="TPSQ" device="PAD1-13Y" package3d_urn="urn:adsk.eagle:package:27947/1"/>
+<part name="TP6" library="testpad" library_urn="urn:adsk.eagle:library:385" deviceset="TPSQ" device="PAD1-13Y" package3d_urn="urn:adsk.eagle:package:27947/1"/>
+<part name="TP7" library="testpad" library_urn="urn:adsk.eagle:library:385" deviceset="TPSQ" device="PAD1-13Y" package3d_urn="urn:adsk.eagle:package:27947/1"/>
+<part name="TP8" library="testpad" library_urn="urn:adsk.eagle:library:385" deviceset="TPSQ" device="PAD1-13Y" package3d_urn="urn:adsk.eagle:package:27947/1"/>
+<part name="TP9" library="testpad" library_urn="urn:adsk.eagle:library:385" deviceset="TPSQ" device="PAD1-13Y" package3d_urn="urn:adsk.eagle:package:27947/1"/>
+<part name="TP10" library="testpad" library_urn="urn:adsk.eagle:library:385" deviceset="TPSQ" device="PAD1-13Y" package3d_urn="urn:adsk.eagle:package:27947/1"/>
+<part name="TP11" library="testpad" library_urn="urn:adsk.eagle:library:385" deviceset="TPSQ" device="PAD1-13Y" package3d_urn="urn:adsk.eagle:package:27947/1"/>
+<part name="TP12" library="testpad" library_urn="urn:adsk.eagle:library:385" deviceset="TPSQ" device="PAD1-13Y" package3d_urn="urn:adsk.eagle:package:27947/1"/>
+<part name="TP13" library="testpad" library_urn="urn:adsk.eagle:library:385" deviceset="TPSQ" device="PAD1-13Y" package3d_urn="urn:adsk.eagle:package:27947/1"/>
+<part name="TP14" library="testpad" library_urn="urn:adsk.eagle:library:385" deviceset="TPSQ" device="PAD1-13Y" package3d_urn="urn:adsk.eagle:package:27947/1"/>
+<part name="TP15" library="testpad" library_urn="urn:adsk.eagle:library:385" deviceset="TPSQ" device="PAD1-13Y" package3d_urn="urn:adsk.eagle:package:27947/1"/>
+<part name="TP16" library="testpad" library_urn="urn:adsk.eagle:library:385" deviceset="TPSQ" device="PAD1-13Y" package3d_urn="urn:adsk.eagle:package:27947/1"/>
+<part name="TP17" library="testpad" library_urn="urn:adsk.eagle:library:385" deviceset="TPSQ" device="PAD1-13Y" package3d_urn="urn:adsk.eagle:package:27947/1"/>
+<part name="TP18" library="testpad" library_urn="urn:adsk.eagle:library:385" deviceset="TPSQ" device="PAD1-13Y" package3d_urn="urn:adsk.eagle:package:27947/1"/>
+<part name="TP19" library="testpad" library_urn="urn:adsk.eagle:library:385" deviceset="TPSQ" device="PAD1-13Y" package3d_urn="urn:adsk.eagle:package:27947/1"/>
+<part name="SUPPLY172" library="supply1" library_urn="urn:adsk.eagle:library:371" deviceset="GND" device=""/>
+<part name="SUPPLY173" library="supply2" library_urn="urn:adsk.eagle:library:372" deviceset="+5V" device=""/>
+<part name="TP20" library="testpad" library_urn="urn:adsk.eagle:library:385" deviceset="TPSQ" device="PAD1-13Y" package3d_urn="urn:adsk.eagle:package:27947/1"/>
+<part name="SUPPLY174" library="SparkFun-PowerSymbols" library_urn="urn:adsk.eagle:library:530" deviceset="VDD" device=""/>
 </parts>
 <sheets>
@@
 <attribute name="VALUE" x="-14.605" y="546.735" size="1.778" layer="96"/>
 </instance>
+<instance part="TP1" gate="G$1" x="17.78" y="127" rot="R90"/>
+<instance part="TP2" gate="G$1" x="17.78" y="124.46" rot="R90"/>
+<instance part="TP3" gate="G$1" x="17.78" y="121.92" rot="R90"/>
+<instance part="TP4" gate="G$1" x="17.78" y="119.38" rot="R90"/>
+<instance part="TP5" gate="G$1" x="17.78" y="116.84" rot="R90"/>
+<instance part="TP6" gate="G$1" x="17.78" y="114.3" rot="R90"/>
+<instance part="TP7" gate="G$1" x="17.78" y="109.22" rot="R90"/>
+<instance part="TP8" gate="G$1" x="17.78" y="111.76" rot="R90"/>
+<instance part="TP9" gate="G$1" x="17.78" y="106.68" rot="R90"/>
+<instance part="TP10" gate="G$1" x="17.78" y="104.14" rot="R90"/>
+<instance part="TP11" gate="G$1" x="17.78" y="101.6" rot="R90"/>
+<instance part="TP12" gate="G$1" x="17.78" y="99.06" rot="R90"/>
+<instance part="TP13" gate="G$1" x="17.78" y="96.52" rot="R90"/>
+<instance part="TP14" gate="G$1" x="17.78" y="93.98" rot="R90"/>
+<instance part="TP15" gate="G$1" x="17.78" y="91.44" rot="R90"/>
+<instance part="TP16" gate="G$1" x="-27.94" y="96.52" rot="R270"/>
+<instance part="TP17" gate="G$1" x="17.78" y="129.54" rot="R90"/>
+<instance part="TP18" gate="G$1" x="27.94" y="116.84" rot="R180"/>
+<instance part="TP19" gate="G$1" x="33.02" y="116.84" rot="R180"/>
+<instance part="SUPPLY172" gate="1" x="33.02" y="111.76">
+<attribute name="VALUE" x="30.48" y="109.22" size="1.778" layer="96"/>
+</instance>
+<instance part="SUPPLY173" gate="+5V" x="27.94" y="111.76" rot="R180">
+<attribute name="VALUE" x="29.845" y="108.585" size="1.778" layer="96" rot="R180"/>
+</instance>
+<instance part="TP20" gate="G$1" x="38.1" y="116.84" rot="R180"/>
+<instance part="SUPPLY174" gate="VDD" x="38.1" y="114.3" rot="R180">
+<attribute name="VALUE" x="38.1" y="111.506" size="1.778" layer="96" rot="R180" align="bottom-center"/>
+</instance>
 </instances>
 <busses>
@@
 <wire x1="-83.82" y1="505.968" x2="-83.82" y2="506.222" width="0.1524" layer="91"/>
 </segment>
+<segment>
+<pinref part="TP19" gate="G$1" pin="TP"/>
+<pinref part="SUPPLY172" gate="1" pin="GND"/>
+</segment>
 </net>
 <net name="N$5" class="0">
@@
 <pinref part="SUPPLY171" gate="+5V" pin="+5V"/>
 </segment>
+<segment>
+<pinref part="TP18" gate="G$1" pin="TP"/>
+<pinref part="SUPPLY173" gate="+5V" pin="+5V"/>
+</segment>
 </net>
 <net name="VDD" class="0">
@@
 <pinref part="SUPPLY51" gate="VDD" pin="VDD"/>
 </segment>
+<segment>
+<pinref part="TP20" gate="G$1" pin="TP"/>
+<pinref part="SUPPLY174" gate="VDD" pin="VDD"/>
+</segment>
 </net>
 <net name="2" class="0">
@@
 </segment>
 </net>
+<net name="N$9" class="0">
+<segment>
+<pinref part="U$1" gate="G$1" pin="3V3_LO"/>
+<pinref part="TP1" gate="G$1" pin="TP"/>
+</segment>
+</net>
+<net name="N$13" class="0">
+<segment>
+<pinref part="U$1" gate="G$1" pin="23/A9"/>
+<pinref part="TP2" gate="G$1" pin="TP"/>
+</segment>
+</net>
+<net name="N$15" class="0">
+<segment>
+<pinref part="U$1" gate="G$1" pin="22/A8"/>
+<pinref part="TP3" gate="G$1" pin="TP"/>
+</segment>
+</net>
+<net name="N$16" class="0">
+<segment>
+<pinref part="U$1" gate="G$1" pin="21/A7"/>
+<pinref part="TP4" gate="G$1" pin="TP"/>
+</segment>
+</net>
+<net name="N$17" class="0">
+<segment>
+<pinref part="U$1" gate="G$1" pin="20/A6"/>
+<pinref part="TP5" gate="G$1" pin="TP"/>
+</segment>
+</net>
+<net name="N$18" class="0">
+<segment>
+<pinref part="U$1" gate="G$1" pin="19/A5/SCL"/>
+<pinref part="TP6" gate="G$1" pin="TP"/>
+</segment>
+</net>
+<net name="N$19" class="0">
+<segment>
+<pinref part="U$1" gate="G$1" pin="17/A3"/>
+<pinref part="TP7" gate="G$1" pin="TP"/>
+</segment>
+</net>
+<net name="N$20" class="0">
+<segment>
+<pinref part="U$1" gate="G$1" pin="18/A4/SDA"/>
+<pinref part="TP8" gate="G$1" pin="TP"/>
+</segment>
+</net>
+<net name="N$21" class="0">
+<segment>
+<pinref part="U$1" gate="G$1" pin="16/A2"/>
+<pinref part="TP9" gate="G$1" pin="TP"/>
+</segment>
+</net>
+<net name="N$22" class="0">
+<segment>
+<pinref part="U$1" gate="G$1" pin="15/A1"/>
+<pinref part="TP10" gate="G$1" pin="TP"/>
+</segment>
+</net>
+<net name="N$26" class="0">
+<segment>
+<pinref part="U$1" gate="G$1" pin="14/A0"/>
+<pinref part="TP11" gate="G$1" pin="TP"/>
+</segment>
+</net>
+<net name="N$27" class="0">
+<segment>
+<pinref part="U$1" gate="G$1" pin="13/SCK"/>
+<pinref part="TP12" gate="G$1" pin="TP"/>
+</segment>
+</net>
+<net name="N$28" class="0">
+<segment>
+<pinref part="U$1" gate="G$1" pin="GND2"/>
+<pinref part="TP13" gate="G$1" pin="TP"/>
+</segment>
+</net>
+<net name="N$29" class="0">
+<segment>
+<pinref part="U$1" gate="G$1" pin="A22/DAC1"/>
+<pinref part="TP14" gate="G$1" pin="TP"/>
+</segment>
+</net>
+<net name="N$30" class="0">
+<segment>
+<pinref part="U$1" gate="G$1" pin="A21/DAC0"/>
+<pinref part="TP15" gate="G$1" pin="TP"/>
+</segment>
+</net>
+<net name="N$31" class="0">
+<segment>
+<pinref part="U$1" gate="G$1" pin="3V3"/>
+<pinref part="TP16" gate="G$1" pin="TP"/>
+</segment>
+</net>
+<net name="N$33" class="0">
+<segment>
+<pinref part="U$1" gate="G$1" pin="AGND"/>
+<pinref part="TP17" gate="G$1" pin="TP"/>
+</segment>
+</net>

Commit message: V0 of driver board needs checked
Parts:
- added TP21, TP22, TP23, TP24, TP25, TP26, TP27, TP28, TP29, TP30, TP31, TP32, TP33, TP34, TP35, TP36, TP37, TP38, TP39, TP40, TP41: TPSQPAD1-13Y, testpad:TPSQPAD1-13Y
- DATA_1, DATA_2, DATA_3: device con-lstb:MA05-2 -> Pin_headers:MA05-2
Connections:
- net 65: now also TP25.TP
- net 66: now also TP24.TP
- net 69: now also TP30.TP
- net 70: now also TP29.TP
- net GND: now also TP26.TP, TP31.TP
- net N$1: now also TP35.TP
- net N$3: now also TP36.TP
- net N$32: now also TP37.TP
- net N$5: now also TP21.TP
- net TEENSY_DATA_4: now also TP34.TP
- net TEENSY_DATA_5: now also TP41.TP
- net TEENSY_DATA_6: now also TP40.TP
- net TEENSY_DATA_7: now also TP39.TP
- net TEENSY_DATA_8: now also TP38.TP
- net TO_TRAN_65: now also TP23.TP
- net TO_TRAN_66: now also TP22.TP
- net TO_TRAN_69: now also TP27.TP
- net TO_TRAN_70: now also TP28.TP
- net VDD: now also TP32.TP, TP33.TP
