File: eagle/ProjectX/Transducer_board_niall.sch (EAGLE design)
At the start: 104 parts, among them T1 MA40S4S, T10 MA40S4S, T100 MA40S4S, T11 MA40S4S, T12 MA40S4S, T13 MA40S4S, T14 MA40S4S, T15 MA40S4S, T16 MA40S4S, T17 MA40S4S, T18 MA40S4S, T19 MA40S4S, T2 MA40S4S, T20 MA40S4S, T21 MA40S4S, T22 MA40S4S, T23 MA40S4S, T24 MA40S4S, T25 MA40S4S, T26 MA40S4S, T27 MA40S4S, T28 MA40S4S, T29 MA40S4S, T3 MA40S4S, T30 MA40S4S, T31 MA40S4S, T32 MA40S4S, T33 MA40S4S, T34 MA40S4S, T35 MA40S4S, T36 MA40S4S, T37 MA40S4S, T38 MA40S4S, T39 MA40S4S, T4 MA40S4S, T40 MA40S4S, T41 MA40S4S, T42 MA40S4S, T43 MA40S4S, T44 MA40S4S, T45 MA40S4S, T46 MA40S4S, T47 MA40S4S, T48 MA40S4S, T49 MA40S4S, T5 MA40S4S, T50 MA40S4S, T51 MA40S4S, T52 MA40S4S, T53 MA40S4S, T54 MA40S4S, T55 MA40S4S, T56 MA40S4S, T57 MA40S4S, T58 MA40S4S, T59 MA40S4S, T6 MA40S4S, T60 MA40S4S, T61 MA40S4S, T62 MA40S4S, T63 MA40S4S, T64 MA40S4S, T65 MA40S4S, T66 MA40S4S, T67 MA40S4S, T68 MA40S4S, T69 MA40S4S, T7 MA40S4S, T70 MA40S4S, T71 MA40S4S, T72 MA40S4S, T73 MA40S4S, T74 MA40S4S, T75 MA40S4S, T76 MA40S4S, T77 MA40S4S, T78 MA40S4S, T79 MA40S4S, T8 MA40S4S, T80 MA40S4S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

Commit message: Tangled web
Connections:
- net FROM_T_11: now also 4.49
- net FROM_T_12: now also 4.44
- net FROM_T_13: now also 4.37
- net FROM_T_14: now also 4.33
- net FROM_T_15: now also 4.28
- net FROM_T_16: now also 4.24
- net FROM_T_25: now also 4.21
- net FROM_T_26: now also 4.41
- net FROM_T_27: now also 4.32
- net FROM_T_29: now also 4.29
- net FROM_T_30: now also 4.48
- net FROM_T_5: now also 4.25
- net FROM_T_7: now also 4.36
- net FROM_T_8: now also 4.40
- net FROM_T_9: now also 4.45
- net TO_T_11: now also 4.50
- net TO_T_12: now also 4.43
- net TO_T_13: now also 4.38
- net TO_T_14: now also 4.34
- net TO_T_15: now also 4.27
- net TO_T_16: now also 4.23
- net TO_T_25: now also 4.22
- net TO_T_26: now also 4.42
- net TO_T_27: now also 4.31
- net TO_T_29: now also 4.30
- net TO_T_30: now also 4.47
- net TO_T_5: now also 4.26
- net TO_T_7: now also 4.35
- net TO_T_8: now also 4.39
- net TO_T_9: now also 4.46
Changed lines of the file:
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@@
 <pinref part="T5" gate="G$1" pin="1"/>
+</segment>
+<segment>
+<pinref part="4" gate="G$1" pin="25"/>
+<wire x1="-195.58" y1="154.94" x2="-170.18" y2="154.94" width="0.1524" layer="91" style="shortdash"/>
+<label x="-190.5" y="154.94" size="1.778" layer="95"/>
 </segment>
 </net>
@@
 <pinref part="T5" gate="G$1" pin="2"/>
 </segment>
+<segment>
+<pinref part="4" gate="G$1" pin="26"/>
+<wire x1="-210.82" y1="154.94" x2="-231.14" y2="154.94" width="0.1524" layer="91"/>
+<label x="-226.06" y="154.94" size="1.778" layer="95"/>
+</segment>
 </net>
 <net name="FROM_T_6" class="0">
@@
 <pinref part="T7" gate="G$1" pin="1"/>
 </segment>
+<segment>
+<pinref part="4" gate="G$1" pin="36"/>
+<wire x1="-210.82" y1="167.64" x2="-228.6" y2="167.64" width="0.1524" layer="91" style="shortdash"/>
+<label x="-226.06" y="167.64" size="1.778" layer="95"/>
+</segment>
 </net>
 <net name="TO_T_7" class="0">
@@
 <pinref part="T7" gate="G$1" pin="2"/>
 </segment>
+<segment>
+<pinref part="4" gate="G$1" pin="35"/>
+<wire x1="-195.58" y1="167.64" x2="-172.72" y2="167.64" width="0.1524" layer="91"/>
+<label x="-190.5" y="167.64" size="1.778" layer="95"/>
+</segment>
 </net>
 <net name="FROM_T_8" class="0">
@@
 <pinref part="T8" gate="G$1" pin="1"/>
 </segment>
+<segment>
+<pinref part="4" gate="G$1" pin="40"/>
+<wire x1="-210.82" y1="172.72" x2="-228.6" y2="172.72" width="0.1524" layer="91" style="shortdash"/>
+<label x="-226.06" y="172.72" size="1.778" layer="95"/>
+</segment>
 </net>
 <net name="TO_T_8" class="0">
@@
 <pinref part="T8" gate="G$1" pin="2"/>
 </segment>
+<segment>
+<pinref part="4" gate="G$1" pin="39"/>
+<wire x1="-195.58" y1="172.72" x2="-172.72" y2="172.72" width="0.1524" layer="91"/>
+<label x="-190.5" y="172.72" size="1.778" layer="95"/>
+</segment>
 </net>
 <net name="FROM_T_9" class="0">
@@
 <pinref part="T9" gate="G$1" pin="1"/>
 </segment>
+<segment>
+<pinref part="4" gate="G$1" pin="45"/>
+<wire x1="-195.58" y1="180.34" x2="-170.18" y2="180.34" width="0.1524" layer="91" style="dashdot"/>
+<label x="-190.5" y="180.34" size="1.778" layer="95"/>
+</segment>
 </net>
 <net name="TO_T_9" class="0">
@@
 <pinref part="T9" gate="G$1" pin="2"/>
 </segment>
+<segment>
+<pinref part="4" gate="G$1" pin="46"/>
+<wire x1="-210.82" y1="180.34" x2="-231.14" y2="180.34" width="0.1524" layer="91"/>
+<label x="-226.06" y="180.34" size="1.778" layer="95"/>
+</segment>
 </net>
 <net name="FROM_T_10" class="0">
@@
 <pinref part="T11" gate="G$1" pin="1"/>
 </segment>
+<segment>
+<pinref part="4" gate="G$1" pin="49"/>
+<wire x1="-195.58" y1="185.42" x2="-170.18" y2="185.42" width="0.1524" layer="91" style="dashdot"/>
+<label x="-190.5" y="185.42" size="1.778" layer="95"/>
+</segment>
 </net>
 <net name="TO_T_11" class="0">
@@
 <pinref part="T11" gate="G$1" pin="2"/>
 </segment>
+<segment>
+<pinref part="4" gate="G$1" pin="50"/>
+<wire x1="-210.82" y1="185.42" x2="-231.14" y2="185.42" width="0.1524" layer="91"/>
+<label x="-226.06" y="185.42" size="1.778" layer="95"/>
+</segment>
 </net>
 <net name="FROM_T_12" class="0">
@@
 <pinref part="T12" gate="G$1" pin="1"/>
 </segment>
+<segment>
+<pinref part="4" gate="G$1" pin="44"/>
+<wire x1="-210.82" y1="177.8" x2="-228.6" y2="177.8" width="0.1524" layer="91" style="shortdash"/>
+<label x="-226.06" y="177.8" size="1.778" layer="95"/>
+</segment>
 </net>
 <net name="TO_T_12" class="0">
@@
 <pinref part="T12" gate="G$1" pin="2"/>
 </segment>
+<segment>
+<pinref part="4" gate="G$1" pin="43"/>
+<wire x1="-195.58" y1="177.8" x2="-172.72" y2="177.8" width="0.1524" layer="91"/>
+<label x="-190.5" y="177.8" size="1.778" layer="95"/>
+</segment>
 </net>
 <net name="FROM_T_13" class="0">
@@
 <pinref part="T13" gate="G$1" pin="1"/>
 </segment>
+<segment>
+<pinref part="4" gate="G$1" pin="37"/>
+<wire x1="-195.58" y1="170.18" x2="-170.18" y2="170.18" width="0.1524" layer="91" style="shortdash"/>
+<label x="-190.5" y="170.18" size="1.778" layer="95"/>
+</segment>
 </net>
 <net name="TO_T_13" class="0">
@@
 <pinref part="T13" gate="G$1" pin="2"/>
 </segment>
+<segment>
+<pinref part="4" gate="G$1" pin="38"/>
+<wire x1="-210.82" y1="170.18" x2="-231.14" y2="170.18" width="0.1524" layer="91"/>
+<label x="-226.06" y="170.18" size="1.778" layer="95"/>
+</segment>
 </net>
 <net name="FROM_T_14" class="0">
@@
 <pinref part="T14" gate="G$1" pin="1"/>
 </segment>
+<segment>
+<pinref part="4" gate="G$1" pin="33"/>
+<wire x1="-195.58" y1="165.1" x2="-170.18" y2="165.1" width="0.1524" layer="91" style="shortdash"/>
+<label x="-190.5" y="165.1" size="1.778" layer="95"/>
+</segment>
 </net>
 <net name="TO_T_14" class="0">
@@
 <pinref part="T14" gate="G$1" pin="2"/>
 </segment>
+<segment>
+<pinref part="4" gate="G$1" pin="34"/>
+<wire x1="-210.82" y1="165.1" x2="-231.14" y2="165.1" width="0.1524" layer="91"/>
+<label x="-226.06" y="165.1" size="1.778" layer="95"/>
+</segment>
 </net>
 <net name="FROM_T_15" class="0">
@@
 <pinref part="T15" gate="G$1" pin="1"/>
 </segment>
+<segment>
+<pinref part="4" gate="G$1" pin="28"/>
+<wire x1="-210.82" y1="157.48" x2="-228.6" y2="157.48" width="0.1524" layer="91" style="shortdash"/>
+<label x="-226.06" y="157.48" size="1.778" layer="95"/>
+</segment>
 </net>
 <net name="TO_T_15" class="0">
@@
 <pinref part="T15" gate="G$1" pin="2"/>
 </segment>
+<segment>
+<pinref part="4" gate="G$1" pin="27"/>
+<wire x1="-195.58" y1="157.48" x2="-172.72" y2="157.48" width="0.1524" layer="91"/>
+<label x="-190.5" y="157.48" size="1.778" layer="95"/>
+</segment>
 </net>
 <net name="FROM_T_16" class="0">
@@
 <pinref part="T16" gate="G$1" pin="1"/>
 </segment>
+<segment>
+<pinref part="4" gate="G$1" pin="24"/>
+<wire x1="-210.82" y1="152.4" x2="-228.6" y2="152.4" width="0.1524" layer="91" style="shortdash"/>
+<label x="-226.06" y="152.4" size="1.778" layer="95"/>
+</segment>
 </net>
 <net name="TO_T_16" class="0">
@@
 <pinref part="T16" gate="G$1" pin="2"/>
 </segment>
+<segment>
+<pinref part="4" gate="G$1" pin="23"/>
+<wire x1="-195.58" y1="152.4" x2="-172.72" y2="152.4" width="0.1524" layer="91"/>
+<label x="-190.5" y="152.4" size="1.778" layer="95"/>
+</segment>
 </net>
 <net name="FROM_T_17" class="0">
@@
 <pinref part="T25" gate="G$1" pin="1"/>
 </segment>
+<segment>
+<pinref part="4" gate="G$1" pin="21"/>
+<wire x1="-195.58" y1="149.86" x2="-170.18" y2="149.86" width="0.1524" layer="91" style="shortdash"/>
+<label x="-190.5" y="149.86" size="1.778" layer="95"/>
+</segment>
 </net>
 <net name="TO_T_25" class="0">
@@
 <pinref part="T25" gate="G$1" pin="2"/>
 </segment>
+<segment>
+<pinref part="4" gate="G$1" pin="22"/>
+<wire x1="-210.82" y1="149.86" x2="-231.14" y2="149.86" width="0.1524" layer="91"/>
+<label x="-226.06" y="149.86" size="1.778" layer="95"/>
+</segment>
 </net>
 <net name="FROM_T_26" class="0">
@@
 <pinref part="T26" gate="G$1" pin="1"/>
 </segment>
+<segment>
+<pinref part="4" gate="G$1" pin="41"/>
+<wire x1="-195.58" y1="175.26" x2="-170.18" y2="175.26" width="0.1524" layer="91" style="shortdash"/>
+<label x="-190.5" y="175.26" size="1.778" layer="95"/>
+</segment>
 </net>
 <net name="TO_T_26" class="0">
@@
 <pinref part="T26" gate="G$1" pin="2"/>
 </segment>
+<segment>
+<pinref part="4" gate="G$1" pin="42"/>
+<wire x1="-210.82" y1="175.26" x2="-231.14" y2="175.26" width="0.1524" layer="91"/>
+<label x="-226.06" y="175.26" size="1.778" layer="95"/>
+</segment>
 </net>
 <net name="FROM_T_27" class="0">
@@
 <pinref part="T27" gate="G$1" pin="1"/>
 </segment>
+<segment>
+<pinref part="4" gate="G$1" pin="32"/>
+<wire x1="-210.82" y1="162.56" x2="-228.6" y2="162.56" width="0.1524" layer="91" style="shortdash"/>
+<label x="-226.06" y="162.56" size="1.778" layer="95"/>
+</segment>
 </net>
 <net name="TO_T_27" class="0">
@@
 <pinref part="T27" gate="G$1" pin="2"/>
 </segment>
+<segment>
+<pinref part="4" gate="G$1" pin="31"/>
+<wire x1="-195.58" y1="162.56" x2="-172.72" y2="162.56" width="0.1524" layer="91"/>
+<label x="-190.5" y="162.56" size="1.778" layer="95"/>
+</segment>
 </net>
 <net name="FROM_T_28" class="0">
@@
 <pinref part="T29" gate="G$1" pin="1"/>
 </segment>
+<segment>
+<pinref part="4" gate="G$1" pin="29"/>
+<wire x1="-195.58" y1="160.02" x2="-170.18" y2="160.02" width="0.1524" layer="91" style="shortdash"/>
+<label x="-190.5" y="160.02" size="1.778" layer="95"/>
+</segment>
 </net>
 <net name="TO_T_29" class="0">
@@
 <pinref part="T29" gate="G$1" pin="2"/>
 </segment>
+<segment>
+<pinref part="4" gate="G$1" pin="30"/>
+<wire x1="-210.82" y1="160.02" x2="-231.14" y2="160.02" width="0.1524" layer="91"/>
+<label x="-226.06" y="160.02" size="1.778" layer="95"/>
+</segment>
 </net>
 <net name="FROM_T_30" class="0">
@@
 <pinref part="T30" gate="G$1" pin="1"/>
 </segment>
+<segment>
+<pinref part="4" gate="G$1" pin="48"/>
+<wire x1="-210.82" y1="182.88" x2="-228.6" y2="182.88" width="0.1524" layer="91" style="dashdot"/>
+<label x="-226.06" y="182.88" size="1.778" layer="95"/>
+</segment>
 </net>
 <net name="TO_T_30" class="0">
@@
 <pinref part="T30" gate="G$1" pin="2"/>
 </segment>
-</net>
+<segment>
+<pinref part="4" gate="G$1" pin="47"/>
+<wire x1="-195.58" y1="182.88" x2="-172.72" y2="182.88" width="0.1524" layer="91"/>
+<label x="-190.5" y="182.88" size="1.778" layer="95"/>
+</segment>
+</net>

Commit message: Niall board better wiring
Connections:
- net FROM_T_12: now also 4.48; no longer 4.44
- net FROM_T_13: now also 4.44; no longer 4.37
- net FROM_T_14: now also 4.40; no longer 4.33
- net FROM_T_15: now also 4.36; no longer 4.28
- net FROM_T_16: now also 4.32; no longer 4.24
- net FROM_T_17: now also 4.28; no longer 4.17
- net FROM_T_18: now also 4.24; no longer 4.12
- net FROM_T_2: now also 4.9; no longer 4.8
- net FROM_T_20: now also 4.13; no longer 4.4
- net FROM_T_21: now also 4.17; no longer 4.1
- net FROM_T_23: now also 4.21; no longer 4.9
- net FROM_T_24: now also 4.25; no longer 4.16
- net FROM_T_25: now also 4.45; no longer 4.21
- net FROM_T_27: now also 4.37; no longer 4.32
- net FROM_T_29: now also 4.33; no longer 4.29
- net FROM_T_3: now also 4.1; no longer 4.13
- net FROM_T_30: now also 4.29; no longer 4.48
- net FROM_T_4: now also 4.4; no longer 4.20
- net FROM_T_5: now also 4.8; no longer 4.25
- net FROM_T_7: now also 4.12; no longer 4.36
- net FROM_T_8: now also 4.16; no longer 4.40
- net FROM_T_9: now also 4.20; no longer 4.45
- net TO_T_12: now also 4.46; no longer 4.43
- net TO_T_13: now also 4.42; no longer 4.38
- net TO_T_14: now also 4.38; no longer 4.34
- net TO_T_15: now also 4.34; no longer 4.27
- net TO_T_16: now also 4.30; no longer 4.23
- net TO_T_17: now also 4.26; no longer 4.18
- net TO_T_18: now also 4.22; no longer 4.11
- net TO_T_19: now also 4.7; no longer 4.6
- net TO_T_2: now also 4.11; no longer 4.7
- net TO_T_20: now also 4.15; no longer 4.3
- net TO_T_21: now also 4.19; no longer 4.2
- net TO_T_23: now also 4.23; no longer 4.10
- net TO_T_24: now also 4.27; no longer 4.15
- net TO_T_25: now also 4.47; no longer 4.22
- net TO_T_26: now also 4.43; no longer 4.42
- net TO_T_27: now also 4.39; no longer 4.31
- net TO_T_29: now also 4.35; no longer 4.30
- net TO_T_3: now also 4.3; no longer 4.14
- net TO_T_30: now also 4.31; no longer 4.47
- net TO_T_4: now also 4.2; no longer 4.19
- net TO_T_5: now also 4.6; no longer 4.26
- net TO_T_7: now also 4.10; no longer 4.35
- net TO_T_8: now also 4.14; no longer 4.39
- net TO_T_9: now also 4.18; no longer 4.46
