File: eagle/ProjectX/Transducer_board_niall.brd (EAGLE design)
At the start: 100 x 100 mm, 104 parts

Commit message: Finished board 1
Routing:
- net FROM_T_3: track 23.9 -> 26.4 mm
- net FROM_T_23: track 15.9 -> 17.9 mm
- net FROM_T_19: track 18.6 -> 16.7 mm
- net TO_T_3: track 31.8 -> 33.4 mm, vias 1 -> 3
- net TO_T_19: track 16.7 -> 18.0 mm

Commit message: Transducer board tidied up a bit and submitted
Routing:
- net TO_T_84: track 39.0 -> 3.57 mm
- net TO_T_89: track 42.1 -> 8.05 mm
- net FROM_T_89: track 37.9 -> 7.94 mm
- net FROM_T_84: track 33.7 -> 4.15 mm
- net TO_T_97: track 41.0 -> 15.1 mm
- net FROM_T_97: track 34.7 -> 17.1 mm, vias 1 -> 2
- net TO_T_9: track 87.2 -> 78.2 mm
- net FROM_T_64: track 35.2 -> 27.0 mm, vias 1 -> 3
- net FROM_T_9: track 85.2 -> 77.1 mm, vias 1 -> 3
- net TO_T_92: track 21.6 -> 13.6 mm
- net TO_T_69: track 20.7 -> 28.6 mm, vias 1 -> 2
- net TO_T_91: track 26.9 -> 34.4 mm, vias 2 -> 4
- net TO_T_64: track 36.3 -> 29.1 mm
- net TO_T_98: track 31.3 -> 26.8 mm
- net FROM_T_62: track 30.9 -> 27.1 mm
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